Commit message: Implementing a simple air pressure sensor

File: rotors_description/urdf/atlantik_solar.xacro (robot description, xacro)
@@ -22,6 +22,6 @@
   <xacro:property name="use_mesh_file" value="false" />
   <xacro:property name="mesh_file" value="" />
-  <xacro:property name="mass_fuselage" value="10.0" /> <!-- [kg] -->
-  <xacro:property name="mass_front_wing" value="5.0" /> <!-- [kg] -->
+  <xacro:property name="mass_fuselage" value="1.0" /> <!-- [kg] -->
+  <xacro:property name="mass_front_wing" value="1.0" /> <!-- [kg] -->
   <xacro:property name="body_length" value="3.0" /> <!-- [m] -->
   <xacro:property name="body_width" value="0.3" /> <!-- [m] -->
@@ -31,5 +31,9 @@
   <xacro:property name="front_wing_height" value="0.02" /> <!-- [m] -->
   <xacro:property name="front_wing_dihedral_angle" value="5" /> <!-- [deg] -->
-  <xacro:property name="PI" value="3.14159" /> <!-- [deg] -->
+  <xacro:property name="alpha_0" value="0.0" /> <!-- [deg] -->
+  <xacro:property name="alpha_stall" value="15.0" /> <!-- [deg] -->
+  <xacro:property name="c_L_alpha" value="${2.0 * PI}" />
+  <xacro:property name="air_density" value="1.225" /> <!-- [kg/m^3] -->
+  <xacro:property name="PI" value="3.1415926535897931" />
   <!-- Front wing length -->
   <xacro:property name="front_wing_length" value="${0.5 * (wingspan - body_width) /
@@ -66,5 +70,9 @@
     wing_height="${front_wing_height}"
     use_mesh="false"
-    mesh="">
+    mesh=""
+    alpha_0="${alpha_0}"
+    alpha_stall="${alpha_stall}"
+    c_L_alpha="${c_L_alpha}"
+    air_density="${air_density}">
     <origin xyz="0.5 ${0.25 * (wingspan + body_width)} ${0.5*body_height}" rpy="0.0 ${front_wing_dihedral_angle*PI/180.0} -1.57" />
     <xacro:insert_block name="front_wing_inertia" />
@@ -79,5 +87,9 @@
     wing_height="${front_wing_height}"
     use_mesh="false"
-    mesh="">
+    mesh=""
+    alpha_0="${alpha_0}"
+    alpha_stall="${alpha_stall}"
+    c_L_alpha="${c_L_alpha}"
+    air_density="${air_density}">
     <origin xyz="0.5 ${-0.25 * (wingspan + body_width)} ${0.5*body_height}" rpy="0.0 ${front_wing_dihedral_angle*PI/180.0} 1.57" />
     <xacro:insert_block name="front_wing_inertia" />

File: rotors_description/urdf/atlantik_solar_base.xacro (robot description, xacro)
@@ -28,4 +28,6 @@
   <!-- Mount a magnetometer. -->
   <xacro:default_magnetometer namespace="${namespace}" parent_link="${namespace}/base_link" />
+  <!-- Mount a pressure sensor. -->
+  <xacro:default_pressure_sensor namespace="${namespace}" parent_link="${namespace}/base_link" />
   <xacro:if value="$(arg enable_ground_truth)">
     <xacro:ground_truth_imu_and_odometry namespace="${namespace}" parent_link="${namespace}/base_link" />

File: rotors_description/urdf/component_snippets.xacro (robot description, xacro)
@@ -375,5 +375,5 @@
   </link>
   <!-- GPS joint -->
-  <joint name="${namespace}/gps${gps_suffix}_link" type="revolute">
+  <joint name="${namespace}/gps${gps_suffix}_joint" type="revolute">
     <xacro:insert_block name="origin" />
     <parent link="${parent_link}" />
@@ -409,5 +409,5 @@
   </link>
   <!-- Magnetometer joint -->
-  <joint name="${namespace}/magnetometer${magnetometer_suffix}_link" type="revolute">
+  <joint name="${namespace}/magnetometer${magnetometer_suffix}_joint" type="revolute">
     <xacro:insert_block name="origin" />
     <parent link="${parent_link}" />
@@ -427,4 +427,33 @@
       <referenceMagEast>${reference_magnetic_field_east}</referenceMagEast>
       <referenceMagDown>${reference_magnetic_field_down}</referenceMagDown>
+    </plugin>
+  </gazebo>
+  </xacro:macro>
+  <!-- Macro to add an air pressure sensor. -->
+  <xacro:macro name="pressure_sensor_plugin_macro"
+    params="namespace pressure_sensor_suffix parent_link pressure_topic mass_pressure_sensor
+      reference_altitude pressure_variance *inertia *origin">
+  <!-- Pressure sensor link -->
+  <link name="${namespace}/pressure_sensor${pressure_sensor_suffix}_link">
+    <inertial>
+      <xacro:insert_block name="inertia" />
+      <mass value="${mass_pressure_sensor}" />  <!-- [kg] -->
+      <origin xyz="0 0 0" rpy="0 0 0" />
+    </inertial>
+  </link>
+  <!-- Pressure sensor joint -->
+  <joint name="${namespace}/pressure_sensor${pressure_sensor_suffix}_joint" type="revolute">
+    <xacro:insert_block name="origin" />
+    <parent link="${parent_link}" />
+    <child link="${namespace}/pressure_sensor${pressure_sensor_suffix}_link" />
+    <limit upper="0" lower="0" effort="0" velocity="0" />
+  </joint>
+  <gazebo>
+    <plugin filename="librotors_gazebo_pressure_plugin.so" name="rotors_gazebo_pressure_sensor${pressure_sensor_suffix}_plugin">
+      <robotNamespace>${namespace}</robotNamespace> <!-- (string, required): ros namespace in which the messages are published -->
+      <linkName>${namespace}/pressure_sensor${pressure_sensor_suffix}_link</linkName> <!-- (string, required): name of the body which holds the pressure sensor -->
+      <pressureTopic>${pressure_topic}</pressureTopic> <!-- (string): name of the sensor output topic and prefix of service names (defaults to 'air_pressure') -->
+      <referenceAltitude>${reference_altitude}</referenceAltitude> <!-- the initial altitude [m] -->
+      <pressureVariance>${pressure_variance}</pressureVariance> <!-- the air pressure variance [Pa^2] -->
     </plugin>
   </gazebo>
@@ -741,3 +770,16 @@
     </xacro:magnetometer_plugin_macro>
   </xacro:macro>
+  <xacro:macro name="default_pressure_sensor" params="namespace parent_link">
+    <xacro:pressure_sensor_plugin_macro
+      namespace="${namespace}"
+      pressure_sensor_suffix=""
+      parent_link="${parent_link}"
+      pressure_topic="air_pressure"
+      mass_pressure_sensor="0.015"
+      reference_altitude="500.0"
+      pressure_variance="0.0">
+      <inertia ixx="0.00001" ixy="0.0" ixz="0.0" iyy="0.00001" iyz="0.0" izz="0.00001" />
+      <origin xyz="0 0 0" rpy="0 0 0" />
+    </xacro:pressure_sensor_plugin_macro>
+  </xacro:macro>
 </robot>

File: rotors_description/urdf/fixed_wing_base.xacro (robot description, xacro)
@@ -64,9 +64,15 @@
       </collision>
     </link>
+    <gazebo>
+      <plugin name="fixed_wing_base_plugin" filename="librotors_gazebo_fixedwing_base_plugin.so">
+        <robotNamespace>${robot_namespace}</robotNamespace>
+        <linkName>${robot_namespace}/base_link</linkName>
+      </plugin>
+    </gazebo>
   </xacro:macro>
   <!-- Wing joint and link -->
   <xacro:macro name="wing"
-    params="robot_namespace suffix parent mass_wing
-      wing_length wing_width wing_height use_mesh mesh *origin *inertia">
+    params="robot_namespace suffix parent mass_wing wing_length wing_width wing_height
+      use_mesh mesh alpha_0 alpha_stall c_L_alpha air_density *origin *inertia">
     <joint name="${robot_namespace}/wing_${suffix}_joint" type="revolute">
       <xacro:insert_block name="origin" />
@@ -102,4 +108,9 @@
         <robotNamespace>${robot_namespace}</robotNamespace>
         <linkName>${robot_namespace}/wing_${suffix}</linkName>
+        <alpha0>${alpha_0}</alpha0> <!-- the starting angle of attack [deg] -->
+        <alphaStall>${alpha_stall}</alphaStall> <!-- stall angle [deg] -->
+        <cLAlpha>${c_L_alpha}</cLAlpha> <!-- coefficient of lift to angle of attack ratio -->
+        <airDensity>${air_density}</airDensity> <!-- air density [kg/m^3] -->
+        <wingArea>${wing_length * wing_width}</wingArea> <!-- area of the wing [m^2] -->
       </plugin>
     </gazebo>

Commit message: Adding rear wings and the mavlink interface package

File: rotors_description/urdf/atlantik_solar.xacro (robot description, xacro)
@@ -24,4 +24,6 @@
   <xacro:property name="mass_fuselage" value="1.0" /> <!-- [kg] -->
   <xacro:property name="mass_front_wing" value="1.0" /> <!-- [kg] -->
+  <xacro:property name="mass_tail" value="1.0" /> <!-- [kg] -->
+  <xacro:property name="mass_rear_wing" value="1.0" /> <!-- [kg] -->
   <xacro:property name="body_length" value="3.0" /> <!-- [m] -->
   <xacro:property name="body_width" value="0.3" /> <!-- [m] -->
@@ -31,4 +33,9 @@
   <xacro:property name="front_wing_height" value="0.02" /> <!-- [m] -->
   <xacro:property name="front_wing_dihedral_angle" value="5" /> <!-- [deg] -->
+  <xacro:property name="tail_length" value="0.4" /> <!-- [m] -->
+  <xacro:property name="tail_width" value="0.05" /> <!-- [m] -->
+  <xacro:property name="tail_height" value="0.3" /> <!-- [m] -->
+  <xacro:property name="rear_wingspan" value="1.0" /> <!-- [m] -->
+  <xacro:property name="rear_wing_height" value="0.02" /> <!-- [m] -->
   <xacro:property name="alpha_0" value="0.0" /> <!-- [deg] -->
   <xacro:property name="alpha_stall" value="15.0" /> <!-- [deg] -->
@@ -39,4 +46,6 @@
   <xacro:property name="front_wing_length" value="${0.5 * (wingspan - body_width) /
     (1.0 - 0.5 * (front_wing_dihedral_angle * front_wing_dihedral_angle * PI * PI / (180.0 * 180.0)))}" />
+  <!-- Rear wing length -->
+  <xacro:property name="rear_wing_length" value="${0.5 * (rear_wingspan - tail_width)}" />
   <!-- Inertia of the fuselage -->
   <xacro:property name="body_inertia">
@@ -45,5 +54,13 @@
   <!-- Inertia of a single front wing, assuming it is a cuboid -->
   <xacro:property name="front_wing_inertia">
-    <xacro:box_inertia x="${front_wing_length}" y="${root_chord}" z="${front_wing_height}" mass="${mass_front_wing}" />
+    <xacro:box_inertia x="${front_wing_length}" y="${tail_length}" z="${rear_wing_height}" mass="${mass_front_wing}" />
+  </xacro:property>
+  <!-- Inertia of the tail, assuming it is a cuboid -->
+  <xacro:property name="tail_inertia">
+    <xacro:box_inertia x="${tail_length}" y="${tail_width}" z="${tail_height}" mass="${mass_tail}" />
+  </xacro:property>
+  <!-- Inertia of a single rear wing, assuming it is a cuboid -->
+  <xacro:property name="rear_wing_inertia">
+    <xacro:box_inertia x="${rear_wing_length}" y="${tail_width}" z="${tail_height}" mass="${mass_rear_wing}" />
   </xacro:property>
   <!-- Included URDF Files -->
@@ -63,5 +80,5 @@
   <xacro:wing
     robot_namespace="${namespace}"
-    suffix="front_left"
+    suffix="left"
     parent="${namespace}/base_link"
     mass_wing="${mass_front_wing}"
@@ -75,10 +92,10 @@
     c_L_alpha="${c_L_alpha}"
     air_density="${air_density}">
-    <origin xyz="0.5 ${0.25 * (wingspan + body_width)} ${0.5*body_height}" rpy="0.0 ${front_wing_dihedral_angle*PI/180.0} -1.57" />
+    <origin xyz="0.5 ${0.25 * (wingspan + body_width)} ${0.5*body_height}" rpy="0.0 ${front_wing_dihedral_angle*PI/180.0} ${-PI*0.5}" />
     <xacro:insert_block name="front_wing_inertia" />
   </xacro:wing>
   <xacro:wing
     robot_namespace="${namespace}"
-    suffix="front_right"
+    suffix="right"
     parent="${namespace}/base_link"
     mass_wing="${mass_front_wing}"
@@ -92,6 +109,46 @@
     c_L_alpha="${c_L_alpha}"
     air_density="${air_density}">
-    <origin xyz="0.5 ${-0.25 * (wingspan + body_width)} ${0.5*body_height}" rpy="0.0 ${front_wing_dihedral_angle*PI/180.0} 1.57" />
+    <origin xyz="0.5 ${-0.25 * (wingspan + body_width)} ${0.5*body_height}" rpy="0.0 ${front_wing_dihedral_angle*PI/180.0} ${PI*0.5}" />
     <xacro:insert_block name="front_wing_inertia" />
   </xacro:wing>
+  <!-- Instantiate the tail -->
+  <xacro:tail
+    robot_namespace="${namespace}"
+    parent="${namespace}/base_link"
+    mass_tail="${mass_tail}"
+    tail_length="${tail_length}"
+    tail_width="${tail_width}"
+    tail_height="${tail_height}"
+    use_mesh="false"
+    mesh="">
+    <origin xyz="${-0.5*body_length + 0.5*tail_length} 0.0 ${0.5*body_height + 0.5*tail_height}" rpy="0.0 0.0 0.0" />
+    <xacro:insert_block name="tail_inertia" />
+  </xacro:tail>
+  <!-- Instantiate the rear wings-->
+  <xacro:rear_wing
+    robot_namespace="${namespace}"
+    suffix="left"
+    parent="${namespace}/tail"
+    mass_rear_wing="${mass_rear_wing}"
+    rear_wing_length="${rear_wing_length}"
+    rear_wing_width="${tail_length}"
+    rear_wing_height="${rear_wing_height}"
+    use_mesh="false"
+    mesh="">
+    <origin xyz="0.0 ${0.25 * (rear_wingspan + tail_width)} ${0.5 * (tail_height - rear_wing_height)}" rpy="0.0 0.0 ${PI*0.5}" />
+    <xacro:insert_block name="rear_wing_inertia" />
+  </xacro:rear_wing>
+  <xacro:rear_wing
+    robot_namespace="${namespace}"
+    suffix="right"
+    parent="${namespace}/tail"
+    mass_rear_wing="${mass_rear_wing}"
+    rear_wing_length="${rear_wing_length}"
+    rear_wing_width="${tail_length}"
+    rear_wing_height="${rear_wing_height}"
+    use_mesh="false"
+    mesh="">
+    <origin xyz="0.0 ${-0.25 * (rear_wingspan + tail_width)} ${0.5 * (tail_height - rear_wing_height)}" rpy="0.0 0.0 ${-PI*0.5}" />
+    <xacro:insert_block name="rear_wing_inertia" />
+  </xacro:rear_wing>
 </robot>

File: rotors_description/urdf/fixed_wing_base.xacro (robot description, xacro)
@@ -116,3 +116,71 @@
     </gazebo>
   </xacro:macro>
+  <!-- Tail joint and link -->
+  <xacro:macro name="tail"
+    params="robot_namespace parent mass_tail tail_length tail_width tail_height
+      use_mesh mesh *origin *inertia">
+    <joint name="${robot_namespace}/tail_joint" type="revolute">
+      <xacro:insert_block name="origin" />
+      <axis xyz="0 0 1" />
+      <parent link="${parent}" />
+      <child link="${robot_namespace}/tail" />
+      <limit upper="0" lower="0" effort="0" velocity="0" />
+    </joint>
+    <link name="${robot_namespace}/tail">
+      <inertial>
+        <mass value="${mass_tail}" /> <!-- [kg] -->
+        <xacro:insert_block name="inertia" />
+      </inertial>
+      <visual>
+        <geometry>
+          <xacro:if value="${use_mesh}">
+            <mesh filename="${mesh}"
+              scale="1 1 1" />
+          </xacro:if>
+          <xacro:unless value="${use_mesh}">
+            <box size="${tail_length} ${tail_width} ${tail_height}"/> <!-- [m] [m] [m] -->
+          </xacro:unless>
+        </geometry>
+      </visual>
+      <collision>
+        <geometry>
+          <box size="${tail_length} ${tail_width} ${tail_height}"/> <!-- [m] [m] [m] -->
+        </geometry>
+      </collision>
+    </link>
+  </xacro:macro>
+  <!-- Rear wing joint and link -->
+  <xacro:macro name="rear_wing"
+    params="robot_namespace suffix parent mass_rear_wing rear_wing_length rear_wing_width
+      rear_wing_height use_mesh mesh *origin *inertia">
+    <joint name="${robot_namespace}/rear_wing_${suffix}_joint" type="revolute">
+      <xacro:insert_block name="origin" />
+      <axis xyz="0 0 1" />
+      <parent link="${parent}" />
+      <child link="${robot_namespace}/rear_wing_${suffix}" />
+      <limit upper="0" lower="0" effort="0" velocity="0" />
+    </joint>
+    <link name="${robot_namespace}/rear_wing_${suffix}">
+      <inertial>
+        <mass value="${mass_rear_wing}" /> <!-- [kg] -->
+        <xacro:insert_block name="inertia" />
+      </inertial>
+      <visual>
+        <geometry>
+          <xacro:if value="${use_mesh}">
+            <mesh filename="${mesh}"
+              scale="1 1 1" />
+          </xacro:if>
+          <xacro:unless value="${use_mesh}">
+            <box size="${rear_wing_length} ${rear_wing_width} ${rear_wing_height}"/> <!-- [m] [m] [m] -->
+          </xacro:unless>
+        </geometry>
+      </visual>
+      <collision>
+        <geometry>
+          <box size="${rear_wing_length} ${rear_wing_width} ${rear_wing_height}"/> <!-- [m] [m] [m] -->
+        </geometry>
+      </collision>
+    </link>
+  </xacro:macro>
 </robot>

Commit message: Adding a GUI for HIL interface, fixing several bugs in sensor plugins, extending mavlink_interface functionality

File: rotors_description/urdf/atlantik_solar.xacro (robot description, xacro)
@@ -22,11 +22,11 @@
   <xacro:property name="use_mesh_file" value="false" />
   <xacro:property name="mesh_file" value="" />
-  <xacro:property name="mass_fuselage" value="1.0" /> <!-- [kg] -->
-  <xacro:property name="mass_front_wing" value="1.0" /> <!-- [kg] -->
-  <xacro:property name="mass_tail" value="1.0" /> <!-- [kg] -->
-  <xacro:property name="mass_rear_wing" value="1.0" /> <!-- [kg] -->
+  <xacro:property name="mass_fuselage" value="0.2" /> <!-- [kg] -->
+  <xacro:property name="mass_front_wing" value="0.1" /> <!-- [kg] -->
+  <xacro:property name="mass_tail" value="0.1" /> <!-- [kg] -->
+  <xacro:property name="mass_rear_wing" value="0.1" /> <!-- [kg] -->
   <xacro:property name="body_length" value="3.0" /> <!-- [m] -->
-  <xacro:property name="body_width" value="0.3" /> <!-- [m] -->
-  <xacro:property name="body_height" value="0.16" /> <!-- [m] -->
+  <xacro:property name="body_width" value="0.1" /> <!-- [m] -->
+  <xacro:property name="body_height" value="0.1" /> <!-- [m] -->
   <xacro:property name="wingspan" value="6.0" /> <!-- [m] -->
   <xacro:property name="root_chord" value="0.3" /> <!-- [m] -->
@@ -38,5 +38,5 @@
   <xacro:property name="rear_wingspan" value="1.0" /> <!-- [m] -->
   <xacro:property name="rear_wing_height" value="0.02" /> <!-- [m] -->
-  <xacro:property name="alpha_0" value="0.0" /> <!-- [deg] -->
+  <xacro:property name="alpha_0" value="2.0" /> <!-- [deg] -->
   <xacro:property name="alpha_stall" value="15.0" /> <!-- [deg] -->
   <xacro:property name="c_L_alpha" value="${2.0 * PI}" />
@@ -91,8 +91,11 @@
     alpha_stall="${alpha_stall}"
     c_L_alpha="${c_L_alpha}"
-    air_density="${air_density}">
-    <origin xyz="0.5 ${0.25 * (wingspan + body_width)} ${0.5*body_height}" rpy="0.0 ${front_wing_dihedral_angle*PI/180.0} ${-PI*0.5}" />
+    air_density="${air_density}"
+    link_x="${0.5*front_wing_length}"
+    link_y="0.0"
+    link_z="0.0">
+    <origin xyz="0.5 ${0.5*body_width} 0.0" rpy="0.0 ${-front_wing_dihedral_angle*PI/180.0} ${PI*0.5}" />
     <xacro:insert_block name="front_wing_inertia" />
-  </xacro:wing>
+  </xacro:wing>-->
   <xacro:wing
     robot_namespace="${namespace}"
@@ -108,6 +111,9 @@
     alpha_stall="${alpha_stall}"
     c_L_alpha="${c_L_alpha}"
-    air_density="${air_density}">
-    <origin xyz="0.5 ${-0.25 * (wingspan + body_width)} ${0.5*body_height}" rpy="0.0 ${front_wing_dihedral_angle*PI/180.0} ${PI*0.5}" />
+    air_density="${air_density}"
+    link_x="${0.5*front_wing_length}"
+    link_y="0.0"
+    link_z="0.0">
+    <origin xyz="0.5 ${-0.5*body_width} 0.0" rpy="0.0 ${-front_wing_dihedral_angle*PI/180.0} ${-PI*0.5}" />
     <xacro:insert_block name="front_wing_inertia" />
   </xacro:wing>

File: rotors_description/urdf/fixed_wing_base.xacro (robot description, xacro)
@@ -74,8 +74,8 @@
   <xacro:macro name="wing"
     params="robot_namespace suffix parent mass_wing wing_length wing_width wing_height
-      use_mesh mesh alpha_0 alpha_stall c_L_alpha air_density *origin *inertia">
+      use_mesh mesh alpha_0 alpha_stall c_L_alpha air_density link_x link_y link_z *origin *inertia">
     <joint name="${robot_namespace}/wing_${suffix}_joint" type="revolute">
       <xacro:insert_block name="origin" />
-      <axis xyz="0 0 1" />
+      <axis xyz="1 0 0" />
       <parent link="${parent}" />
       <child link="${robot_namespace}/wing_${suffix}" />
@@ -84,8 +84,10 @@
     <link name="${robot_namespace}/wing_${suffix}">
       <inertial>
+        <origin xyz="${link_x} ${link_y} ${link_z}" rpy="0 0 0" />
         <mass value="${mass_wing}" /> <!-- [kg] -->
         <xacro:insert_block name="inertia" />
       </inertial>
       <visual>
+        <origin xyz="${link_x} ${link_y} ${link_z}" rpy="0 0 0" />
         <geometry>
           <xacro:if value="${use_mesh}">
@@ -99,4 +101,5 @@
       </visual>
       <collision>
+        <origin xyz="${link_x} ${link_y} ${link_z}" rpy="0 0 0" />
         <geometry>
           <box size="${wing_length} ${wing_width} ${wing_height}"/> <!-- [m] [m] [m] -->
@@ -104,13 +107,32 @@
       </collision>
     </link>
+<!--
     <gazebo>
       <plugin name="${robot_namespace}_${suffix}_wing_model" filename="librotors_gazebo_wing_model.so">
         <robotNamespace>${robot_namespace}</robotNamespace>
         <linkName>${robot_namespace}/wing_${suffix}</linkName>
-        <alpha0>${alpha_0}</alpha0> <!-- the starting angle of attack [deg] -->
-        <alphaStall>${alpha_stall}</alphaStall> <!-- stall angle [deg] -->
-        <cLAlpha>${c_L_alpha}</cLAlpha> <!-- coefficient of lift to angle of attack ratio -->
-        <airDensity>${air_density}</airDensity> <!-- air density [kg/m^3] -->
-        <wingArea>${wing_length * wing_width}</wingArea> <!-- area of the wing [m^2] -->
+        <alpha0>${alpha_0}</alpha0> --> <!-- the starting angle of attack [deg] -->
+        <!--<alphaStall>${alpha_stall}</alphaStall> --> <!-- stall angle [deg] -->
+        <!--<cLAlpha>${c_L_alpha}</cLAlpha> --> <!-- coefficient of lift to angle of attack ratio -->
+        <!--<airDensity>${air_density}</airDensity> --> <!-- air density [kg/m^3] -->
+        <!--<wingArea>${wing_length * wing_width}</wingArea> --> <!-- area of the wing [m^2] -->
+<!--      </plugin>
+    </gazebo> -->
+    <gazebo>
+      <plugin name="${robot_namespace}_${suffix}_lift_drag" filename="libLiftDragPlugin.so">
+        <a0>0.1</a0>
+        <cla>4.0</cla>
+        <cda>0.001</cda>
+        <cma>0.00</cma>
+        <alpha_stall>10.0</alpha_stall>
+        <cla_stall>0.0</cla_stall>
+        <cda_stall>0.01</cda_stall>
+        <cma_stall>0.0</cma_stall>
+        <cp>0.0 0.5 0.0</cp>
+        <area>${wing_length * wing_width}</area>
+        <air_density>${air_density}</air_density>
+        <forward>1 0 0</forward>
+        <upward>0 0 1</upward>
+        <link_name>${robot_namespace}/wing_${suffix}</link_name>
       </plugin>
     </gazebo>
@@ -183,4 +205,22 @@
       </collision>
     </link>
+    <gazebo>
+      <plugin name="${robot_namespace}_${suffix}_rear_lift_drag" filename="libLiftDragPlugin.so">
+        <a0>0.1</a0>
+        <cla>4.0</cla>
+        <cda>0.001</cda>
+        <cma>0.00</cma>
+        <alpha_stall>10.0</alpha_stall>
+        <cla_stall>0.0</cla_stall>
+        <cda_stall>0.01</cda_stall>
+        <cma_stall>0.0</cma_stall>
+        <cp>0.0 0.5 0.0</cp>
+        <area>${rear_wing_length * rear_wing_width}</area>
+        <air_density>1.225</air_density>
+        <forward>1 0 0</forward>
+        <upward>0 0 1</upward>
+        <link_name>${robot_namespace}/rear_wing_${suffix}</link_name>
+      </plugin>
+    </gazebo>
   </xacro:macro>
 </robot>
