Commit message: Adding max_thrust as a parameter to URDF

File: rotors_description/urdf/atlantik_solar.xacro (robot description, xacro)
@@ -38,4 +38,5 @@
   <xacro:property name="rear_wingspan" value="1.0" /> <!-- [m] -->
   <xacro:property name="rear_wing_height" value="0.02" /> <!-- [m] -->
+  <xacro:property name="max_thrust" value="100.0" /> <!-- [N] -->
   <xacro:property name="alpha_0" value="2.0" /> <!-- [deg] -->
   <xacro:property name="alpha_stall" value="15.0" /> <!-- [deg] -->
@@ -73,4 +74,6 @@
     body_width="${body_width}"
     body_height="${body_height}"
+    actuator_topic="actuators"
+    max_thrust="200.0"
     use_mesh_file="${use_mesh_file}"
     mesh_file="${mesh_file}">

File: rotors_description/urdf/fixed_wing_base.xacro (robot description, xacro)
@@ -33,5 +33,6 @@
   <!-- Fixed-wing fuselage link -->
   <xacro:macro name="fixed_wing_base_macro"
-    params="robot_namespace mass body_length body_width body_height use_mesh_file mesh_file *inertia">
+    params="robot_namespace mass body_length body_width body_height
+      actuator_topic max_thrust use_mesh_file mesh_file *inertia">
     <link name="${robot_namespace}/base_link"></link>
     <joint name="${robot_namespace}/base_joint" type="fixed">
@@ -68,4 +69,6 @@
         <robotNamespace>${robot_namespace}</robotNamespace>
         <linkName>${robot_namespace}/base_link</linkName>
+	<actuatorsTopic>${actuator_topic}</actuatorsTopic>
+        <maxThrust>${max_thrust}</maxThrust>
       </plugin>
     </gazebo>

Commit message: Replacing mavlink_interface with hil_interface

File: rotors_description/urdf/atlantik_solar.xacro (robot description, xacro)
@@ -22,8 +22,8 @@
   <xacro:property name="use_mesh_file" value="false" />
   <xacro:property name="mesh_file" value="" />
-  <xacro:property name="mass_fuselage" value="0.2" /> <!-- [kg] -->
-  <xacro:property name="mass_front_wing" value="0.1" /> <!-- [kg] -->
-  <xacro:property name="mass_tail" value="0.1" /> <!-- [kg] -->
-  <xacro:property name="mass_rear_wing" value="0.1" /> <!-- [kg] -->
+  <xacro:property name="mass_fuselage" value="5.0" /> <!-- [kg] -->
+  <xacro:property name="mass_front_wing" value="1.0" /> <!-- [kg] -->
+  <xacro:property name="mass_tail" value="1.0" /> <!-- [kg] -->
+  <xacro:property name="mass_rear_wing" value="0.5" /> <!-- [kg] -->
   <xacro:property name="body_length" value="3.0" /> <!-- [m] -->
   <xacro:property name="body_width" value="0.1" /> <!-- [m] -->
@@ -38,5 +38,5 @@
   <xacro:property name="rear_wingspan" value="1.0" /> <!-- [m] -->
   <xacro:property name="rear_wing_height" value="0.02" /> <!-- [m] -->
-  <xacro:property name="max_thrust" value="100.0" /> <!-- [N] -->
+  <xacro:property name="max_thrust" value="300.0" /> <!-- [N] -->
   <xacro:property name="alpha_0" value="2.0" /> <!-- [deg] -->
   <xacro:property name="alpha_stall" value="15.0" /> <!-- [deg] -->
@@ -75,5 +75,5 @@
     body_height="${body_height}"
     actuator_topic="actuators"
-    max_thrust="200.0"
+    max_thrust="${max_thrust}"
     use_mesh_file="${use_mesh_file}"
     mesh_file="${mesh_file}">
@@ -86,6 +86,6 @@
     parent="${namespace}/base_link"
     mass_wing="${mass_front_wing}"
-    wing_length="${front_wing_length}"
-    wing_width="${root_chord}"
+    wing_length="${root_chord}"
+    wing_width="${front_wing_length}"
     wing_height="${front_wing_height}"
     use_mesh="false"
@@ -95,10 +95,14 @@
     c_L_alpha="${c_L_alpha}"
     air_density="${air_density}"
-    link_x="${0.5*front_wing_length}"
+    link_x="0.0"
     link_y="0.0"
     link_z="0.0">
-    <origin xyz="0.5 ${0.5*body_width} 0.0" rpy="0.0 ${-front_wing_dihedral_angle*PI/180.0} ${PI*0.5}" />
+    <origin xyz="0.1 1.5 0.0" rpy="0.0 0.0 0.0" />
     <xacro:insert_block name="front_wing_inertia" />
   </xacro:wing>-->
+<!--wing_length="${front_wing_length}"
+    wing_width="${root_chord}"
+    link_x="${0.5*front_wing_length}"
+    <origin xyz="0.5 ${0.5*body_width} 0.0" rpy="0.0 ${-front_wing_dihedral_angle*PI/180.0} ${PI*0.5}" /> -->
   <xacro:wing
     robot_namespace="${namespace}"
@@ -106,6 +110,6 @@
     parent="${namespace}/base_link"
     mass_wing="${mass_front_wing}"
-    wing_length="${front_wing_length}"
-    wing_width="${root_chord}"
+    wing_length="${root_chord}"
+    wing_width="${front_wing_length}"
     wing_height="${front_wing_height}"
     use_mesh="false"
@@ -115,10 +119,11 @@
     c_L_alpha="${c_L_alpha}"
     air_density="${air_density}"
-    link_x="${0.5*front_wing_length}"
+    link_x="0.0"
     link_y="0.0"
     link_z="0.0">
-    <origin xyz="0.5 ${-0.5*body_width} 0.0" rpy="0.0 ${-front_wing_dihedral_angle*PI/180.0} ${-PI*0.5}" />
+    <origin xyz="0.1 -1.5 0.0" rpy="0.0 0.0 0.0" />
     <xacro:insert_block name="front_wing_inertia" />
   </xacro:wing>
+<!-- <origin xyz="0.5 ${-0.5*body_width} 0.0" rpy="0.0 ${-front_wing_dihedral_angle*PI/180.0} ${-PI*0.5}" /> -->
   <!-- Instantiate the tail -->
   <xacro:tail
@@ -140,12 +145,15 @@
     parent="${namespace}/tail"
     mass_rear_wing="${mass_rear_wing}"
-    rear_wing_length="${rear_wing_length}"
-    rear_wing_width="${tail_length}"
+    rear_wing_length="${tail_length}"
+    rear_wing_width="${rear_wing_length}"
     rear_wing_height="${rear_wing_height}"
     use_mesh="false"
     mesh="">
-    <origin xyz="0.0 ${0.25 * (rear_wingspan + tail_width)} ${0.5 * (tail_height - rear_wing_height)}" rpy="0.0 0.0 ${PI*0.5}" />
+    <origin xyz="0.0 ${0.25 * (rear_wingspan + tail_width)} ${0.5 * (tail_height - rear_wing_height)}" rpy="0.0 0.0 0.0" />
     <xacro:insert_block name="rear_wing_inertia" />
   </xacro:rear_wing>
+<!--rear_wing_length="${rear_wing_length}"
+    rear_wing_width="${tail_length}"
+    <origin xyz="0.0 ${0.25 * (rear_wingspan + tail_width)} ${0.5 * (tail_height - rear_wing_height)}" rpy="0.0 0.0 ${PI*0.5}" /> -->
   <xacro:rear_wing
     robot_namespace="${namespace}"
@@ -153,11 +161,12 @@
     parent="${namespace}/tail"
     mass_rear_wing="${mass_rear_wing}"
-    rear_wing_length="${rear_wing_length}"
-    rear_wing_width="${tail_length}"
+    rear_wing_length="${tail_length}"
+    rear_wing_width="${rear_wing_length}"
     rear_wing_height="${rear_wing_height}"
     use_mesh="false"
     mesh="">
-    <origin xyz="0.0 ${-0.25 * (rear_wingspan + tail_width)} ${0.5 * (tail_height - rear_wing_height)}" rpy="0.0 0.0 ${-PI*0.5}" />
+    <origin xyz="0.0 ${-0.25 * (rear_wingspan + tail_width)} ${0.5 * (tail_height - rear_wing_height)}" rpy="0.0 0.0 0.0" />
     <xacro:insert_block name="rear_wing_inertia" />
   </xacro:rear_wing>
+<!--<origin xyz="0.0 ${-0.25 * (rear_wingspan + tail_width)} ${0.5 * (tail_height - rear_wing_height)}" rpy="0.0 0.0 ${-PI*0.5}" /> -->
 </robot>

File: rotors_description/urdf/fixed_wing_base.xacro (robot description, xacro)
@@ -126,11 +126,11 @@
         <a0>0.1</a0>
         <cla>4.0</cla>
-        <cda>0.001</cda>
+        <cda>0.01</cda>
         <cma>0.00</cma>
-        <alpha_stall>10.0</alpha_stall>
+        <alpha_stall>0.3</alpha_stall>
         <cla_stall>0.0</cla_stall>
         <cda_stall>0.01</cda_stall>
         <cma_stall>0.0</cma_stall>
-        <cp>0.0 0.5 0.0</cp>
+        <cp>0.0 0.0 0.0</cp>
         <area>${wing_length * wing_width}</area>
         <air_density>${air_density}</air_density>
@@ -210,13 +210,13 @@
     <gazebo>
       <plugin name="${robot_namespace}_${suffix}_rear_lift_drag" filename="libLiftDragPlugin.so">
-        <a0>0.1</a0>
+        <a0>0.03</a0>
         <cla>4.0</cla>
-        <cda>0.001</cda>
+        <cda>0.01</cda>
         <cma>0.00</cma>
-        <alpha_stall>10.0</alpha_stall>
+        <alpha_stall>0.3</alpha_stall>
         <cla_stall>0.0</cla_stall>
         <cda_stall>0.01</cda_stall>
         <cma_stall>0.0</cma_stall>
-        <cp>0.0 0.5 0.0</cp>
+        <cp>0.0 0.0 0.0</cp>
         <area>${rear_wing_length * rear_wing_width}</area>
         <air_density>1.225</air_density>
