Commit message: Adding wheels and better parameters to the fixed wing model

File: rotors_description/urdf/atlantik_solar.xacro (robot description, xacro)
@@ -19,15 +19,20 @@
   <!-- Properties -->
   <xacro:property name="namespace" value="$(arg mav_name)" />
-  <xacro:property name="rotor_velocity_slowdown_sim" value="10" />
+  <xacro:property name="propeller_velocity_slowdown_sim" value="10" />
   <xacro:property name="use_mesh_file" value="false" />
   <xacro:property name="mesh_file" value="" />
-  <xacro:property name="mass_fuselage" value="5.0" /> <!-- [kg] -->
+  <xacro:property name="mass_fuselage" value="3.0" /> <!-- [kg] -->
+  <xacro:property name="mass_wheel" value="0.1" /> <!-- [kg] -->
   <xacro:property name="mass_front_wing" value="1.0" /> <!-- [kg] -->
-  <xacro:property name="mass_tail" value="1.0" /> <!-- [kg] -->
-  <xacro:property name="mass_rear_wing" value="0.5" /> <!-- [kg] -->
+  <xacro:property name="mass_tail" value="0.5" /> <!-- [kg] -->
+  <xacro:property name="mass_rear_wing" value="0.2" /> <!-- [kg] -->
+  <xacro:property name="mass_propeller" value="0.005" /> <!-- [kg] -->
   <xacro:property name="body_length" value="3.0" /> <!-- [m] -->
   <xacro:property name="body_width" value="0.1" /> <!-- [m] -->
   <xacro:property name="body_height" value="0.1" /> <!-- [m] -->
-  <xacro:property name="wingspan" value="6.0" /> <!-- [m] -->
+  <xacro:property name="body_color" value="Red" />
+  <xacro:property name="wheel_radius" value="0.05" /> <!-- [m] -->
+  <xacro:property name="wheel_width" value="0.01" /> <!-- [m] -->
+  <xacro:property name="wingspan" value="4.0" /> <!-- [m] -->
   <xacro:property name="root_chord" value="0.3" /> <!-- [m] -->
   <xacro:property name="front_wing_height" value="0.02" /> <!-- [m] -->
@@ -38,9 +43,19 @@
   <xacro:property name="rear_wingspan" value="1.0" /> <!-- [m] -->
   <xacro:property name="rear_wing_height" value="0.02" /> <!-- [m] -->
-  <xacro:property name="max_thrust" value="300.0" /> <!-- [N] -->
+  <xacro:property name="max_thrust" value="200.0" /> <!-- [N] -->
   <xacro:property name="alpha_0" value="2.0" /> <!-- [deg] -->
   <xacro:property name="alpha_stall" value="15.0" /> <!-- [deg] -->
   <xacro:property name="c_L_alpha" value="${2.0 * PI}" />
   <xacro:property name="air_density" value="1.225" /> <!-- [kg/m^3] -->
+  <xacro:property name="radius_propeller" value="0.15" /> <!-- [m] -->
+  <xacro:property name="propeller_offset" value="0.025" /> <!-- [m] -->
+  <xacro:property name="motor_constant" value="6.14858e-04" /> <!-- [kg m/s^2] -->
+  <!--<xacro:property name="motor_constant" value="8.54858e-06" />--> <!-- [kg m/s^2] -->
+  <xacro:property name="moment_constant" value="0.016" /> <!-- [m] -->
+  <xacro:property name="time_constant_up" value="0.0125" /> <!-- [s] -->
+  <xacro:property name="time_constant_down" value="0.025" /> <!-- [s] -->
+  <xacro:property name="max_propeller_velocity" value="838" /> <!-- [rad/s] -->
+  <xacro:property name="rotor_drag_coefficient" value="8.06428e-05" />
+  <xacro:property name="rolling_moment_coefficient" value="0.000001" />
   <xacro:property name="PI" value="3.1415926535897931" />
   <!-- Front wing length -->
@@ -53,4 +68,8 @@
     <xacro:box_inertia x="${body_length}" y="${body_width}" z="${body_height}" mass="${mass_fuselage}" />
   </xacro:property>
+  <!-- Inertia of a single wheel, assuming it is a cylinder -->
+  <xacro:property name="wheel_inertia">
+    <xacro:cylinder_inertia r="${wheel_radius}" h="${wheel_width}" mass="${mass_wheel}" />
+  </xacro:property>
   <!-- Inertia of a single front wing, assuming it is a cuboid -->
   <xacro:property name="front_wing_inertia">
@@ -64,4 +83,8 @@
   <xacro:property name="rear_wing_inertia">
     <xacro:box_inertia x="${rear_wing_length}" y="${tail_width}" z="${tail_height}" mass="${mass_rear_wing}" />
+  </xacro:property>
+  <!-- Inertia of the propeller, assuming it is a cuboid. Height=3mm, width=40mm -->
+  <xacro:property name="propeller_inertia">
+    <xacro:box_inertia x="${radius_propeller}" y="0.04" z="0.003" mass="${mass_propeller * propeller_velocity_slowdown_sim}" />
   </xacro:property>
   <!-- Included URDF Files -->
@@ -76,8 +99,49 @@
     actuator_topic="actuators"
     max_thrust="${max_thrust}"
+    color="${body_color}"
     use_mesh_file="${use_mesh_file}"
     mesh_file="${mesh_file}">
     <xacro:insert_block name="body_inertia" />
   </xacro:fixed_wing_base_macro>
+  <!-- Instantiate wheels -->
+  <xacro:wheel
+    robot_namespace="${namespace}"
+    suffix="front_left"
+    parent="${namespace}/base_link"
+    mass_wheel="${mass_wheel}"
+    color="${body_color}"
+    use_mesh="false"
+    mesh=""
+    wheel_radius="${wheel_radius}"
+    wheel_width="${wheel_width}">
+    <origin xyz="0.75 0.1 0.0" rpy="${0.5 * PI} 0.0 0.0" />
+    <xacro:insert_block name="wheel_inertia" />
+  </xacro:wheel>
+  <xacro:wheel
+    robot_namespace="${namespace}"
+    suffix="front_right"
+    parent="${namespace}/base_link"
+    mass_wheel="${mass_wheel}"
+    color="${body_color}"
+    use_mesh="false"
+    mesh=""
+    wheel_radius="${wheel_radius}"
+    wheel_width="${wheel_width}">
+    <origin xyz="0.75 -0.1 0.0" rpy="${0.5 * PI} 0.0 0.0" />
+    <xacro:insert_block name="wheel_inertia" />
+  </xacro:wheel>
+  <xacro:wheel
+    robot_namespace="${namespace}"
+    suffix="back"
+    parent="${namespace}/base_link"
+    mass_wheel="${mass_wheel}"
+    color="${body_color}"
+    use_mesh="false"
+    mesh=""
+    wheel_radius="${wheel_radius}"
+    wheel_width="${wheel_width}">
+    <origin xyz="-1.0 0.0 0.0" rpy="${0.5 * PI} 0.0 0.0" />
+    <xacro:insert_block name="wheel_inertia" />
+  </xacro:wheel>
   <!-- Instantiate wings -->
   <xacro:wing
@@ -89,4 +153,5 @@
     wing_width="${front_wing_length}"
     wing_height="${front_wing_height}"
+    color="${body_color}"
     use_mesh="false"
     mesh=""
@@ -94,15 +159,8 @@
     alpha_stall="${alpha_stall}"
     c_L_alpha="${c_L_alpha}"
-    air_density="${air_density}"
-    link_x="0.0"
-    link_y="0.0"
-    link_z="0.0">
-    <origin xyz="0.1 1.5 0.0" rpy="0.0 0.0 0.0" />
+    air_density="${air_density}">
+    <origin xyz="0.5 ${0.25 * wingspan} 0.1" rpy="0.0 0.0 0.0" />
     <xacro:insert_block name="front_wing_inertia" />
   </xacro:wing>-->
-<!--wing_length="${front_wing_length}"
-    wing_width="${root_chord}"
-    link_x="${0.5*front_wing_length}"
-    <origin xyz="0.5 ${0.5*body_width} 0.0" rpy="0.0 ${-front_wing_dihedral_angle*PI/180.0} ${PI*0.5}" /> -->
   <xacro:wing
     robot_namespace="${namespace}"
@@ -113,4 +171,5 @@
     wing_width="${front_wing_length}"
     wing_height="${front_wing_height}"
+    color="${body_color}"
     use_mesh="false"
     mesh=""
@@ -118,12 +177,8 @@
     alpha_stall="${alpha_stall}"
     c_L_alpha="${c_L_alpha}"
-    air_density="${air_density}"
-    link_x="0.0"
-    link_y="0.0"
-    link_z="0.0">
-    <origin xyz="0.1 -1.5 0.0" rpy="0.0 0.0 0.0" />
+    air_density="${air_density}">
+    <origin xyz="0.5 -${0.25 * wingspan} 0.1" rpy="0.0 0.0 0.0" />
     <xacro:insert_block name="front_wing_inertia" />
   </xacro:wing>
-<!-- <origin xyz="0.5 ${-0.5*body_width} 0.0" rpy="0.0 ${-front_wing_dihedral_angle*PI/180.0} ${-PI*0.5}" /> -->
   <!-- Instantiate the tail -->
   <xacro:tail
@@ -134,7 +189,8 @@
     tail_width="${tail_width}"
     tail_height="${tail_height}"
-    use_mesh="false"
-    mesh="">
-    <origin xyz="${-0.5*body_length + 0.5*tail_length} 0.0 ${0.5*body_height + 0.5*tail_height}" rpy="0.0 0.0 0.0" />
+    color="${body_color}"
+    use_mesh="false"
+    mesh="">
+    <origin xyz="${-0.5*body_length + 0.5*tail_length} 0.0 ${0.5*body_height + 0.5*tail_height + 0.1}" rpy="0.0 0.0 0.0" />
     <xacro:insert_block name="tail_inertia" />
   </xacro:tail>
@@ -148,4 +204,5 @@
     rear_wing_width="${rear_wing_length}"
     rear_wing_height="${rear_wing_height}"
+    color="${body_color}"
     use_mesh="false"
     mesh="">
@@ -153,7 +210,4 @@
     <xacro:insert_block name="rear_wing_inertia" />
   </xacro:rear_wing>
-<!--rear_wing_length="${rear_wing_length}"
-    rear_wing_width="${tail_length}"
-    <origin xyz="0.0 ${0.25 * (rear_wingspan + tail_width)} ${0.5 * (tail_height - rear_wing_height)}" rpy="0.0 0.0 ${PI*0.5}" /> -->
   <xacro:rear_wing
     robot_namespace="${namespace}"
@@ -164,4 +218,5 @@
     rear_wing_width="${rear_wing_length}"
     rear_wing_height="${rear_wing_height}"
+    color="${body_color}"
     use_mesh="false"
     mesh="">
@@ -169,4 +224,24 @@
     <xacro:insert_block name="rear_wing_inertia" />
   </xacro:rear_wing>
-<!--<origin xyz="0.0 ${-0.25 * (rear_wingspan + tail_width)} ${0.5 * (tail_height - rear_wing_height)}" rpy="0.0 0.0 ${-PI*0.5}" /> -->
+  <!-- Instantiate the propeller -->
+  <xacro:propeller
+    robot_namespace="${namespace}"
+    direction="cw"
+    motor_constant="${motor_constant}"
+    moment_constant="${moment_constant}"
+    parent="${namespace}/base_link"
+    mass_propeller="${mass_propeller}"
+    radius_propeller="${radius_propeller}"
+    time_constant_up="${time_constant_up}"
+    time_constant_down="${time_constant_down}"
+    max_propeller_velocity="${max_propeller_velocity}"
+    motor_number="0"
+    rotor_drag_coefficient="${rotor_drag_coefficient}"
+    rolling_moment_coefficient="${rolling_moment_coefficient}"
+    color="Blue"
+    use_own_mesh="false"
+    mesh="">
+    <origin xyz="${0.5 * body_length + propeller_offset} 0.0 0.1" rpy="0.0 ${0.5 * PI} 0.0" />
+    <xacro:insert_block name="propeller_inertia" />
+  </xacro:propeller>
 </robot>

File: rotors_description/urdf/fixed_wing_base.xacro (robot description, xacro)
@@ -23,4 +23,10 @@
       izz="${0.0833333 * mass * (x*x + y*y)}" />
   </xacro:macro>
+  <!-- Macro for the inertia of a cylinder -->
+  <xacro:macro name="cylinder_inertia" params="r h mass">
+    <inertia ixx="${0.0833333 * mass * (3*r*r + h*h)}" ixy="0.0" ixz="0.0"
+      iyy="${0.0833333 * mass * (3*r*r + h*h)}" iyz="0.0"
+      izz="${0.5 * mass * r * r}" />
+  </xacro:macro>
   <!-- Macro for the inertial properties of a box -->
   <xacro:macro name="box_inertial" params="x y z mass *origin">
@@ -34,8 +40,8 @@
   <xacro:macro name="fixed_wing_base_macro"
     params="robot_namespace mass body_length body_width body_height
-      actuator_topic max_thrust use_mesh_file mesh_file *inertia">
+      actuator_topic max_thrust color use_mesh_file mesh_file *inertia">
     <link name="${robot_namespace}/base_link"></link>
     <joint name="${robot_namespace}/base_joint" type="fixed">
-      <origin xyz="0 0 0" rpy="0 0 0" />
+      <origin xyz="0 0 0.1" rpy="0 0 0" />
       <parent link="${robot_namespace}/base_link" />
       <child link="${robot_namespace}/base_link_inertia" />
@@ -73,9 +79,48 @@
       </plugin>
     </gazebo>
+    <gazebo reference="${robot_namespace}/base_link">
+      <material>Gazebo/${color}</material>
+    </gazebo>
+  </xacro:macro>
+  <!-- Wheel joint and link -->
+  <xacro:macro name="wheel"
+    params="robot_namespace suffix parent mass_wheel color use_mesh mesh wheel_radius wheel_width *origin *inertia">
+    <joint name="${robot_namespace}/wheel_${suffix}_joint" type="revolute">
+      <xacro:insert_block name="origin" />
+      <axis xyz="0 1 0" />
+      <parent link="${parent}" />
+      <child link="${robot_namespace}/wheel_${suffix}" />
+      <limit upper="0" lower="0" effort="0" velocity="0" />
+    </joint>
+    <link name="${robot_namespace}/wheel_${suffix}">
+      <inertial>
+        <mass value="${mass_wheel}" /> <!-- [kg] -->
+        <xacro:insert_block name="inertia" />
+      </inertial>
+      <visual>
+        <geometry>
+          <xacro:if value="${use_mesh}">
+            <mesh filename="${mesh}"
+              scale="1 1 1" />
+          </xacro:if>
+          <xacro:unless value="${use_mesh}">
+            <cylinder length="${wheel_width}" radius="${wheel_radius}" /> <!-- [m] -->
+          </xacro:unless>
+        </geometry>
+      </visual>
+      <collision>
+        <geometry>
+          <cylinder length="${wheel_width}" radius="${wheel_radius}" /> <!-- [m] -->
+        </geometry>
+      </collision>
+    </link>
+    <gazebo reference="${robot_namespace}/wheel_${suffix}">
+      <material>Gazebo/${color}</material>
+    </gazebo>
   </xacro:macro>
   <!-- Wing joint and link -->
   <xacro:macro name="wing"
     params="robot_namespace suffix parent mass_wing wing_length wing_width wing_height
-      use_mesh mesh alpha_0 alpha_stall c_L_alpha air_density link_x link_y link_z *origin *inertia">
+      color use_mesh mesh alpha_0 alpha_stall c_L_alpha air_density *origin *inertia">
     <joint name="${robot_namespace}/wing_${suffix}_joint" type="revolute">
       <xacro:insert_block name="origin" />
@@ -87,10 +132,10 @@
     <link name="${robot_namespace}/wing_${suffix}">
       <inertial>
-        <origin xyz="${link_x} ${link_y} ${link_z}" rpy="0 0 0" />
+        <origin xyz="0 0 0" rpy="0 0 0" />
         <mass value="${mass_wing}" /> <!-- [kg] -->
         <xacro:insert_block name="inertia" />
       </inertial>
       <visual>
-        <origin xyz="${link_x} ${link_y} ${link_z}" rpy="0 0 0" />
+        <origin xyz="0 0 0" rpy="0 0 0" />
         <geometry>
           <xacro:if value="${use_mesh}">
@@ -104,5 +149,5 @@
       </visual>
       <collision>
-        <origin xyz="${link_x} ${link_y} ${link_z}" rpy="0 0 0" />
+        <origin xyz="0 0 0" rpy="0 0 0" />
         <geometry>
           <box size="${wing_length} ${wing_width} ${wing_height}"/> <!-- [m] [m] [m] -->
@@ -110,23 +155,12 @@
       </collision>
     </link>
-<!--
-    <gazebo>
-      <plugin name="${robot_namespace}_${suffix}_wing_model" filename="librotors_gazebo_wing_model.so">
-        <robotNamespace>${robot_namespace}</robotNamespace>
-        <linkName>${robot_namespace}/wing_${suffix}</linkName>
-        <alpha0>${alpha_0}</alpha0> --> <!-- the starting angle of attack [deg] -->
-        <!--<alphaStall>${alpha_stall}</alphaStall> --> <!-- stall angle [deg] -->
-        <!--<cLAlpha>${c_L_alpha}</cLAlpha> --> <!-- coefficient of lift to angle of attack ratio -->
-        <!--<airDensity>${air_density}</airDensity> --> <!-- air density [kg/m^3] -->
-        <!--<wingArea>${wing_length * wing_width}</wingArea> --> <!-- area of the wing [m^2] -->
-<!--      </plugin>
-    </gazebo> -->
     <gazebo>
       <plugin name="${robot_namespace}_${suffix}_lift_drag" filename="libLiftDragPlugin.so">
-        <a0>0.1</a0>
+      <!--<plugin name="${robot_namespace}_${suffix}_lift_drag" filename="librotors_gazebo_lift_drag_plugin.so">-->
+        <a0>0.01</a0>
         <cla>4.0</cla>
         <cda>0.01</cda>
         <cma>0.00</cma>
-        <alpha_stall>0.3</alpha_stall>
+        <alpha_stall>0.09</alpha_stall>
         <cla_stall>0.0</cla_stall>
         <cda_stall>0.01</cda_stall>
@@ -140,9 +174,12 @@
       </plugin>
     </gazebo>
+    <gazebo reference="${robot_namespace}/wing_${suffix}">
+      <material>Gazebo/${color}</material>
+    </gazebo>
   </xacro:macro>
   <!-- Tail joint and link -->
   <xacro:macro name="tail"
     params="robot_namespace parent mass_tail tail_length tail_width tail_height
-      use_mesh mesh *origin *inertia">
+      color use_mesh mesh *origin *inertia">
     <joint name="${robot_namespace}/tail_joint" type="revolute">
       <xacro:insert_block name="origin" />
@@ -174,9 +211,12 @@
       </collision>
     </link>
+    <gazebo reference="${robot_namespace}/tail">
+      <material>Gazebo/${color}</material>
+    </gazebo>
   </xacro:macro>
   <!-- Rear wing joint and link -->
   <xacro:macro name="rear_wing"
     params="robot_namespace suffix parent mass_rear_wing rear_wing_length rear_wing_width
-      rear_wing_height use_mesh mesh *origin *inertia">
+      rear_wing_height color use_mesh mesh *origin *inertia">
     <joint name="${robot_namespace}/rear_wing_${suffix}_joint" type="revolute">
       <xacro:insert_block name="origin" />
@@ -210,9 +250,10 @@
     <gazebo>
       <plugin name="${robot_namespace}_${suffix}_rear_lift_drag" filename="libLiftDragPlugin.so">
-        <a0>0.03</a0>
+      <!--<plugin name="${robot_namespace}_${suffix}_lift_drag" filename="librotors_gazebo_lift_drag_plugin.so">-->
+        <a0>0.01</a0>
         <cla>4.0</cla>
         <cda>0.01</cda>
         <cma>0.00</cma>
-        <alpha_stall>0.3</alpha_stall>
+        <alpha_stall>0.09</alpha_stall>
         <cla_stall>0.0</cla_stall>
         <cda_stall>0.01</cda_stall>
@@ -226,4 +267,64 @@
       </plugin>
     </gazebo>
+    <gazebo reference="${robot_namespace}/rear_wing_${suffix}">
+      <material>Gazebo/${color}</material>
+    </gazebo>
+  </xacro:macro>
+  <!-- Propeller joint and link -->
+  <xacro:macro name="propeller"
+    params="robot_namespace direction motor_constant moment_constant parent mass_propeller
+      radius_propeller time_constant_up time_constant_down max_propeller_velocity motor_number
+      rotor_drag_coefficient rolling_moment_coefficient use_own_mesh mesh color *origin *inertia">
+    <joint name="${robot_namespace}/propeller_joint" type="continuous">
+      <xacro:insert_block name="origin" />
+      <axis xyz="0 0 1" />
+      <parent link="${parent}" />
+      <child link="${robot_namespace}/propeller" />
+    </joint>
+    <link name="${robot_namespace}/propeller">
+      <inertial>
+        <mass value="${mass_propeller}" /> <!-- [kg] -->
+        <xacro:insert_block name="inertia" />
+      </inertial>
+      <visual>
+        <geometry>
+          <xacro:if value="${use_own_mesh}">
+            <mesh filename="${mesh}"
+              scale="1 1 1" />
+          </xacro:if>
+          <xacro:unless value="${use_own_mesh}">
+            <mesh filename="package://rotors_description/meshes/propeller_${direction}.dae"
+              scale="${radius_propeller} ${radius_propeller} ${radius_propeller}" /> <!-- The propeller meshes have a radius of 1m -->
+          </xacro:unless>
+        </geometry>
+      </visual>
+      <collision>
+        <geometry>
+          <cylinder length="0.005" radius="0.1" /> <!-- [m] -->
+        </geometry>
+      </collision>
+    </link>
+    <gazebo>
+      <plugin name="${robot_namespace}_propeller" filename="librotors_gazebo_motor_model.so">
+        <robotNamespace>${robot_namespace}</robotNamespace>
+        <jointName>${robot_namespace}/propeller_joint</jointName>
+        <linkName>${robot_namespace}/propeller</linkName>
+        <turningDirection>${direction}</turningDirection>
+        <timeConstantUp>${time_constant_up}</timeConstantUp>
+        <timeConstantDown>${time_constant_down}</timeConstantDown>
+        <maxRotVelocity>${max_propeller_velocity}</maxRotVelocity>
+        <motorConstant>${motor_constant}</motorConstant>
+        <momentConstant>${moment_constant}</momentConstant>
+        <commandSubTopic>gazebo/command/motor_speed</commandSubTopic>
+        <motorNumber>${motor_number}</motorNumber>
+        <rotorDragCoefficient>${rotor_drag_coefficient}</rotorDragCoefficient>
+        <rollingMomentCoefficient>${rolling_moment_coefficient}</rollingMomentCoefficient>
+        <motorSpeedPubTopic>motor_speed/${motor_number}</motorSpeedPubTopic>
+        <rotorVelocitySlowdownSim>${propeller_velocity_slowdown_sim}</rotorVelocitySlowdownSim>
+      </plugin>
+    </gazebo>
+    <gazebo reference="${robot_namespace}/propeller">
+      <material>Gazebo/${color}</material>
+    </gazebo>
   </xacro:macro>
 </robot>
