Commit message: Adding control surfaces to the model

File: rotors_description/urdf/atlantik_solar.xacro (robot description, xacro)
@@ -17,39 +17,29 @@
 -->
 <robot name="atlantik_solar" xmlns:xacro="http://ros.org/wiki/xacro">
-  <!-- Properties -->
+  <!-- Global properties -->
   <xacro:property name="namespace" value="$(arg mav_name)" />
   <xacro:property name="propeller_velocity_slowdown_sim" value="10" />
   <xacro:property name="use_mesh_file" value="false" />
   <xacro:property name="mesh_file" value="" />
+  <!-- Component masses -->
   <xacro:property name="mass_fuselage" value="3.0" /> <!-- [kg] -->
-  <xacro:property name="mass_wheel" value="0.1" /> <!-- [kg] -->
+  <xacro:property name="mass_wheel" value="0.05" /> <!-- [kg] -->
   <xacro:property name="mass_front_wing" value="1.0" /> <!-- [kg] -->
   <xacro:property name="mass_tail" value="0.5" /> <!-- [kg] -->
   <xacro:property name="mass_rear_wing" value="0.2" /> <!-- [kg] -->
-  <xacro:property name="mass_propeller" value="0.005" /> <!-- [kg] -->
+  <xacro:property name="mass_propeller" value="0.01" /> <!-- [kg] -->
+  <xacro:property name="mass_rudder" value="0.2" /> <!-- [kg] -->
+  <!-- Fuselage properties -->
   <xacro:property name="body_length" value="3.0" /> <!-- [m] -->
   <xacro:property name="body_width" value="0.1" /> <!-- [m] -->
   <xacro:property name="body_height" value="0.1" /> <!-- [m] -->
   <xacro:property name="body_color" value="Red" />
+  <!-- Wheel properties -->
   <xacro:property name="wheel_radius" value="0.05" /> <!-- [m] -->
   <xacro:property name="wheel_width" value="0.01" /> <!-- [m] -->
-  <xacro:property name="wingspan" value="4.0" /> <!-- [m] -->
-  <xacro:property name="root_chord" value="0.3" /> <!-- [m] -->
-  <xacro:property name="front_wing_height" value="0.02" /> <!-- [m] -->
-  <xacro:property name="front_wing_dihedral_angle" value="5" /> <!-- [deg] -->
-  <xacro:property name="tail_length" value="0.4" /> <!-- [m] -->
-  <xacro:property name="tail_width" value="0.05" /> <!-- [m] -->
-  <xacro:property name="tail_height" value="0.3" /> <!-- [m] -->
-  <xacro:property name="rear_wingspan" value="1.0" /> <!-- [m] -->
-  <xacro:property name="rear_wing_height" value="0.02" /> <!-- [m] -->
-  <xacro:property name="max_thrust" value="200.0" /> <!-- [N] -->
-  <xacro:property name="alpha_0" value="2.0" /> <!-- [deg] -->
-  <xacro:property name="alpha_stall" value="15.0" /> <!-- [deg] -->
-  <xacro:property name="c_L_alpha" value="${2.0 * PI}" />
-  <xacro:property name="air_density" value="1.225" /> <!-- [kg/m^3] -->
+  <!-- Propeller properties -->
+  <xacro:property name="propeller_offset" value="0.025" /> <!-- [m] -->
   <xacro:property name="radius_propeller" value="0.15" /> <!-- [m] -->
-  <xacro:property name="propeller_offset" value="0.025" /> <!-- [m] -->
   <xacro:property name="motor_constant" value="6.14858e-04" /> <!-- [kg m/s^2] -->
-  <!--<xacro:property name="motor_constant" value="8.54858e-06" />--> <!-- [kg m/s^2] -->
   <xacro:property name="moment_constant" value="0.016" /> <!-- [m] -->
   <xacro:property name="time_constant_up" value="0.0125" /> <!-- [s] -->
@@ -58,4 +48,26 @@
   <xacro:property name="rotor_drag_coefficient" value="8.06428e-05" />
   <xacro:property name="rolling_moment_coefficient" value="0.000001" />
+  <!-- Wing properties -->
+  <xacro:property name="wingspan" value="4.0" /> <!-- [m] -->
+  <xacro:property name="root_chord" value="0.3" /> <!-- [m] -->
+  <xacro:property name="front_wing_height" value="0.02" /> <!-- [m] -->
+  <xacro:property name="front_wing_dihedral_angle" value="5" /> <!-- [deg] -->
+  <xacro:property name="rear_wingspan" value="1.0" /> <!-- [m] -->
+  <xacro:property name="rear_wing_height" value="0.02" /> <!-- [m] -->
+  <xacro:property name="alpha_0" value="0.02" /> <!-- [rad] -->
+  <xacro:property name="alpha_stall" value="0.2" /> <!-- [rad] -->
+  <xacro:property name="c_L_alpha" value="4.0" />
+  <xacro:property name="air_density" value="1.225" /> <!-- [kg/m^3] -->
+  <!-- Tail properties -->
+  <xacro:property name="tail_length" value="0.4" /> <!-- [m] -->
+  <xacro:property name="tail_width" value="0.05" /> <!-- [m] -->
+  <xacro:property name="tail_height" value="0.3" /> <!-- [m] -->
+  <!-- Rudder properties -->
+  <xacro:property name="rudder_length" value="0.1" /> <!-- [m] -->
+  <xacro:property name="rudder_width" value="${tail_width}" /> <!-- [m] -->
+  <xacro:property name="rudder_height" value="${tail_height}" /> <!-- [m] -->
+  <xacro:property name="rudder_min_angle" value="-0.55" /> <!-- [rad] -->
+  <xacro:property name="rudder_max_angle" value="0.55" /> <!-- [rad] -->
+  <!-- Constants -->
   <xacro:property name="PI" value="3.1415926535897931" />
   <!-- Front wing length -->
@@ -88,4 +100,8 @@
     <xacro:box_inertia x="${radius_propeller}" y="0.04" z="0.003" mass="${mass_propeller * propeller_velocity_slowdown_sim}" />
   </xacro:property>
+  <!-- Inertia of the rudder, assuming it is a cuboid -->
+  <xacro:property name="rudder_inertia">
+    <xacro:box_inertia x="${rudder_length}" y="${rudder_width}" z="${rudder_height}" mass="${mass_rudder}" />
+  </xacro:property>
   <!-- Included URDF Files -->
   <xacro:include filename="$(find rotors_description)/urdf/fixed_wing_base.xacro" />
@@ -97,6 +113,4 @@
     body_width="${body_width}"
     body_height="${body_height}"
-    actuator_topic="actuators"
-    max_thrust="${max_thrust}"
     color="${body_color}"
     use_mesh_file="${use_mesh_file}"
@@ -206,5 +220,8 @@
     color="${body_color}"
     use_mesh="false"
-    mesh="">
+    mesh=""
+    alpha_0="${alpha_0}"
+    alpha_stall="${alpha_stall}"
+    c_L_alpha="${c_L_alpha}">
     <origin xyz="0.0 ${0.25 * (rear_wingspan + tail_width)} ${0.5 * (tail_height - rear_wing_height)}" rpy="0.0 0.0 0.0" />
     <xacro:insert_block name="rear_wing_inertia" />
@@ -220,5 +237,8 @@
     color="${body_color}"
     use_mesh="false"
-    mesh="">
+    mesh=""
+    alpha_0="${alpha_0}"
+    alpha_stall="${alpha_stall}"
+    c_L_alpha="${c_L_alpha}">
     <origin xyz="0.0 ${-0.25 * (rear_wingspan + tail_width)} ${0.5 * (tail_height - rear_wing_height)}" rpy="0.0 0.0 0.0" />
     <xacro:insert_block name="rear_wing_inertia" />
@@ -245,3 +265,22 @@
     <xacro:insert_block name="propeller_inertia" />
   </xacro:propeller>
+  <!-- Instantiate the control surfaces -->
+  <xacro:control_surface
+    robot_namespace="${namespace}"
+    surface_name="rudder"
+    parent="${namespace}/tail"
+    mass_surface="${mass_rudder}"
+    min_angle="${rudder_min_angle}"
+    max_angle="${rudder_max_angle}"
+    color="${body_color}"
+    use_mesh="false"
+    mesh=""
+    surface_length="${rudder_length}"
+    surface_width="${rudder_width}"
+    surface_height="${rudder_height}">
+    <axis xyz="0 0 1" />
+    <origin xyz="${-0.5 * tail_length} 0.0 0.0" rpy="0.0 0.0 0.0" /> <!-- Joint origin -->
+    <origin xyz="${-0.5 * rudder_length} 0.0 0.0" rpy="0.0 0.0 0.0" /> <!-- Link origin -->
+    <xacro:insert_block name="rudder_inertia" />
+  </xacro:control_surface>
 </robot>

File: rotors_description/urdf/fixed_wing_base.xacro (robot description, xacro)
@@ -40,5 +40,5 @@
   <xacro:macro name="fixed_wing_base_macro"
     params="robot_namespace mass body_length body_width body_height
-      actuator_topic max_thrust color use_mesh_file mesh_file *inertia">
+      color use_mesh_file mesh_file *inertia">
     <link name="${robot_namespace}/base_link"></link>
     <joint name="${robot_namespace}/base_joint" type="fixed">
@@ -71,12 +71,4 @@
       </collision>
     </link>
-    <gazebo>
-      <plugin name="fixed_wing_base_plugin" filename="librotors_gazebo_fixedwing_base_plugin.so">
-        <robotNamespace>${robot_namespace}</robotNamespace>
-        <linkName>${robot_namespace}/base_link</linkName>
-	<actuatorsTopic>${actuator_topic}</actuatorsTopic>
-        <maxThrust>${max_thrust}</maxThrust>
-      </plugin>
-    </gazebo>
     <gazebo reference="${robot_namespace}/base_link">
       <material>Gazebo/${color}</material>
@@ -85,5 +77,6 @@
   <!-- Wheel joint and link -->
   <xacro:macro name="wheel"
-    params="robot_namespace suffix parent mass_wheel color use_mesh mesh wheel_radius wheel_width *origin *inertia">
+    params="robot_namespace suffix parent mass_wheel color use_mesh mesh
+      wheel_radius wheel_width *origin *inertia">
     <joint name="${robot_namespace}/wheel_${suffix}_joint" type="revolute">
       <xacro:insert_block name="origin" />
@@ -158,9 +151,9 @@
       <plugin name="${robot_namespace}_${suffix}_lift_drag" filename="libLiftDragPlugin.so">
       <!--<plugin name="${robot_namespace}_${suffix}_lift_drag" filename="librotors_gazebo_lift_drag_plugin.so">-->
-        <a0>0.01</a0>
-        <cla>4.0</cla>
+        <a0>${alpha_0}</a0>
+        <cla>${c_L_alpha}</cla>
         <cda>0.01</cda>
         <cma>0.00</cma>
-        <alpha_stall>0.09</alpha_stall>
+        <alpha_stall>${alpha_stall}</alpha_stall>
         <cla_stall>0.0</cla_stall>
         <cda_stall>0.01</cda_stall>
@@ -218,5 +211,5 @@
   <xacro:macro name="rear_wing"
     params="robot_namespace suffix parent mass_rear_wing rear_wing_length rear_wing_width
-      rear_wing_height color use_mesh mesh *origin *inertia">
+      rear_wing_height color use_mesh mesh alpha_0 alpha_stall c_L_alpha *origin *inertia">
     <joint name="${robot_namespace}/rear_wing_${suffix}_joint" type="revolute">
       <xacro:insert_block name="origin" />
@@ -251,9 +244,9 @@
       <plugin name="${robot_namespace}_${suffix}_rear_lift_drag" filename="libLiftDragPlugin.so">
       <!--<plugin name="${robot_namespace}_${suffix}_lift_drag" filename="librotors_gazebo_lift_drag_plugin.so">-->
-        <a0>0.01</a0>
-        <cla>4.0</cla>
+        <a0>${alpha_0}</a0>
+        <cla>${c_L_alpha}</cla>
         <cda>0.01</cda>
         <cma>0.00</cma>
-        <alpha_stall>0.09</alpha_stall>
+        <alpha_stall>${alpha_stall}</alpha_stall>
         <cla_stall>0.0</cla_stall>
         <cda_stall>0.01</cda_stall>
@@ -328,3 +321,44 @@
     </gazebo>
   </xacro:macro>
+  <!-- Control surface joint and link -->
+  <xacro:macro name="control_surface"
+    params="robot_namespace surface_name parent mass_surface min_angle
+      max_angle color use_mesh mesh surface_length surface_width surface_height
+      *axis *joint_origin *link_origin *inertia">
+    <joint name="${robot_namespace}/${surface_name}_joint" type="revolute">
+      <xacro:insert_block name="joint_origin" />
+      <xacro:insert_block name="axis" />
+      <parent link="${parent}" />
+      <child link="${robot_namespace}/${surface_name}" />
+      <limit upper="${max_angle}" lower="${min_angle}" effort="100.0" velocity="3.0" />
+    </joint>
+    <link name="${robot_namespace}/${surface_name}">
+      <inertial>
+        <xacro:insert_block name="link_origin" />
+        <mass value="${mass_surface}" /> <!-- [kg] -->
+        <xacro:insert_block name="inertia" />
+      </inertial>
+      <visual>
+        <xacro:insert_block name="link_origin" />
+        <geometry>
+          <xacro:if value="${use_mesh}">
+            <mesh filename="${mesh}"
+              scale="1 1 1" />
+          </xacro:if>
+          <xacro:unless value="${use_mesh}">
+            <box size="${surface_length} ${surface_width} ${surface_height}"/> <!-- [m] [m] [m] -->
+          </xacro:unless>
+        </geometry>
+      </visual>
+      <collision>
+        <xacro:insert_block name="link_origin" />
+        <geometry>
+          <box size="${surface_length} ${surface_width} ${surface_height}"/> <!-- [m] [m] [m] -->
+        </geometry>
+      </collision>
+    </link>
+    <gazebo reference="${robot_namespace}/${surface_name}">
+      <material>Gazebo/${color}</material>
+    </gazebo>
+  </xacro:macro>
 </robot>

Commit message: Implementing the servo plugin

File: rotors_description/urdf/atlantik_solar.xacro (robot description, xacro)
@@ -67,4 +67,5 @@
   <xacro:property name="rudder_width" value="${tail_width}" /> <!-- [m] -->
   <xacro:property name="rudder_height" value="${tail_height}" /> <!-- [m] -->
+  <xacro:property name="rudder_velocity_gain" value="1.0" />
   <xacro:property name="rudder_min_angle" value="-0.55" /> <!-- [rad] -->
   <xacro:property name="rudder_max_angle" value="0.55" /> <!-- [rad] -->
@@ -271,6 +272,8 @@
     parent="${namespace}/tail"
     mass_surface="${mass_rudder}"
+    velocity_gain="${rudder_velocity_gain}"
     min_angle="${rudder_min_angle}"
     max_angle="${rudder_max_angle}"
+    channel="0"
     color="${body_color}"
     use_mesh="false"

File: rotors_description/urdf/fixed_wing_base.xacro (robot description, xacro)
@@ -71,4 +71,10 @@
       </collision>
     </link>
+    <gazebo>
+      <plugin name="${robot_namespace}_base" filename="librotors_gazebo_fixedwing_base_plugin.so">
+        <robotNamespace>${robot_namespace}</robotNamespace>
+        <linkName>${robot_namespace}/base_link</linkName>
+      </plugin>
+    </gazebo>
     <gazebo reference="${robot_namespace}/base_link">
       <material>Gazebo/${color}</material>
@@ -323,7 +329,7 @@
   <!-- Control surface joint and link -->
   <xacro:macro name="control_surface"
-    params="robot_namespace surface_name parent mass_surface min_angle
-      max_angle color use_mesh mesh surface_length surface_width surface_height
-      *axis *joint_origin *link_origin *inertia">
+    params="robot_namespace surface_name parent mass_surface velocity_gain
+      min_angle max_angle channel color use_mesh mesh surface_length surface_width
+      surface_height *axis *joint_origin *link_origin *inertia">
     <joint name="${robot_namespace}/${surface_name}_joint" type="revolute">
       <xacro:insert_block name="joint_origin" />
@@ -358,4 +364,15 @@
       </collision>
     </link>
+    <gazebo>
+      <plugin name="${robot_namespace}_${surface_name}" filename="librotors_gazebo_servo_plugin.so">
+        <robotNamespace>${robot_namespace}</robotNamespace>
+        <jointName>${robot_namespace}/${surface_name}_joint</jointName>
+        <commandSubTopic>gazebo/command/motor_speed</commandSubTopic>
+        <velocityGain>${velocity_gain}</velocityGain>
+        <minAngle>${min_angle}</minAngle>
+        <maxAngle>${max_angle}</maxAngle>
+        <channel>${channel}</channel>
+      </plugin>
+    </gazebo>
     <gazebo reference="${robot_namespace}/${surface_name}">
       <material>Gazebo/${color}</material>
