Commit message: Moving elevators to the back of the plane

File: rotors_description/urdf/atlantik_solar.xacro (robot description, xacro)
@@ -26,10 +26,11 @@
   <xacro:property name="mass_wheel" value="0.05" /> <!-- [kg] -->
   <xacro:property name="mass_front_wing" value="1.0" /> <!-- [kg] -->
+  <xacro:property name="mass_small_wing" value="${0.3 * mass_front_wing}" /> <!-- [kg] -->
   <xacro:property name="mass_tail" value="0.5" /> <!-- [kg] -->
   <xacro:property name="mass_rear_wing" value="0.2" /> <!-- [kg] -->
   <xacro:property name="mass_propeller" value="0.01" /> <!-- [kg] -->
   <xacro:property name="mass_aileron" value="0.2" /> <!-- [kg] -->
-  <xacro:property name="mass_elevator" value="0.2" /> <!-- [kg] -->
-  <xacro:property name="mass_rudder" value="0.2" /> <!-- [kg] -->
+  <xacro:property name="mass_elevator" value="0.1" /> <!-- [kg] -->
+  <xacro:property name="mass_rudder" value="0.1" /> <!-- [kg] -->
   <!-- Fuselage properties -->
   <xacro:property name="body_length" value="3.0" /> <!-- [m] -->
@@ -66,5 +67,5 @@
   <!-- Aileron properties -->
   <xacro:property name="aileron_length" value="${0.5 * root_chord}" /> <!-- [m] -->
-  <xacro:property name="aileron_width" value="${0.5 * front_wing_length - 0.05}" /> <!-- [m] -->
+  <xacro:property name="aileron_width" value="${0.5 * front_wing_width}" /> <!-- [m] -->
   <xacro:property name="aileron_height" value="0.02" /> <!-- [m] -->
   <xacro:property name="aileron_velocity_gain" value="1.0" />
@@ -73,6 +74,6 @@
   <xacro:property name="aileron_channel" value="0" />
   <!-- Elevator properties -->
-  <xacro:property name="elevator_length" value="${0.5 * root_chord}" /> <!-- [m] -->
-  <xacro:property name="elevator_width" value="${0.5 * front_wing_length - 0.05}" /> <!-- [m] -->
+  <xacro:property name="elevator_length" value="0.15" /> <!-- [m] -->
+  <xacro:property name="elevator_width" value="${rear_wing_width}" /> <!-- [m] -->
   <xacro:property name="elevator_height" value="0.02" /> <!-- [m] -->
   <xacro:property name="elevator_velocity_gain" value="1.0" />
@@ -91,7 +92,7 @@
   <xacro:property name="PI" value="3.1415926535897931" />
   <!-- Front wing length -->
-  <xacro:property name="front_wing_length" value="${0.5 * (wingspan - body_width)}" />
+  <xacro:property name="front_wing_width" value="${0.5 * (wingspan - body_width)}" />
   <!-- Rear wing length -->
-  <xacro:property name="rear_wing_length" value="${0.5 * (rear_wingspan - tail_width)}" />
+  <xacro:property name="rear_wing_width" value="${0.5 * (rear_wingspan - tail_width)}" />
   <!-- Inertia of the fuselage -->
   <xacro:property name="body_inertia">
@@ -104,5 +105,9 @@
   <!-- Inertia of a single front wing, assuming it is a cuboid -->
   <xacro:property name="front_wing_inertia">
-    <xacro:box_inertia x="${root_chord}" y="${front_wing_length}" z="${front_wing_height}" mass="${mass_front_wing}" />
+    <xacro:box_inertia x="${root_chord}" y="${front_wing_width}" z="${front_wing_height}" mass="${mass_front_wing}" />
+  </xacro:property>
+  <!-- Inertia of a single small front wing, assuming it is a cuboid -->
+  <xacro:property name="small_wing_inertia">
+    <xacro:box_inertia x="${aileron_length}" y="${front_wing_width - aileron_width}" z="${front_wing_height}" mass="${0.3 * mass_small_wing}" />
   </xacro:property>
   <!-- Inertia of the tail, assuming it is a cuboid -->
@@ -112,5 +117,5 @@
   <!-- Inertia of a single rear wing, assuming it is a cuboid -->
   <xacro:property name="rear_wing_inertia">
-    <xacro:box_inertia x="${tail_length}" y="${rear_wing_length}" z="${rear_wing_height}" mass="${mass_rear_wing}" />
+    <xacro:box_inertia x="${tail_length - elevator_length}" y="${rear_wing_width}" z="${rear_wing_height}" mass="${mass_rear_wing}" />
   </xacro:property>
   <!-- Inertia of the propeller, assuming it is a cuboid. Height=3mm, width=40mm -->
@@ -187,9 +192,9 @@
   <xacro:wing
     robot_namespace="${namespace}"
-    suffix="left"
+    suffix="left_big"
     parent="${namespace}/base_link"
     mass_wing="${mass_front_wing}"
     wing_length="${root_chord}"
-    wing_width="${front_wing_length}"
+    wing_width="${front_wing_width}"
     wing_height="${front_wing_height}"
     color="${body_color}"
@@ -200,14 +205,14 @@
     c_L_alpha="${c_L_alpha}"
     air_density="${air_density}">
-    <origin xyz="0.5 ${0.25 * (wingspan + body_width)} 0.1" rpy="0.0 0.0 0.0" />
+    <origin xyz="0.5 ${0.5 * (body_width + front_wing_width)} 0.1" rpy="0.0 0.0 0.0" />
     <xacro:insert_block name="front_wing_inertia" />
   </xacro:wing>-->
   <xacro:wing
     robot_namespace="${namespace}"
-    suffix="right"
+    suffix="right_big"
     parent="${namespace}/base_link"
     mass_wing="${mass_front_wing}"
     wing_length="${root_chord}"
-    wing_width="${front_wing_length}"
+    wing_width="${front_wing_width}"
     wing_height="${front_wing_height}"
     color="${body_color}"
@@ -218,6 +223,42 @@
     c_L_alpha="${c_L_alpha}"
     air_density="${air_density}">
-    <origin xyz="0.5 ${-0.25 * (wingspan + body_width)} 0.1" rpy="0.0 0.0 0.0" />
+    <origin xyz="0.5 ${-0.5 * (body_width + front_wing_width)} 0.1" rpy="0.0 0.0 0.0" />
     <xacro:insert_block name="front_wing_inertia" />
+  </xacro:wing>
+  <xacro:wing
+    robot_namespace="${namespace}"
+    suffix="left_small"
+    parent="${namespace}/base_link"
+    mass_wing="${mass_small_wing}"
+    wing_length="${aileron_length}"
+    wing_width="${front_wing_width - aileron_width}"
+    wing_height="${front_wing_height}"
+    color="${body_color}"
+    use_mesh="false"
+    mesh=""
+    alpha_0="${alpha_0}"
+    alpha_stall="${alpha_stall}"
+    c_L_alpha="${c_L_alpha}"
+    air_density="${air_density}">
+    <origin xyz="${0.5 * (1 - root_chord - aileron_length)} ${0.5 * (body_width + front_wing_width - aileron_width)} 0.1" rpy="0.0 0.0 0.0" />
+    <xacro:insert_block name="small_wing_inertia" />
+  </xacro:wing>
+  <xacro:wing
+    robot_namespace="${namespace}"
+    suffix="right_small"
+    parent="${namespace}/base_link"
+    mass_wing="${mass_small_wing}"
+    wing_length="${aileron_length}"
+    wing_width="${front_wing_width - aileron_width}"
+    wing_height="${front_wing_height}"
+    color="${body_color}"
+    use_mesh="false"
+    mesh=""
+    alpha_0="${alpha_0}"
+    alpha_stall="${alpha_stall}"
+    c_L_alpha="${c_L_alpha}"
+    air_density="${air_density}">
+    <origin xyz="${0.5 * (1 - root_chord - aileron_length)} ${-0.5 * (body_width + front_wing_width - aileron_width)} 0.1" rpy="0.0 0.0 0.0" />
+    <xacro:insert_block name="small_wing_inertia" />
   </xacro:wing>
   <!-- Instantiate the tail -->
@@ -241,6 +282,6 @@
     parent="${namespace}/tail"
     mass_rear_wing="${mass_rear_wing}"
-    rear_wing_length="${tail_length}"
-    rear_wing_width="${rear_wing_length}"
+    rear_wing_length="${tail_length - elevator_length}"
+    rear_wing_width="${rear_wing_width}"
     rear_wing_height="${rear_wing_height}"
     color="${body_color}"
@@ -249,6 +290,7 @@
     alpha_0="${alpha_0}"
     alpha_stall="${alpha_stall}"
-    c_L_alpha="${c_L_alpha}">
-    <origin xyz="0.0 ${0.25 * (rear_wingspan + tail_width)} ${0.5 * (tail_height - rear_wing_height)}" rpy="0.0 0.0 0.0" />
+    c_L_alpha="${c_L_alpha}"
+    air_density="${air_density}">
+    <origin xyz="${0.5 * elevator_length} ${0.5 * (tail_width + rear_wing_width)} ${0.5 * (tail_height - rear_wing_height)}" rpy="0.0 0.0 0.0" />
     <xacro:insert_block name="rear_wing_inertia" />
   </xacro:rear_wing>
@@ -258,6 +300,6 @@
     parent="${namespace}/tail"
     mass_rear_wing="${mass_rear_wing}"
-    rear_wing_length="${tail_length}"
-    rear_wing_width="${rear_wing_length}"
+    rear_wing_length="${tail_length - elevator_length}"
+    rear_wing_width="${rear_wing_width}"
     rear_wing_height="${rear_wing_height}"
     color="${body_color}"
@@ -266,6 +308,7 @@
     alpha_0="${alpha_0}"
     alpha_stall="${alpha_stall}"
-    c_L_alpha="${c_L_alpha}">
-    <origin xyz="0.0 ${-0.25 * (rear_wingspan + tail_width)} ${0.5 * (tail_height - rear_wing_height)}" rpy="0.0 0.0 0.0" />
+    c_L_alpha="${c_L_alpha}"
+    air_density="${air_density}">
+    <origin xyz="${0.5 * elevator_length} ${-0.5 * (tail_width + rear_wing_width)} ${0.5 * (tail_height - rear_wing_height)}" rpy="0.0 0.0 0.0" />
     <xacro:insert_block name="rear_wing_inertia" />
   </xacro:rear_wing>
@@ -295,5 +338,5 @@
     robot_namespace="${namespace}"
     surface_name="aileron_left"
-    parent="${namespace}/wing_left"
+    parent="${namespace}/wing_left_big"
     mass_surface="${mass_aileron}"
     velocity_gain="${aileron_velocity_gain}"
@@ -307,7 +350,16 @@
     surface_length="${aileron_length}"
     surface_width="${aileron_width}"
-    surface_height="${aileron_height}">
+    surface_height="${aileron_height}"
+    area="${aileron_length * aileron_width}"
+    forward_x="1"
+    forward_y="0"
+    forward_z="0"
+    up_x="0"
+    up_y="0"
+    up_z="1"
+    c_L_alpha="${c_L_alpha}"
+    alpha_stall="${alpha_stall}">
     <axis xyz="0 1 0" />
-    <origin xyz="${-0.5 * root_chord} ${-0.25 * front_wing_length} 0.0" rpy="0.0 0.0 0.0" /> <!-- Joint origin -->
+    <origin xyz="${-0.5 * root_chord} ${0.25 * front_wing_width} 0.0" rpy="0.0 0.0 0.0" /> <!-- Joint origin -->
     <origin xyz="${-0.5 * aileron_length} 0.0 0.0" rpy="0.0 0.0 0.0" /> <!-- Link origin -->
     <xacro:insert_block name="aileron_inertia" />
@@ -316,5 +368,5 @@
     robot_namespace="${namespace}"
     surface_name="aileron_right"
-    parent="${namespace}/wing_right"
+    parent="${namespace}/wing_right_big"
     mass_surface="${mass_aileron}"
     velocity_gain="${aileron_velocity_gain}"
@@ -328,7 +380,16 @@
     surface_length="${aileron_length}"
     surface_width="${aileron_width}"
-    surface_height="${aileron_height}">
+    surface_height="${aileron_height}"
+    area="${aileron_length * aileron_width}"
+    forward_x="1"
+    forward_y="0"
+    forward_z="0"
+    up_x="0"
+    up_y="0"
+    up_z="1"
+    c_L_alpha="${c_L_alpha}"
+    alpha_stall="${alpha_stall}">
     <axis xyz="0 1 0" />
-    <origin xyz="${-0.5 * root_chord} ${0.25 * front_wing_length} 0.0" rpy="0.0 0.0 0.0" /> <!-- Joint origin -->
+    <origin xyz="${-0.5 * root_chord} ${-0.25 * front_wing_width} 0.0" rpy="0.0 0.0 0.0" /> <!-- Joint origin -->
     <origin xyz="${-0.5 * aileron_length} 0.0 0.0" rpy="0.0 0.0 0.0" /> <!-- Link origin -->
     <xacro:insert_block name="aileron_inertia" />
@@ -337,5 +398,5 @@
     robot_namespace="${namespace}"
     surface_name="elevator_left"
-    parent="${namespace}/wing_left"
+    parent="${namespace}/rear_wing_left"
     mass_surface="${mass_elevator}"
     velocity_gain="${elevator_velocity_gain}"
@@ -349,7 +410,16 @@
     surface_length="${elevator_length}"
     surface_width="${elevator_width}"
-    surface_height="${elevator_height}">
+    surface_height="${elevator_height}"
+    area="${elevator_length * elevator_width}"
+    forward_x="1"
+    forward_y="0"
+    forward_z="0"
+    up_x="0"
+    up_y="0"
+    up_z="1"
+    c_L_alpha="${c_L_alpha}"
+    alpha_stall="${alpha_stall}">
     <axis xyz="0 1 0" />
-    <origin xyz="${-0.5 * root_chord} ${0.25 * front_wing_length} 0.0" rpy="0.0 0.0 0.0" /> <!-- Joint origin -->
+    <origin xyz="${-0.5 * (tail_length - elevator_length)} 0.0 0.0" rpy="0.0 0.0 0.0" /> <!-- Joint origin -->
     <origin xyz="${-0.5 * elevator_length} 0.0 0.0" rpy="0.0 0.0 0.0" /> <!-- Link origin -->
     <xacro:insert_block name="elevator_inertia" />
@@ -358,5 +428,5 @@
     robot_namespace="${namespace}"
     surface_name="elevator_right"
-    parent="${namespace}/wing_right"
+    parent="${namespace}/rear_wing_right"
     mass_surface="${mass_elevator}"
     velocity_gain="${elevator_velocity_gain}"
@@ -370,7 +440,16 @@
     surface_length="${elevator_length}"
     surface_width="${elevator_width}"
-    surface_height="${elevator_height}">
+    surface_height="${elevator_height}"
+    area="${elevator_length * elevator_width}"
+    forward_x="1"
+    forward_y="0"
+    forward_z="0"
+    up_x="0"
+    up_y="0"
+    up_z="1"
+    c_L_alpha="${c_L_alpha}"
+    alpha_stall="${alpha_stall}">
     <axis xyz="0 1 0" />
-    <origin xyz="${-0.5 * root_chord} ${-0.25 * front_wing_length} 0.0" rpy="0.0 0.0 0.0" /> <!-- Joint origin -->
+    <origin xyz="${-0.5 * (tail_length - elevator_length)} 0.0 0.0" rpy="0.0 0.0 0.0" /> <!-- Joint origin -->
     <origin xyz="${-0.5 * elevator_length} 0.0 0.0" rpy="0.0 0.0 0.0" /> <!-- Link origin -->
     <xacro:insert_block name="elevator_inertia" />
@@ -391,5 +470,14 @@
     surface_length="${rudder_length}"
     surface_width="${rudder_width}"
-    surface_height="${rudder_height}">
+    surface_height="${rudder_height}"
+    area="0.0"
+    forward_x="0"
+    forward_y="0"
+    forward_z="0"
+    up_x="0"
+    up_y="0"
+    up_z="0"
+    c_L_alpha="0.0"
+    alpha_stall="0.0">
     <axis xyz="0 0 1" />
     <origin xyz="${-0.5 * tail_length} 0.0 0.0" rpy="0.0 0.0 0.0" /> <!-- Joint origin -->

File: rotors_description/urdf/fixed_wing_base.xacro (robot description, xacro)
@@ -216,5 +216,5 @@
   <xacro:macro name="rear_wing"
     params="robot_namespace suffix parent mass_rear_wing rear_wing_length rear_wing_width
-      rear_wing_height color use_mesh mesh alpha_0 alpha_stall c_L_alpha *origin *inertia">
+      rear_wing_height color use_mesh mesh alpha_0 alpha_stall c_L_alpha air_density *origin *inertia">
     <joint name="${robot_namespace}/rear_wing_${suffix}_joint" type="revolute">
       <xacro:insert_block name="origin" />
@@ -258,5 +258,5 @@
         <cp>0.0 0.0 0.0</cp>
         <area>${rear_wing_length * rear_wing_width}</area>
-        <air_density>1.225</air_density>
+        <air_density>${air_density}</air_density>
         <forward>1 0 0</forward>
         <upward>0 0 1</upward>
@@ -329,6 +329,6 @@
     params="robot_namespace surface_name parent mass_surface velocity_gain
       positive_direction min_angle max_angle channel color use_mesh mesh
-      surface_length surface_width surface_height *axis *joint_origin
-      *link_origin *inertia">
+      surface_length surface_width surface_height area forward_x forward_y
+      forward_z up_x up_y up_z c_L_alpha alpha_stall *axis *joint_origin *link_origin *inertia">
     <joint name="${robot_namespace}/${surface_name}_joint" type="revolute">
       <xacro:insert_block name="joint_origin" />
@@ -365,5 +365,5 @@
     </link>
     <gazebo>
-      <plugin name="${robot_namespace}_${surface_name}" filename="librotors_gazebo_servo_plugin.so">
+      <plugin name="${robot_namespace}_${surface_name}_servo" filename="librotors_gazebo_servo_plugin.so">
         <robotNamespace>${robot_namespace}</robotNamespace>
         <jointName>${robot_namespace}/${surface_name}_joint</jointName>
@@ -377,4 +377,22 @@
       </plugin>
     </gazebo>
+    <gazebo>
+      <plugin name="${robot_namespace}_${surface_name}_lift_drag" filename="libLiftDragPlugin.so">
+        <a0>0.0</a0>
+        <cla>${c_L_alpha}</cla>
+        <cda>0.1</cda>
+        <cma>-0.1</cma>
+        <alpha_stall>${alpha_stall}</alpha_stall>
+        <cla_stall>-0.1</cla_stall>
+        <cda_stall>0.1</cda_stall>
+        <cma_stall>-0.2</cma_stall>
+        <cp>0.0 0.0 0.0</cp>
+        <area>${area}</area>
+        <air_density>1.225</air_density>
+        <forward>${forward_x} ${forward_y} ${forward_z}</forward>
+        <upward>${up_x} ${up_y} ${up_z}</upward>
+        <link_name>${robot_namespace}/${surface_name}</link_name>
+      </plugin>
+    </gazebo>
     <gazebo reference="${robot_namespace}/${surface_name}">
       <material>Gazebo/${color}</material>
