Commit message: Committing all changes for transfer to another machine

File: rotors_description/urdf/atlantik_solar.xacro (robot description, xacro)
@@ -149,339 +149,3 @@
     <xacro:insert_block name="body_inertia" />
   </xacro:fixed_wing_base_macro>
-  <!-- Instantiate wheels -->
-  <xacro:wheel
-    robot_namespace="${namespace}"
-    suffix="front_left"
-    parent="${namespace}/base_link"
-    mass_wheel="${mass_wheel}"
-    color="${body_color}"
-    use_mesh="false"
-    mesh=""
-    wheel_radius="${wheel_radius}"
-    wheel_width="${wheel_width}">
-    <origin xyz="0.75 0.1 0.0" rpy="${0.5 * PI} 0.0 0.0" />
-    <xacro:insert_block name="wheel_inertia" />
-  </xacro:wheel>
-  <xacro:wheel
-    robot_namespace="${namespace}"
-    suffix="front_right"
-    parent="${namespace}/base_link"
-    mass_wheel="${mass_wheel}"
-    color="${body_color}"
-    use_mesh="false"
-    mesh=""
-    wheel_radius="${wheel_radius}"
-    wheel_width="${wheel_width}">
-    <origin xyz="0.75 -0.1 0.0" rpy="${0.5 * PI} 0.0 0.0" />
-    <xacro:insert_block name="wheel_inertia" />
-  </xacro:wheel>
-  <xacro:wheel
-    robot_namespace="${namespace}"
-    suffix="back"
-    parent="${namespace}/base_link"
-    mass_wheel="${mass_wheel}"
-    color="${body_color}"
-    use_mesh="false"
-    mesh=""
-    wheel_radius="${wheel_radius}"
-    wheel_width="${wheel_width}">
-    <origin xyz="-1.0 0.0 0.0" rpy="${0.5 * PI} 0.0 0.0" />
-    <xacro:insert_block name="wheel_inertia" />
-  </xacro:wheel>
-  <!-- Instantiate wings -->
-  <xacro:wing
-    robot_namespace="${namespace}"
-    suffix="left_big"
-    parent="${namespace}/base_link"
-    mass_wing="${mass_front_wing}"
-    wing_length="${root_chord}"
-    wing_width="${front_wing_width}"
-    wing_height="${front_wing_height}"
-    color="${body_color}"
-    use_mesh="false"
-    mesh=""
-    alpha_0="${alpha_0}"
-    alpha_stall="${alpha_stall}"
-    c_L_alpha="${c_L_alpha}"
-    air_density="${air_density}">
-    <origin xyz="0.5 ${0.5 * (body_width + front_wing_width)} 0.1" rpy="0.0 0.0 0.0" />
-    <xacro:insert_block name="front_wing_inertia" />
-  </xacro:wing>-->
-  <xacro:wing
-    robot_namespace="${namespace}"
-    suffix="right_big"
-    parent="${namespace}/base_link"
-    mass_wing="${mass_front_wing}"
-    wing_length="${root_chord}"
-    wing_width="${front_wing_width}"
-    wing_height="${front_wing_height}"
-    color="${body_color}"
-    use_mesh="false"
-    mesh=""
-    alpha_0="${alpha_0}"
-    alpha_stall="${alpha_stall}"
-    c_L_alpha="${c_L_alpha}"
-    air_density="${air_density}">
-    <origin xyz="0.5 ${-0.5 * (body_width + front_wing_width)} 0.1" rpy="0.0 0.0 0.0" />
-    <xacro:insert_block name="front_wing_inertia" />
-  </xacro:wing>
-  <xacro:wing
-    robot_namespace="${namespace}"
-    suffix="left_small"
-    parent="${namespace}/base_link"
-    mass_wing="${mass_small_wing}"
-    wing_length="${aileron_length}"
-    wing_width="${front_wing_width - aileron_width}"
-    wing_height="${front_wing_height}"
-    color="${body_color}"
-    use_mesh="false"
-    mesh=""
-    alpha_0="${alpha_0}"
-    alpha_stall="${alpha_stall}"
-    c_L_alpha="${c_L_alpha}"
-    air_density="${air_density}">
-    <origin xyz="${0.5 * (1 - root_chord - aileron_length)} ${0.5 * (body_width + front_wing_width - aileron_width)} 0.1" rpy="0.0 0.0 0.0" />
-    <xacro:insert_block name="small_wing_inertia" />
-  </xacro:wing>
-  <xacro:wing
-    robot_namespace="${namespace}"
-    suffix="right_small"
-    parent="${namespace}/base_link"
-    mass_wing="${mass_small_wing}"
-    wing_length="${aileron_length}"
-    wing_width="${front_wing_width - aileron_width}"
-    wing_height="${front_wing_height}"
-    color="${body_color}"
-    use_mesh="false"
-    mesh=""
-    alpha_0="${alpha_0}"
-    alpha_stall="${alpha_stall}"
-    c_L_alpha="${c_L_alpha}"
-    air_density="${air_density}">
-    <origin xyz="${0.5 * (1 - root_chord - aileron_length)} ${-0.5 * (body_width + front_wing_width - aileron_width)} 0.1" rpy="0.0 0.0 0.0" />
-    <xacro:insert_block name="small_wing_inertia" />
-  </xacro:wing>
-  <!-- Instantiate the tail -->
-  <xacro:tail
-    robot_namespace="${namespace}"
-    parent="${namespace}/base_link"
-    mass_tail="${mass_tail}"
-    tail_length="${tail_length}"
-    tail_width="${tail_width}"
-    tail_height="${tail_height}"
-    color="${body_color}"
-    use_mesh="false"
-    mesh="">
-    <origin xyz="${-0.5*body_length + 0.5*tail_length} 0.0 ${0.5*body_height + 0.5*tail_height + 0.1}" rpy="0.0 0.0 0.0" />
-    <xacro:insert_block name="tail_inertia" />
-  </xacro:tail>
-  <!-- Instantiate the rear wings-->
-  <xacro:rear_wing
-    robot_namespace="${namespace}"
-    suffix="left"
-    parent="${namespace}/tail"
-    mass_rear_wing="${mass_rear_wing}"
-    rear_wing_length="${tail_length - elevator_length}"
-    rear_wing_width="${rear_wing_width}"
-    rear_wing_height="${rear_wing_height}"
-    color="${body_color}"
-    use_mesh="false"
-    mesh=""
-    alpha_0="${alpha_0}"
-    alpha_stall="${alpha_stall}"
-    c_L_alpha="${c_L_alpha}"
-    air_density="${air_density}">
-    <origin xyz="${0.5 * elevator_length} ${0.5 * (tail_width + rear_wing_width)} ${0.5 * (tail_height - rear_wing_height)}" rpy="0.0 0.0 0.0" />
-    <xacro:insert_block name="rear_wing_inertia" />
-  </xacro:rear_wing>
-  <xacro:rear_wing
-    robot_namespace="${namespace}"
-    suffix="right"
-    parent="${namespace}/tail"
-    mass_rear_wing="${mass_rear_wing}"
-    rear_wing_length="${tail_length - elevator_length}"
-    rear_wing_width="${rear_wing_width}"
-    rear_wing_height="${rear_wing_height}"
-    color="${body_color}"
-    use_mesh="false"
-    mesh=""
-    alpha_0="${alpha_0}"
-    alpha_stall="${alpha_stall}"
-    c_L_alpha="${c_L_alpha}"
-    air_density="${air_density}">
-    <origin xyz="${0.5 * elevator_length} ${-0.5 * (tail_width + rear_wing_width)} ${0.5 * (tail_height - rear_wing_height)}" rpy="0.0 0.0 0.0" />
-    <xacro:insert_block name="rear_wing_inertia" />
-  </xacro:rear_wing>
-  <!-- Instantiate the propeller -->
-  <xacro:propeller
-    robot_namespace="${namespace}"
-    direction="cw"
-    motor_constant="${motor_constant}"
-    moment_constant="${moment_constant}"
-    parent="${namespace}/base_link"
-    mass_propeller="${mass_propeller}"
-    radius_propeller="${radius_propeller}"
-    time_constant_up="${time_constant_up}"
-    time_constant_down="${time_constant_down}"
-    max_propeller_velocity="${max_propeller_velocity}"
-    motor_number="0"
-    rotor_drag_coefficient="${rotor_drag_coefficient}"
-    rolling_moment_coefficient="${rolling_moment_coefficient}"
-    color="Blue"
-    use_own_mesh="false"
-    mesh="">
-    <origin xyz="${0.5 * body_length + propeller_offset} 0.0 0.1" rpy="0.0 ${0.5 * PI} 0.0" />
-    <xacro:insert_block name="propeller_inertia" />
-  </xacro:propeller>
-  <!-- Instantiate the control surfaces -->
-  <xacro:control_surface
-    robot_namespace="${namespace}"
-    surface_name="aileron_left"
-    parent="${namespace}/wing_left_big"
-    mass_surface="${mass_aileron}"
-    velocity_gain="${aileron_velocity_gain}"
-    positive_direction="ccw"
-    min_angle="${aileron_min_angle}"
-    max_angle="${aileron_max_angle}"
-    channel="${aileron_channel}"
-    color="Orange"
-    use_mesh="false"
-    mesh=""
-    surface_length="${aileron_length}"
-    surface_width="${aileron_width}"
-    surface_height="${aileron_height}"
-    area="${aileron_length * aileron_width}"
-    forward_x="1"
-    forward_y="0"
-    forward_z="0"
-    up_x="0"
-    up_y="0"
-    up_z="1"
-    c_L_alpha="${c_L_alpha}"
-    alpha_stall="${alpha_stall}">
-    <axis xyz="0 1 0" />
-    <origin xyz="${-0.5 * root_chord} ${0.25 * front_wing_width} 0.0" rpy="0.0 0.0 0.0" /> <!-- Joint origin -->
-    <origin xyz="${-0.5 * aileron_length} 0.0 0.0" rpy="0.0 0.0 0.0" /> <!-- Link origin -->
-    <xacro:insert_block name="aileron_inertia" />
-  </xacro:control_surface>
-  <xacro:control_surface
-    robot_namespace="${namespace}"
-    surface_name="aileron_right"
-    parent="${namespace}/wing_right_big"
-    mass_surface="${mass_aileron}"
-    velocity_gain="${aileron_velocity_gain}"
-    positive_direction="cw"
-    min_angle="${aileron_min_angle}"
-    max_angle="${aileron_max_angle}"
-    channel="${aileron_channel}"
-    color="Orange"
-    use_mesh="false"
-    mesh=""
-    surface_length="${aileron_length}"
-    surface_width="${aileron_width}"
-    surface_height="${aileron_height}"
-    area="${aileron_length * aileron_width}"
-    forward_x="1"
-    forward_y="0"
-    forward_z="0"
-    up_x="0"
-    up_y="0"
-    up_z="1"
-    c_L_alpha="${c_L_alpha}"
-    alpha_stall="${alpha_stall}">
-    <axis xyz="0 1 0" />
-    <origin xyz="${-0.5 * root_chord} ${-0.25 * front_wing_width} 0.0" rpy="0.0 0.0 0.0" /> <!-- Joint origin -->
-    <origin xyz="${-0.5 * aileron_length} 0.0 0.0" rpy="0.0 0.0 0.0" /> <!-- Link origin -->
-    <xacro:insert_block name="aileron_inertia" />
-  </xacro:control_surface>
-  <xacro:control_surface
-    robot_namespace="${namespace}"
-    surface_name="elevator_left"
-    parent="${namespace}/rear_wing_left"
-    mass_surface="${mass_elevator}"
-    velocity_gain="${elevator_velocity_gain}"
-    positive_direction="ccw"
-    min_angle="${elevator_min_angle}"
-    max_angle="${elevator_max_angle}"
-    channel="${elevator_channel}"
-    color="Blue"
-    use_mesh="false"
-    mesh=""
-    surface_length="${elevator_length}"
-    surface_width="${elevator_width}"
-    surface_height="${elevator_height}"
-    area="${elevator_length * elevator_width}"
-    forward_x="1"
-    forward_y="0"
-    forward_z="0"
-    up_x="0"
-    up_y="0"
-    up_z="1"
-    c_L_alpha="${c_L_alpha}"
-    alpha_stall="${alpha_stall}">
-    <axis xyz="0 1 0" />
-    <origin xyz="${-0.5 * (tail_length - elevator_length)} 0.0 0.0" rpy="0.0 0.0 0.0" /> <!-- Joint origin -->
-    <origin xyz="${-0.5 * elevator_length} 0.0 0.0" rpy="0.0 0.0 0.0" /> <!-- Link origin -->
-    <xacro:insert_block name="elevator_inertia" />
-  </xacro:control_surface>
-  <xacro:control_surface
-    robot_namespace="${namespace}"
-    surface_name="elevator_right"
-    parent="${namespace}/rear_wing_right"
-    mass_surface="${mass_elevator}"
-    velocity_gain="${elevator_velocity_gain}"
-    positive_direction="ccw"
-    min_angle="${elevator_min_angle}"
-    max_angle="${elevator_max_angle}"
-    channel="${elevator_channel}"
-    color="Blue"
-    use_mesh="false"
-    mesh=""
-    surface_length="${elevator_length}"
-    surface_width="${elevator_width}"
-    surface_height="${elevator_height}"
-    area="${elevator_length * elevator_width}"
-    forward_x="1"
-    forward_y="0"
-    forward_z="0"
-    up_x="0"
-    up_y="0"
-    up_z="1"
-    c_L_alpha="${c_L_alpha}"
-    alpha_stall="${alpha_stall}">
-    <axis xyz="0 1 0" />
-    <origin xyz="${-0.5 * (tail_length - elevator_length)} 0.0 0.0" rpy="0.0 0.0 0.0" /> <!-- Joint origin -->
-    <origin xyz="${-0.5 * elevator_length} 0.0 0.0" rpy="0.0 0.0 0.0" /> <!-- Link origin -->
-    <xacro:insert_block name="elevator_inertia" />
-  </xacro:control_surface>
-  <xacro:control_surface
-    robot_namespace="${namespace}"
-    surface_name="rudder"
-    parent="${namespace}/tail"
-    mass_surface="${mass_rudder}"
-    velocity_gain="${rudder_velocity_gain}"
-    positive_direction="cw"
-    min_angle="${rudder_min_angle}"
-    max_angle="${rudder_max_angle}"
-    channel="${rudder_channel}"
-    color="Gray"
-    use_mesh="false"
-    mesh=""
-    surface_length="${rudder_length}"
-    surface_width="${rudder_width}"
-    surface_height="${rudder_height}"
-    area="0.0"
-    forward_x="0"
-    forward_y="0"
-    forward_z="0"
-    up_x="0"
-    up_y="0"
-    up_z="0"
-    c_L_alpha="0.0"
-    alpha_stall="0.0">
-    <axis xyz="0 0 1" />
-    <origin xyz="${-0.5 * tail_length} 0.0 0.0" rpy="0.0 0.0 0.0" /> <!-- Joint origin -->
-    <origin xyz="${-0.5 * rudder_length} 0.0 0.0" rpy="0.0 0.0 0.0" /> <!-- Link origin -->
-    <xacro:insert_block name="rudder_inertia" />
-  </xacro:control_surface>
 </robot>
