Commit message: Fixing some moments of inertia

File: rotors_description/urdf/atlantik_solar.xacro (robot description, xacro)
@@ -26,11 +26,11 @@
   <xacro:property name="mass_wheel" value="0.05" /> <!-- [kg] -->
   <xacro:property name="mass_front_wing" value="1.0" /> <!-- [kg] -->
-  <xacro:property name="mass_small_wing" value="${0.3 * mass_front_wing}" /> <!-- [kg] -->
-  <xacro:property name="mass_tail" value="0.5" /> <!-- [kg] -->
-  <xacro:property name="mass_rear_wing" value="0.2" /> <!-- [kg] -->
+  <xacro:property name="mass_small_wing" value="0.3" /> <!-- [kg] -->
+  <xacro:property name="mass_tail" value="0.25" /> <!-- [kg] -->
+  <xacro:property name="mass_rear_wing" value="0.25" /> <!-- [kg] -->
   <xacro:property name="mass_propeller" value="0.01" /> <!-- [kg] -->
-  <xacro:property name="mass_aileron" value="0.2" /> <!-- [kg] -->
-  <xacro:property name="mass_elevator" value="0.1" /> <!-- [kg] -->
-  <xacro:property name="mass_rudder" value="0.1" /> <!-- [kg] -->
+  <xacro:property name="mass_aileron" value="0.3" /> <!-- [kg] -->
+  <xacro:property name="mass_elevator" value="0.2" /> <!-- [kg] -->
+  <xacro:property name="mass_rudder" value="0.2" /> <!-- [kg] -->
   <!-- Fuselage properties -->
   <xacro:property name="body_length" value="3.0" /> <!-- [m] -->
@@ -57,5 +57,5 @@
   <xacro:property name="rear_wingspan" value="1.0" /> <!-- [m] -->
   <xacro:property name="rear_wing_height" value="0.02" /> <!-- [m] -->
-  <xacro:property name="alpha_0" value="0.0" /> <!-- [rad] -->
+  <xacro:property name="alpha_0" value="0.01" /> <!-- [rad] -->
   <xacro:property name="alpha_stall" value="0.2" /> <!-- [rad] -->
   <xacro:property name="c_L_alpha" value="3.0" />
@@ -109,5 +109,5 @@
   <!-- Inertia of a single small front wing, assuming it is a cuboid -->
   <xacro:property name="small_wing_inertia">
-    <xacro:box_inertia x="${aileron_length}" y="${front_wing_width - aileron_width}" z="${front_wing_height}" mass="${0.3 * mass_small_wing}" />
+    <xacro:box_inertia x="${aileron_length}" y="${front_wing_width - aileron_width}" z="${front_wing_height}" mass="${mass_small_wing}" />
   </xacro:property>
   <!-- Inertia of the tail, assuming it is a cuboid -->
@@ -149,3 +149,363 @@
     <xacro:insert_block name="body_inertia" />
   </xacro:fixed_wing_base_macro>
+  <!-- Instantiate the propeller -->
+  <xacro:propeller
+    robot_namespace="${namespace}"
+    direction="cw"
+    motor_constant="${motor_constant}"
+    moment_constant="${moment_constant}"
+    parent="${namespace}/base_link_inertia"
+    mass_propeller="${mass_propeller}"
+    radius_propeller="${radius_propeller}"
+    time_constant_up="${time_constant_up}"
+    time_constant_down="${time_constant_down}"
+    max_propeller_velocity="${max_propeller_velocity}"
+    motor_number="0"
+    rotor_drag_coefficient="${rotor_drag_coefficient}"
+    rolling_moment_coefficient="${rolling_moment_coefficient}"
+    color="Blue"
+    use_own_mesh="false"
+    mesh="">
+    <origin xyz="${0.5 * body_length + propeller_offset} 0.0 0.0" rpy="0.0 ${0.5 * PI} 0.0" />
+    <xacro:insert_block name="propeller_inertia" />
+  </xacro:propeller>
+  <!-- Instantiate wheels -->
+  <xacro:wheel
+    robot_namespace="${namespace}"
+    suffix="front_left"
+    parent="${namespace}/base_link_inertia"
+    mass_wheel="${mass_wheel}"
+    color="${body_color}"
+    use_mesh="false"
+    mesh=""
+    wheel_radius="${wheel_radius}"
+    wheel_width="${wheel_width}">
+    <origin xyz="0.75 0.1 -0.1" rpy="${0.5 * PI} 0.0 0.0" />
+    <xacro:insert_block name="wheel_inertia" />
+  </xacro:wheel>
+  <xacro:wheel
+    robot_namespace="${namespace}"
+    suffix="front_right"
+    parent="${namespace}/base_link_inertia"
+    mass_wheel="${mass_wheel}"
+    color="${body_color}"
+    use_mesh="false"
+    mesh=""
+    wheel_radius="${wheel_radius}"
+    wheel_width="${wheel_width}">
+    <origin xyz="0.75 -0.1 -0.1" rpy="${0.5 * PI} 0.0 0.0" />
+    <xacro:insert_block name="wheel_inertia" />
+  </xacro:wheel>
+  <xacro:wheel
+    robot_namespace="${namespace}"
+    suffix="back"
+    parent="${namespace}/base_link_inertia"
+    mass_wheel="${mass_wheel}"
+    color="${body_color}"
+    use_mesh="false"
+    mesh=""
+    wheel_radius="${wheel_radius}"
+    wheel_width="${wheel_width}">
+    <origin xyz="-1.0 0.0 -0.1" rpy="${0.5 * PI} 0.0 0.0" />
+    <xacro:insert_block name="wheel_inertia" />
+  </xacro:wheel>
+  <!-- Instantiate wings -->
+  <xacro:wing
+    robot_namespace="${namespace}"
+    suffix="left_big"
+    parent="${namespace}/base_link_inertia"
+    mass_wing="${mass_front_wing}"
+    wing_length="${root_chord}"
+    wing_width="${front_wing_width}"
+    wing_height="${front_wing_height}"
+    color="${body_color}"
+    use_mesh="false"
+    mesh=""
+    alpha_0="${alpha_0}"
+    alpha_stall="${alpha_stall}"
+    c_L_alpha="${c_L_alpha}"
+    air_density="${air_density}"
+    cp_x="0.0"
+    cp_y="${0.5 * front_wing_width}"
+    cp_z="0.0">
+    <origin xyz="0.5 ${0.5 * body_width} 0.0" rpy="0.0 0.0 0.0" />
+    <origin xyz="0.0 ${0.5 * front_wing_width} 0.0" rpy="0.0 0.0 0.0" />
+    <xacro:insert_block name="front_wing_inertia" />
+  </xacro:wing>-->
+  <xacro:wing
+    robot_namespace="${namespace}"
+    suffix="right_big"
+    parent="${namespace}/base_link_inertia"
+    mass_wing="${mass_front_wing}"
+    wing_length="${root_chord}"
+    wing_width="${front_wing_width}"
+    wing_height="${front_wing_height}"
+    color="${body_color}"
+    use_mesh="false"
+    mesh=""
+    alpha_0="${alpha_0}"
+    alpha_stall="${alpha_stall}"
+    c_L_alpha="${c_L_alpha}"
+    air_density="${air_density}"
+    cp_x="0.0"
+    cp_y="${-0.5 * front_wing_width}"
+    cp_z="0.0">
+    <origin xyz="0.5 ${-0.5 * body_width} 0.0" rpy="0.0 0.0 0.0" />
+    <origin xyz="0.0 ${-0.5 * front_wing_width} 0.0" rpy="0.0 0.0 0.0" />
+    <xacro:insert_block name="front_wing_inertia" />
+  </xacro:wing>
+  <xacro:wing
+    robot_namespace="${namespace}"
+    suffix="left_small"
+    parent="${namespace}/base_link_inertia"
+    mass_wing="${mass_small_wing}"
+    wing_length="${aileron_length}"
+    wing_width="${front_wing_width - aileron_width}"
+    wing_height="${front_wing_height}"
+    color="${body_color}"
+    use_mesh="false"
+    mesh=""
+    alpha_0="${alpha_0}"
+    alpha_stall="${alpha_stall}"
+    c_L_alpha="${c_L_alpha}"
+    air_density="${air_density}"
+    cp_x="0.0"
+    cp_y="${0.5 * (front_wing_width - aileron_width)}"
+    cp_z="0.0">
+    <origin xyz="${0.5 * (1 - root_chord - aileron_length)} ${0.5 * body_width} 0.0" rpy="0.0 0.0 0.0" />
+    <origin xyz="0.0 ${0.5 * (front_wing_width - aileron_width)} 0.0" rpy="0.0 0.0 0.0" />
+    <xacro:insert_block name="small_wing_inertia" />
+  </xacro:wing>
+  <xacro:wing
+    robot_namespace="${namespace}"
+    suffix="right_small"
+    parent="${namespace}/base_link_inertia"
+    mass_wing="${mass_small_wing}"
+    wing_length="${aileron_length}"
+    wing_width="${front_wing_width - aileron_width}"
+    wing_height="${front_wing_height}"
+    color="${body_color}"
+    use_mesh="false"
+    mesh=""
+    alpha_0="${alpha_0}"
+    alpha_stall="${alpha_stall}"
+    c_L_alpha="${c_L_alpha}"
+    air_density="${air_density}"
+    cp_x="0.0"
+    cp_y="${-0.5 * (front_wing_width - aileron_width)}"
+    cp_z="0.0">
+    <origin xyz="${0.5 * (1 - root_chord - aileron_length)} ${-0.5 * body_width} 0.0" rpy="0.0 0.0 0.0" />
+    <origin xyz="0.0 ${-0.5 * (front_wing_width - aileron_width)} 0.0" rpy="0.0 0.0 0.0" />
+    <xacro:insert_block name="small_wing_inertia" />
+  </xacro:wing>
+  <!-- Instantiate the tail -->
+  <xacro:tail
+    robot_namespace="${namespace}"
+    parent="${namespace}/base_link_inertia"
+    mass_tail="${mass_tail}"
+    tail_length="${tail_length}"
+    tail_width="${tail_width}"
+    tail_height="${tail_height}"
+    color="${body_color}"
+    use_mesh="false"
+    mesh="">
+    <origin xyz="${-0.5*body_length + 0.5*tail_length} 0.0 ${0.5*body_height + 0.5*tail_height}" rpy="0.0 0.0 0.0" />
+    <xacro:insert_block name="tail_inertia" />
+  </xacro:tail>
+  <!-- Instantiate the rear wings-->
+  <xacro:wing
+    robot_namespace="${namespace}"
+    suffix="rear_left"
+    parent="${namespace}/tail"
+    mass_wing="${mass_rear_wing}"
+    wing_length="${tail_length - elevator_length}"
+    wing_width="${rear_wing_width}"
+    wing_height="${rear_wing_height}"
+    color="${body_color}"
+    use_mesh="false"
+    mesh=""
+    alpha_0="${alpha_0}"
+    alpha_stall="${alpha_stall}"
+    c_L_alpha="${c_L_alpha}"
+    air_density="${air_density}"
+    cp_x="0.0"
+    cp_y="${0.5 * rear_wing_width}"
+    cp_z="0.0">
+    <origin xyz="${0.5 * elevator_length} ${0.5 * tail_width} ${0.5 * (tail_height - rear_wing_height)}" rpy="0.0 0.0 0.0" />
+    <origin xyz="0.0 ${0.5 * rear_wing_width} 0.0" rpy="0.0 0.0 0.0" />
+    <xacro:insert_block name="rear_wing_inertia" />
+  </xacro:wing>
+  <xacro:wing
+    robot_namespace="${namespace}"
+    suffix="rear_right"
+    parent="${namespace}/tail"
+    mass_wing="${mass_rear_wing}"
+    wing_length="${tail_length - elevator_length}"
+    wing_width="${rear_wing_width}"
+    wing_height="${rear_wing_height}"
+    color="${body_color}"
+    use_mesh="false"
+    mesh=""
+    alpha_0="${alpha_0}"
+    alpha_stall="${alpha_stall}"
+    c_L_alpha="${c_L_alpha}"
+    air_density="${air_density}"
+    cp_x="0.0"
+    cp_y="${-0.5 * rear_wing_width}"
+    cp_z="0.0">
+    <origin xyz="${0.5 * elevator_length} ${-0.5 * tail_width} ${0.5 * (tail_height - rear_wing_height)}" rpy="0.0 0.0 0.0" />
+    <origin xyz="0.0 ${-0.5 * rear_wing_width} 0.0" rpy="0.0 0.0 0.0" />
+    <xacro:insert_block name="rear_wing_inertia" />
+  </xacro:wing>
+  <!-- Instantiate the control surfaces -->
+  <xacro:control_surface
+    robot_namespace="${namespace}"
+    surface_name="aileron_left"
+    parent="${namespace}/wing_left_big"
+    mass_surface="${mass_aileron}"
+    velocity_gain="${aileron_velocity_gain}"
+    positive_direction="ccw"
+    min_angle="${aileron_min_angle}"
+    max_angle="${aileron_max_angle}"
+    channel="${aileron_channel}"
+    color="Orange"
+    use_mesh="false"
+    mesh=""
+    surface_length="${aileron_length}"
+    surface_width="${aileron_width}"
+    surface_height="${aileron_height}"
+    area="${aileron_length * aileron_width}"
+    forward_x="1"
+    forward_y="0"
+    forward_z="0"
+    up_x="0"
+    up_y="0"
+    up_z="1"
+    c_L_alpha="${c_L_alpha}"
+    alpha_stall="${alpha_stall}">
+    <axis xyz="0 1 0" />
+    <origin xyz="${-0.5 * root_chord} ${front_wing_width - 0.5 * aileron_width} 0.0" rpy="0.0 0.0 0.0" />
+    <origin xyz="${-0.5 * aileron_length} 0.0 0.0" rpy="0.0 0.0 0.0" />
+    <xacro:insert_block name="aileron_inertia" />
+  </xacro:control_surface>
+  <xacro:control_surface
+    robot_namespace="${namespace}"
+    surface_name="aileron_right"
+    parent="${namespace}/wing_right_big"
+    mass_surface="${mass_aileron}"
+    velocity_gain="${aileron_velocity_gain}"
+    positive_direction="cw"
+    min_angle="${aileron_min_angle}"
+    max_angle="${aileron_max_angle}"
+    channel="${aileron_channel}"
+    color="Orange"
+    use_mesh="false"
+    mesh=""
+    surface_length="${aileron_length}"
+    surface_width="${aileron_width}"
+    surface_height="${aileron_height}"
+    area="${aileron_length * aileron_width}"
+    forward_x="1"
+    forward_y="0"
+    forward_z="0"
+    up_x="0"
+    up_y="0"
+    up_z="1"
+    c_L_alpha="${c_L_alpha}"
+    alpha_stall="${alpha_stall}">
+    <axis xyz="0 1 0" />
+    <origin xyz="${-0.5 * root_chord} ${-(front_wing_width - 0.5 * aileron_width)} 0.0" rpy="0.0 0.0 0.0" />
+    <origin xyz="${-0.5 * aileron_length} 0.0 0.0" rpy="0.0 0.0 0.0" />
+    <xacro:insert_block name="aileron_inertia" />
+  </xacro:control_surface>
+  <xacro:control_surface
+    robot_namespace="${namespace}"
+    surface_name="elevator_left"
+    parent="${namespace}/wing_rear_left"
+    mass_surface="${mass_elevator}"
+    velocity_gain="${elevator_velocity_gain}"
+    positive_direction="ccw"
+    min_angle="${elevator_min_angle}"
+    max_angle="${elevator_max_angle}"
+    channel="${elevator_channel}"
+    color="Blue"
+    use_mesh="false"
+    mesh=""
+    surface_length="${elevator_length}"
+    surface_width="${elevator_width}"
+    surface_height="${elevator_height}"
+    area="${elevator_length * elevator_width}"
+    forward_x="1"
+    forward_y="0"
+    forward_z="0"
+    up_x="0"
+    up_y="0"
+    up_z="1"
+    c_L_alpha="${c_L_alpha}"
+    alpha_stall="${alpha_stall}">
+    <axis xyz="0 1 0" />
+    <origin xyz="${-0.5 * (tail_length - elevator_length)} ${0.5 * rear_wing_width} 0.0" rpy="0.0 0.0 0.0" />
+    <origin xyz="${-0.5 * elevator_length} 0.0 0.0" rpy="0.0 0.0 0.0" />
+    <xacro:insert_block name="elevator_inertia" />
+  </xacro:control_surface>
+  <xacro:control_surface
+    robot_namespace="${namespace}"
+    surface_name="elevator_right"
+    parent="${namespace}/wing_rear_right"
+    mass_surface="${mass_elevator}"
+    velocity_gain="${elevator_velocity_gain}"
+    positive_direction="ccw"
+    min_angle="${elevator_min_angle}"
+    max_angle="${elevator_max_angle}"
+    channel="${elevator_channel}"
+    color="Blue"
+    use_mesh="false"
+    mesh=""
+    surface_length="${elevator_length}"
+    surface_width="${elevator_width}"
+    surface_height="${elevator_height}"
+    area="${elevator_length * elevator_width}"
+    forward_x="1"
+    forward_y="0"
+    forward_z="0"
+    up_x="0"
+    up_y="0"
+    up_z="1"
+    c_L_alpha="${c_L_alpha}"
+    alpha_stall="${alpha_stall}">
+    <axis xyz="0 1 0" />
+    <origin xyz="${-0.5 * (tail_length - elevator_length)} ${-0.5 * rear_wing_width} 0.0" rpy="0.0 0.0 0.0" />
+    <origin xyz="${-0.5 * elevator_length} 0.0 0.0" rpy="0.0 0.0 0.0" />
+    <xacro:insert_block name="elevator_inertia" />
+  </xacro:control_surface>
+  <xacro:control_surface
+    robot_namespace="${namespace}"
+    surface_name="rudder"
+    parent="${namespace}/tail"
+    mass_surface="${mass_rudder}"
+    velocity_gain="${rudder_velocity_gain}"
+    positive_direction="cw"
+    min_angle="${rudder_min_angle}"
+    max_angle="${rudder_max_angle}"
+    channel="${rudder_channel}"
+    color="Gray"
+    use_mesh="false"
+    mesh=""
+    surface_length="${rudder_length}"
+    surface_width="${rudder_width}"
+    surface_height="${rudder_height}"
+    area="0.0"
+    forward_x="0"
+    forward_y="0"
+    forward_z="0"
+    up_x="0"
+    up_y="0"
+    up_z="0"
+    c_L_alpha="0.0"
+    alpha_stall="0.0">
+    <axis xyz="0 0 1" />
+    <origin xyz="${-0.5 * tail_length} 0.0 0.0" rpy="0.0 0.0 0.0" />
+    <origin xyz="${-0.5 * rudder_length} 0.0 0.0" rpy="0.0 0.0 0.0" />
+    <xacro:insert_block name="rudder_inertia" />
+  </xacro:control_surface>
 </robot>

File: rotors_description/urdf/atlantik_solar_base.xacro (robot description, xacro)
@@ -23,43 +23,13 @@
   <xacro:controller_plugin_macro namespace="${namespace}" imu_sub_topic="imu" />
   <!-- Mount an ADIS16448 IMU. -->
-  <xacro:default_imu namespace="${namespace}" parent_link="${namespace}/base_link" />
+  <xacro:default_imu namespace="${namespace}" parent_link="${namespace}/base_link_inertia" />
   <!-- Mount a GPS. -->
-  <xacro:default_gps namespace="${namespace}" parent_link="${namespace}/base_link" />
+  <xacro:default_gps namespace="${namespace}" parent_link="${namespace}/base_link_inertia" />
   <!-- Mount a magnetometer. -->
-  <xacro:default_magnetometer namespace="${namespace}" parent_link="${namespace}/base_link" />
+  <xacro:default_magnetometer namespace="${namespace}" parent_link="${namespace}/base_link_inertia" />
   <!-- Mount a pressure sensor. -->
-  <xacro:default_pressure_sensor namespace="${namespace}" parent_link="${namespace}/base_link" />
-  <!-- Mount a generic odometry sensor without odometry map (working everywhere). -->
-  <xacro:odometry_plugin_macro
-    namespace="${namespace}"
-    odometry_sensor_suffix=""
-    parent_link="${namespace}/base_link"
-    pose_topic="pose"
-    pose_with_covariance_topic="pose_with_covariance"
-    position_topic="position"
-    transform_topic="transform"
-    odometry_topic="odometry"
-    parent_frame_id="world"
-    child_frame_id="${namespace}/odometry_sensor"
-    mass_odometry_sensor="0.00001"
-    measurement_divisor="1"
-    measurement_delay="0"
-    unknown_delay="0.0"
-    noise_normal_position="0 0 0"
-    noise_normal_quaternion="0 0 0"
-    noise_normal_linear_velocity="0 0 0"
-    noise_normal_angular_velocity="0 0 0"
-    noise_uniform_position="0 0 0"
-    noise_uniform_quaternion="0 0 0"
-    noise_uniform_linear_velocity="0 0 0"
-    noise_uniform_angular_velocity="0 0 0"
-    enable_odometry_map="false"
-    odometry_map=""
-    image_scale="">
-    <inertia ixx="0.00001" ixy="0.0" ixz="0.0" iyy="0.00001" iyz="0.0" izz="0.00001" /> <!-- [kg m^2] [kg m^2] [kg m^2] [kg m^2] [kg m^2] [kg m^2] -->
-    <origin xyz="0.0 0.0 0.0" rpy="0.0 0.0 0.0" />
-  </xacro:odometry_plugin_macro>
+  <xacro:default_pressure_sensor namespace="${namespace}" parent_link="${namespace}/base_link_inertia" />
   <xacro:if value="$(arg enable_ground_truth)">
-    <xacro:ground_truth_imu_and_odometry namespace="${namespace}" parent_link="${namespace}/base_link" />
+    <xacro:ground_truth_imu_and_odometry namespace="${namespace}" parent_link="${namespace}/base_link_inertia" />
   </xacro:if>
   <xacro:if value="$(arg enable_logging)">

File: rotors_description/urdf/component_snippets.xacro (robot description, xacro)
@@ -302,4 +302,5 @@
         <xacro:insert_block name="inertia" />
         <mass value="${mass_odometry_sensor}" />  <!-- [kg] -->
+        <origin xyz="0 0 0" rpy="0 0 0" />
       </inertial>
     </link>
@@ -678,5 +679,5 @@
       parent_link="${parent_link}"
       imu_topic="ground_truth/imu"
-      mass_imu_sensor="0.00001"
+      mass_imu_sensor="0.015"
       gyroscope_noise_density="0.0"
       gyroscopoe_random_walk="0.0"
@@ -702,5 +703,5 @@
       parent_frame_id="world"
       child_frame_id="${namespace}/base_link"
-      mass_odometry_sensor="0.00001"
+      mass_odometry_sensor="0.015"
       measurement_divisor="1"
       measurement_delay="0"
