Commit message: Fixing some moments of inertia

File: rotors_description/urdf/fixed_wing_base.xacro (robot description, xacro)
@@ -29,12 +29,4 @@
       izz="${0.5 * mass * r * r}" />
   </xacro:macro>
-  <!-- Macro for the inertial properties of a box -->
-  <xacro:macro name="box_inertial" params="x y z mass *origin">
-    <inertial>
-      <mass value="${mass}" />
-      <xacro:insert_block name="origin" />
-      <xacro:box_inertia x="${x}" y="${y}" z="${z}" mass="${mass}" />
-    </inertial>
-  </xacro:macro>
   <!-- Fixed-wing fuselage link -->
   <xacro:macro name="fixed_wing_base_macro"
@@ -50,5 +42,5 @@
       <inertial>
         <mass value="${mass}" />  <!-- [kg] -->
-        <origin xyz="0 0 0" />
+        <origin xyz="0.7 0 0" rpy="0 0 0" />
         <xacro:insert_block name="inertia" />
       </inertial>
@@ -85,5 +77,5 @@
     params="robot_namespace suffix parent mass_wheel color use_mesh mesh
       wheel_radius wheel_width *origin *inertia">
-    <joint name="${robot_namespace}/wheel_${suffix}_joint" type="revolute">
+    <joint name="${robot_namespace}/wheel_${suffix}_joint" type="fixed">
       <xacro:insert_block name="origin" />
       <axis xyz="0 1 0" />
@@ -94,4 +86,5 @@
     <link name="${robot_namespace}/wheel_${suffix}">
       <inertial>
+        <origin xyz="0.0 0.0 0.0" rpy="0.0 0.0 0.0" />
         <mass value="${mass_wheel}" /> <!-- [kg] -->
         <xacro:insert_block name="inertia" />
@@ -121,7 +114,8 @@
   <xacro:macro name="wing"
     params="robot_namespace suffix parent mass_wing wing_length wing_width wing_height
-      color use_mesh mesh alpha_0 alpha_stall c_L_alpha air_density *origin *inertia">
+      color use_mesh mesh alpha_0 alpha_stall c_L_alpha air_density cp_x cp_y cp_z *joint_origin
+      *link_origin *inertia">
     <joint name="${robot_namespace}/wing_${suffix}_joint" type="revolute">
-      <xacro:insert_block name="origin" />
+      <xacro:insert_block name="joint_origin" />
       <axis xyz="1 0 0" />
       <parent link="${parent}" />
@@ -131,10 +125,10 @@
     <link name="${robot_namespace}/wing_${suffix}">
       <inertial>
-        <origin xyz="0 0 0" rpy="0 0 0" />
+        <xacro:insert_block name="link_origin" />
         <mass value="${mass_wing}" /> <!-- [kg] -->
         <xacro:insert_block name="inertia" />
       </inertial>
       <visual>
-        <origin xyz="0 0 0" rpy="0 0 0" />
+        <xacro:insert_block name="link_origin" />
         <geometry>
           <xacro:if value="${use_mesh}">
@@ -148,7 +142,7 @@
       </visual>
       <collision>
-        <origin xyz="0 0 0" rpy="0 0 0" />
-        <geometry>
-          <box size="${wing_length} ${wing_width} ${wing_height}"/> <!-- [m] [m] [m] -->
+        <xacro:insert_block name="link_origin" />
+        <geometry>
+          <box size="${wing_length - 0.01} ${wing_width - 0.01} ${wing_height - 0.01}"/> <!-- [m] [m] [m] -->
         </geometry>
       </collision>
@@ -156,4 +150,5 @@
     <gazebo>
       <plugin name="${robot_namespace}_${suffix}_lift_drag" filename="libLiftDragPlugin.so">
+      <!--<plugin name="${robot_namespace}_${suffix}_lift_drag" filename="librotors_gazebo_lift_drag_plugin.so">-->
         <a0>${alpha_0}</a0>
         <cla>${c_L_alpha}</cla>
@@ -164,5 +159,5 @@
         <cda_stall>0.1</cda_stall>
         <cma_stall>-0.2</cma_stall>
-        <cp>0.0 0.0 0.0</cp>
+        <cp>${cp_x} ${cp_y} ${cp_z}</cp>
         <area>${wing_length * wing_width}</area>
         <air_density>${air_density}</air_density>
@@ -189,4 +184,5 @@
     <link name="${robot_namespace}/tail">
       <inertial>
+        <origin xyz="0.0 0.0 0.0" rpy="0.0 0.0 0.0" />
         <mass value="${mass_tail}" /> <!-- [kg] -->
         <xacro:insert_block name="inertia" />
@@ -210,59 +206,4 @@
     </link>
     <gazebo reference="${robot_namespace}/tail">
-      <material>Gazebo/${color}</material>
-    </gazebo>
-  </xacro:macro>
-  <!-- Rear wing joint and link -->
-  <xacro:macro name="rear_wing"
-    params="robot_namespace suffix parent mass_rear_wing rear_wing_length rear_wing_width
-      rear_wing_height color use_mesh mesh alpha_0 alpha_stall c_L_alpha air_density *origin *inertia">
-    <joint name="${robot_namespace}/rear_wing_${suffix}_joint" type="revolute">
-      <xacro:insert_block name="origin" />
-      <axis xyz="0 0 1" />
-      <parent link="${parent}" />
-      <child link="${robot_namespace}/rear_wing_${suffix}" />
-      <limit upper="0" lower="0" effort="0" velocity="0" />
-    </joint>
-    <link name="${robot_namespace}/rear_wing_${suffix}">
-      <inertial>
-        <mass value="${mass_rear_wing}" /> <!-- [kg] -->
-        <xacro:insert_block name="inertia" />
-      </inertial>
-      <visual>
-        <geometry>
-          <xacro:if value="${use_mesh}">
-            <mesh filename="${mesh}"
-              scale="1 1 1" />
-          </xacro:if>
-          <xacro:unless value="${use_mesh}">
-            <box size="${rear_wing_length} ${rear_wing_width} ${rear_wing_height}"/> <!-- [m] [m] [m] -->
-          </xacro:unless>
-        </geometry>
-      </visual>
-      <collision>
-        <geometry>
-          <box size="${rear_wing_length} ${rear_wing_width} ${rear_wing_height}"/> <!-- [m] [m] [m] -->
-        </geometry>
-      </collision>
-    </link>
-    <gazebo>
-      <plugin name="${robot_namespace}_${suffix}_rear_lift_drag" filename="libLiftDragPlugin.so">
-        <a0>${alpha_0}</a0>
-        <cla>${c_L_alpha}</cla>
-        <cda>0.1</cda>
-        <cma>-0.1</cma>
-        <alpha_stall>${alpha_stall}</alpha_stall>
-        <cla_stall>-0.1</cla_stall>
-        <cda_stall>0.1</cda_stall>
-        <cma_stall>-0.2</cma_stall>
-        <cp>0.0 0.0 0.0</cp>
-        <area>${rear_wing_length * rear_wing_width}</area>
-        <air_density>${air_density}</air_density>
-        <forward>1 0 0</forward>
-        <upward>0 0 1</upward>
-        <link_name>${robot_namespace}/rear_wing_${suffix}</link_name>
-      </plugin>
-    </gazebo>
-    <gazebo reference="${robot_namespace}/rear_wing_${suffix}">
       <material>Gazebo/${color}</material>
     </gazebo>
@@ -281,4 +222,5 @@
     <link name="${robot_namespace}/propeller">
       <inertial>
+        <origin xyz="0.0 0.0 0.0" rpy="0.0 0.0 0.0" />
         <mass value="${mass_propeller}" /> <!-- [kg] -->
         <xacro:insert_block name="inertia" />
@@ -330,5 +272,6 @@
       positive_direction min_angle max_angle channel color use_mesh mesh
       surface_length surface_width surface_height area forward_x forward_y
-      forward_z up_x up_y up_z c_L_alpha alpha_stall *axis *joint_origin *link_origin *inertia">
+      forward_z up_x up_y up_z c_L_alpha alpha_stall *axis *joint_origin
+      *link_origin *inertia">
     <joint name="${robot_namespace}/${surface_name}_joint" type="revolute">
       <xacro:insert_block name="joint_origin" />
@@ -336,5 +279,6 @@
       <parent link="${parent}" />
       <child link="${robot_namespace}/${surface_name}" />
-      <limit upper="${max_angle}" lower="${min_angle}" effort="100.0" velocity="3.0" />
+      <limit upper="${max_angle}" lower="${min_angle}" effort="200.0" velocity="3.0" />
+      <dynamics friction="${9.8 * mass_surface}" damping="${9.8 * mass_surface}" />
     </joint>
     <link name="${robot_namespace}/${surface_name}">
@@ -360,5 +304,5 @@
         <xacro:insert_block name="link_origin" />
         <geometry>
-          <box size="${surface_length} ${surface_width} ${surface_height}"/> <!-- [m] [m] [m] -->
+          <box size="${surface_length - 0.01} ${surface_width - 0.01} ${surface_height - 0.01}"/> <!-- [m] [m] [m] -->
         </geometry>
       </collision>
@@ -377,5 +321,5 @@
       </plugin>
     </gazebo>
-    <gazebo>
+<!--    <gazebo>
       <plugin name="${robot_namespace}_${surface_name}_lift_drag" filename="libLiftDragPlugin.so">
         <a0>0.0</a0>
@@ -394,5 +338,5 @@
         <link_name>${robot_namespace}/${surface_name}</link_name>
       </plugin>
-    </gazebo>
+    </gazebo>-->
     <gazebo reference="${robot_namespace}/${surface_name}">
       <material>Gazebo/${color}</material>

Commit message: Starting to implement combined aerodynamics model

File: rotors_description/urdf/atlantik_solar.xacro (robot description, xacro)
@@ -69,5 +69,5 @@
   <xacro:property name="aileron_width" value="${0.5 * front_wing_width}" /> <!-- [m] -->
   <xacro:property name="aileron_height" value="0.02" /> <!-- [m] -->
-  <xacro:property name="aileron_velocity_gain" value="1.0" />
+  <xacro:property name="aileron_gain" value="2.0" />
   <xacro:property name="aileron_min_angle" value="-0.55" /> <!-- [rad] -->
   <xacro:property name="aileron_max_angle" value="0.55" /> <!-- [rad] -->
@@ -77,5 +77,5 @@
   <xacro:property name="elevator_width" value="${rear_wing_width}" /> <!-- [m] -->
   <xacro:property name="elevator_height" value="0.02" /> <!-- [m] -->
-  <xacro:property name="elevator_velocity_gain" value="1.0" />
+  <xacro:property name="elevator_gain" value="2.0" />
   <xacro:property name="elevator_min_angle" value="-0.55" /> <!-- [rad] -->
   <xacro:property name="elevator_max_angle" value="0.55" /> <!-- [rad] -->
@@ -85,5 +85,5 @@
   <xacro:property name="rudder_width" value="${tail_width}" /> <!-- [m] -->
   <xacro:property name="rudder_height" value="${tail_height}" /> <!-- [m] -->
-  <xacro:property name="rudder_velocity_gain" value="1.0" />
+  <xacro:property name="rudder_gain" value="2.0" />
   <xacro:property name="rudder_min_angle" value="-0.55" /> <!-- [rad] -->
   <xacro:property name="rudder_max_angle" value="0.55" /> <!-- [rad] -->
@@ -95,4 +95,8 @@
   <!-- Rear wing length -->
   <xacro:property name="rear_wing_width" value="${0.5 * (rear_wingspan - tail_width)}" />
+  <!-- Total area of the wings -->
+  <xacro:property name="total_wing_area"
+    value="${2.0 * (front_wing_width * root_chord + (front_wing_width - aileron_width) * aileron_length)}" >
+  </xacro:property>
   <!-- Inertia of the fuselage -->
   <xacro:property name="body_inertia">
@@ -146,5 +150,9 @@
     color="${body_color}"
     use_mesh_file="${use_mesh_file}"
-    mesh_file="${mesh_file}">
+    mesh_file="${mesh_file}"
+    reset_topic="reset"
+    total_wing_area="${total_wing_area}"
+    air_density="${air_density}"
+    alpha_stall="${alpha_stall}">
     <xacro:insert_block name="body_inertia" />
   </xacro:fixed_wing_base_macro>
@@ -221,12 +229,5 @@
     color="${body_color}"
     use_mesh="false"
-    mesh=""
-    alpha_0="${alpha_0}"
-    alpha_stall="${alpha_stall}"
-    c_L_alpha="${c_L_alpha}"
-    air_density="${air_density}"
-    cp_x="0.0"
-    cp_y="${0.5 * front_wing_width}"
-    cp_z="0.0">
+    mesh="">
     <origin xyz="0.5 ${0.5 * body_width} 0.0" rpy="0.0 0.0 0.0" />
     <origin xyz="0.0 ${0.5 * front_wing_width} 0.0" rpy="0.0 0.0 0.0" />
@@ -243,12 +244,5 @@
     color="${body_color}"
     use_mesh="false"
-    mesh=""
-    alpha_0="${alpha_0}"
-    alpha_stall="${alpha_stall}"
-    c_L_alpha="${c_L_alpha}"
-    air_density="${air_density}"
-    cp_x="0.0"
-    cp_y="${-0.5 * front_wing_width}"
-    cp_z="0.0">
+    mesh="">
     <origin xyz="0.5 ${-0.5 * body_width} 0.0" rpy="0.0 0.0 0.0" />
     <origin xyz="0.0 ${-0.5 * front_wing_width} 0.0" rpy="0.0 0.0 0.0" />
@@ -265,12 +259,5 @@
     color="${body_color}"
     use_mesh="false"
-    mesh=""
-    alpha_0="${alpha_0}"
-    alpha_stall="${alpha_stall}"
-    c_L_alpha="${c_L_alpha}"
-    air_density="${air_density}"
-    cp_x="0.0"
-    cp_y="${0.5 * (front_wing_width - aileron_width)}"
-    cp_z="0.0">
+    mesh="">
     <origin xyz="${0.5 * (1 - root_chord - aileron_length)} ${0.5 * body_width} 0.0" rpy="0.0 0.0 0.0" />
     <origin xyz="0.0 ${0.5 * (front_wing_width - aileron_width)} 0.0" rpy="0.0 0.0 0.0" />
@@ -287,12 +274,5 @@
     color="${body_color}"
     use_mesh="false"
-    mesh=""
-    alpha_0="${alpha_0}"
-    alpha_stall="${alpha_stall}"
-    c_L_alpha="${c_L_alpha}"
-    air_density="${air_density}"
-    cp_x="0.0"
-    cp_y="${-0.5 * (front_wing_width - aileron_width)}"
-    cp_z="0.0">
+    mesh="">
     <origin xyz="${0.5 * (1 - root_chord - aileron_length)} ${-0.5 * body_width} 0.0" rpy="0.0 0.0 0.0" />
     <origin xyz="0.0 ${-0.5 * (front_wing_width - aileron_width)} 0.0" rpy="0.0 0.0 0.0" />
@@ -324,12 +304,5 @@
     color="${body_color}"
     use_mesh="false"
-    mesh=""
-    alpha_0="${alpha_0}"
-    alpha_stall="${alpha_stall}"
-    c_L_alpha="${c_L_alpha}"
-    air_density="${air_density}"
-    cp_x="0.0"
-    cp_y="${0.5 * rear_wing_width}"
-    cp_z="0.0">
+    mesh="">
     <origin xyz="${0.5 * elevator_length} ${0.5 * tail_width} ${0.5 * (tail_height - rear_wing_height)}" rpy="0.0 0.0 0.0" />
     <origin xyz="0.0 ${0.5 * rear_wing_width} 0.0" rpy="0.0 0.0 0.0" />
@@ -346,12 +319,5 @@
     color="${body_color}"
     use_mesh="false"
-    mesh=""
-    alpha_0="${alpha_0}"
-    alpha_stall="${alpha_stall}"
-    c_L_alpha="${c_L_alpha}"
-    air_density="${air_density}"
-    cp_x="0.0"
-    cp_y="${-0.5 * rear_wing_width}"
-    cp_z="0.0">
+    mesh="">
     <origin xyz="${0.5 * elevator_length} ${-0.5 * tail_width} ${0.5 * (tail_height - rear_wing_height)}" rpy="0.0 0.0 0.0" />
     <origin xyz="0.0 ${-0.5 * rear_wing_width} 0.0" rpy="0.0 0.0 0.0" />
@@ -364,5 +330,5 @@
     parent="${namespace}/wing_left_big"
     mass_surface="${mass_aileron}"
-    velocity_gain="${aileron_velocity_gain}"
+    gain="${aileron_gain}"
     positive_direction="ccw"
     min_angle="${aileron_min_angle}"
@@ -374,14 +340,5 @@
     surface_length="${aileron_length}"
     surface_width="${aileron_width}"
-    surface_height="${aileron_height}"
-    area="${aileron_length * aileron_width}"
-    forward_x="1"
-    forward_y="0"
-    forward_z="0"
-    up_x="0"
-    up_y="0"
-    up_z="1"
-    c_L_alpha="${c_L_alpha}"
-    alpha_stall="${alpha_stall}">
+    surface_height="${aileron_height}">
     <axis xyz="0 1 0" />
     <origin xyz="${-0.5 * root_chord} ${front_wing_width - 0.5 * aileron_width} 0.0" rpy="0.0 0.0 0.0" />
@@ -394,5 +351,5 @@
     parent="${namespace}/wing_right_big"
     mass_surface="${mass_aileron}"
-    velocity_gain="${aileron_velocity_gain}"
+    gain="${aileron_gain}"
     positive_direction="cw"
     min_angle="${aileron_min_angle}"
@@ -404,14 +361,5 @@
     surface_length="${aileron_length}"
     surface_width="${aileron_width}"
-    surface_height="${aileron_height}"
-    area="${aileron_length * aileron_width}"
-    forward_x="1"
-    forward_y="0"
-    forward_z="0"
-    up_x="0"
-    up_y="0"
-    up_z="1"
-    c_L_alpha="${c_L_alpha}"
-    alpha_stall="${alpha_stall}">
+    surface_height="${aileron_height}">
     <axis xyz="0 1 0" />
     <origin xyz="${-0.5 * root_chord} ${-(front_wing_width - 0.5 * aileron_width)} 0.0" rpy="0.0 0.0 0.0" />
@@ -424,5 +372,5 @@
     parent="${namespace}/wing_rear_left"
     mass_surface="${mass_elevator}"
-    velocity_gain="${elevator_velocity_gain}"
+    gain="${elevator_gain}"
     positive_direction="ccw"
     min_angle="${elevator_min_angle}"
@@ -434,14 +382,5 @@
     surface_length="${elevator_length}"
     surface_width="${elevator_width}"
-    surface_height="${elevator_height}"
-    area="${elevator_length * elevator_width}"
-    forward_x="1"
-    forward_y="0"
-    forward_z="0"
-    up_x="0"
-    up_y="0"
-    up_z="1"
-    c_L_alpha="${c_L_alpha}"
-    alpha_stall="${alpha_stall}">
+    surface_height="${elevator_height}">
     <axis xyz="0 1 0" />
     <origin xyz="${-0.5 * (tail_length - elevator_length)} ${0.5 * rear_wing_width} 0.0" rpy="0.0 0.0 0.0" />
@@ -454,5 +393,5 @@
     parent="${namespace}/wing_rear_right"
     mass_surface="${mass_elevator}"
-    velocity_gain="${elevator_velocity_gain}"
+    gain="${elevator_gain}"
     positive_direction="ccw"
     min_angle="${elevator_min_angle}"
@@ -464,14 +403,5 @@
     surface_length="${elevator_length}"
     surface_width="${elevator_width}"
-    surface_height="${elevator_height}"
-    area="${elevator_length * elevator_width}"
-    forward_x="1"
-    forward_y="0"
-    forward_z="0"
-    up_x="0"
-    up_y="0"
-    up_z="1"
-    c_L_alpha="${c_L_alpha}"
-    alpha_stall="${alpha_stall}">
+    surface_height="${elevator_height}">
     <axis xyz="0 1 0" />
     <origin xyz="${-0.5 * (tail_length - elevator_length)} ${-0.5 * rear_wing_width} 0.0" rpy="0.0 0.0 0.0" />
@@ -484,5 +414,5 @@
     parent="${namespace}/tail"
     mass_surface="${mass_rudder}"
-    velocity_gain="${rudder_velocity_gain}"
+    gain="${rudder_gain}"
     positive_direction="cw"
     min_angle="${rudder_min_angle}"
@@ -494,14 +424,5 @@
     surface_length="${rudder_length}"
     surface_width="${rudder_width}"
-    surface_height="${rudder_height}"
-    area="0.0"
-    forward_x="0"
-    forward_y="0"
-    forward_z="0"
-    up_x="0"
-    up_y="0"
-    up_z="0"
-    c_L_alpha="0.0"
-    alpha_stall="0.0">
+    surface_height="${rudder_height}">
     <axis xyz="0 0 1" />
     <origin xyz="${-0.5 * tail_length} 0.0 0.0" rpy="0.0 0.0 0.0" />

File: rotors_description/urdf/fixed_wing_base.xacro (robot description, xacro)
@@ -31,6 +31,7 @@
   <!-- Fixed-wing fuselage link -->
   <xacro:macro name="fixed_wing_base_macro"
-    params="robot_namespace mass body_length body_width body_height
-      color use_mesh_file mesh_file *inertia">
+    params="robot_namespace mass body_length body_width body_height color
+      use_mesh_file mesh_file reset_topic total_wing_area air_density
+      alpha_stall *inertia">
     <link name="${robot_namespace}/base_link"></link>
     <joint name="${robot_namespace}/base_joint" type="fixed">
@@ -67,4 +68,8 @@
         <robotNamespace>${robot_namespace}</robotNamespace>
         <linkName>${robot_namespace}/base_link</linkName>
+	<totalWingArea>${total_wing_area}</totalWingArea>
+	<resetTopic>${reset_topic}</resetTopic>
+	<airDensity>${air_density}</airDensity>
+	<alphaStall>${alpha_stall}</alphaStall>
       </plugin>
     </gazebo>
@@ -114,6 +119,5 @@
   <xacro:macro name="wing"
     params="robot_namespace suffix parent mass_wing wing_length wing_width wing_height
-      color use_mesh mesh alpha_0 alpha_stall c_L_alpha air_density cp_x cp_y cp_z *joint_origin
-      *link_origin *inertia">
+      color use_mesh mesh *joint_origin *link_origin *inertia">
     <joint name="${robot_namespace}/wing_${suffix}_joint" type="revolute">
       <xacro:insert_block name="joint_origin" />
@@ -148,23 +152,4 @@
       </collision>
     </link>
-    <gazebo>
-      <plugin name="${robot_namespace}_${suffix}_lift_drag" filename="libLiftDragPlugin.so">
-      <!--<plugin name="${robot_namespace}_${suffix}_lift_drag" filename="librotors_gazebo_lift_drag_plugin.so">-->
-        <a0>${alpha_0}</a0>
-        <cla>${c_L_alpha}</cla>
-        <cda>0.1</cda>
-        <cma>-0.1</cma>
-        <alpha_stall>${alpha_stall}</alpha_stall>
-        <cla_stall>-0.1</cla_stall>
-        <cda_stall>0.1</cda_stall>
-        <cma_stall>-0.2</cma_stall>
-        <cp>${cp_x} ${cp_y} ${cp_z}</cp>
-        <area>${wing_length * wing_width}</area>
-        <air_density>${air_density}</air_density>
-        <forward>1 0 0</forward>
-        <upward>0 0 1</upward>
-        <link_name>${robot_namespace}/wing_${suffix}</link_name>
-      </plugin>
-    </gazebo>
     <gazebo reference="${robot_namespace}/wing_${suffix}">
       <material>Gazebo/${color}</material>
@@ -269,8 +254,7 @@
   <!-- Control surface joint and link -->
   <xacro:macro name="control_surface"
-    params="robot_namespace surface_name parent mass_surface velocity_gain
+    params="robot_namespace surface_name parent mass_surface gain
       positive_direction min_angle max_angle channel color use_mesh mesh
-      surface_length surface_width surface_height area forward_x forward_y
-      forward_z up_x up_y up_z c_L_alpha alpha_stall *axis *joint_origin
+      surface_length surface_width surface_height *axis *joint_origin
       *link_origin *inertia">
     <joint name="${robot_namespace}/${surface_name}_joint" type="revolute">
@@ -315,5 +299,5 @@
         <commandSubTopic>gazebo/command/motor_speed</commandSubTopic>
         <positiveDirection>${positive_direction}</positiveDirection>
-        <velocityGain>${velocity_gain}</velocityGain>
+        <gain>${gain}</gain>
         <minAngle>${min_angle}</minAngle>
         <maxAngle>${max_angle}</maxAngle>
@@ -321,22 +305,4 @@
       </plugin>
     </gazebo>
-<!--    <gazebo>
-      <plugin name="${robot_namespace}_${surface_name}_lift_drag" filename="libLiftDragPlugin.so">
-        <a0>0.0</a0>
-        <cla>${c_L_alpha}</cla>
-        <cda>0.1</cda>
-        <cma>-0.1</cma>
-        <alpha_stall>${alpha_stall}</alpha_stall>
-        <cla_stall>-0.1</cla_stall>
-        <cda_stall>0.1</cda_stall>
-        <cma_stall>-0.2</cma_stall>
-        <cp>0.0 0.0 0.0</cp>
-        <area>${area}</area>
-        <air_density>1.225</air_density>
-        <forward>${forward_x} ${forward_y} ${forward_z}</forward>
-        <upward>${up_x} ${up_y} ${up_z}</upward>
-        <link_name>${robot_namespace}/${surface_name}</link_name>
-      </plugin>
-    </gazebo>-->
     <gazebo reference="${robot_namespace}/${surface_name}">
       <material>Gazebo/${color}</material>
