Commit message: Started implementing a service for registering an aero surface

File: rotors_description/urdf/atlantik_solar.xacro (robot description, xacro)
@@ -219,64 +219,48 @@
   </xacro:wheel>
   <!-- Instantiate wings -->
-  <xacro:wing
-    robot_namespace="${namespace}"
-    suffix="left_big"
-    parent="${namespace}/base_link_inertia"
-    mass_wing="${mass_front_wing}"
-    wing_length="${root_chord}"
-    wing_width="${front_wing_width}"
-    wing_height="${front_wing_height}"
-    color="${body_color}"
-    use_mesh="false"
-    mesh="">
+  <xacro:aero_surface
+    robot_namespace="${namespace}"
+    surface_name="left_wing"
+    surface_type="wing"
+    parent="${namespace}/base_link_inertia"
+    mass_surface="${mass_front_wing}"
+    joint_gain="0.0"
+    positive_direction="cw"
+    channel="0"
+    min_angle="0.0"
+    max_angle="0.0"
+    surface_length="${root_chord}"
+    surface_width="${front_wing_width}"
+    surface_height="${front_wing_height}"
+    color="${body_color}"
+    use_mesh="false"
+    mesh="">
+    <axis xyz="1 0 0" />
     <origin xyz="0.5 ${0.5 * body_width} 0.0" rpy="0.0 0.0 0.0" />
     <origin xyz="0.0 ${0.5 * front_wing_width} 0.0" rpy="0.0 0.0 0.0" />
     <xacro:insert_block name="front_wing_inertia" />
-  </xacro:wing>-->
-  <xacro:wing
-    robot_namespace="${namespace}"
-    suffix="right_big"
-    parent="${namespace}/base_link_inertia"
-    mass_wing="${mass_front_wing}"
-    wing_length="${root_chord}"
-    wing_width="${front_wing_width}"
-    wing_height="${front_wing_height}"
-    color="${body_color}"
-    use_mesh="false"
-    mesh="">
+  </xacro:aero_surface>
+  <xacro:aero_surface
+    robot_namespace="${namespace}"
+    surface_name="right_wing"
+    surface_type="wing"
+    parent="${namespace}/base_link_inertia"
+    mass_surface="${mass_front_wing}"
+    joint_gain="0.0"
+    positive_direction="cw"
+    channel="0"
+    min_angle="0.0"
+    max_angle="0.0"
+    surface_length="${root_chord}"
+    surface_width="${front_wing_width}"
+    surface_height="${front_wing_height}"
+    color="${body_color}"
+    use_mesh="false"
+    mesh="">
+    <axis xyz="1 0 0" />
     <origin xyz="0.5 ${-0.5 * body_width} 0.0" rpy="0.0 0.0 0.0" />
     <origin xyz="0.0 ${-0.5 * front_wing_width} 0.0" rpy="0.0 0.0 0.0" />
     <xacro:insert_block name="front_wing_inertia" />
-  </xacro:wing>
-  <xacro:wing
-    robot_namespace="${namespace}"
-    suffix="left_small"
-    parent="${namespace}/base_link_inertia"
-    mass_wing="${mass_small_wing}"
-    wing_length="${aileron_length}"
-    wing_width="${front_wing_width - aileron_width}"
-    wing_height="${front_wing_height}"
-    color="${body_color}"
-    use_mesh="false"
-    mesh="">
-    <origin xyz="${0.5 * (1 - root_chord - aileron_length)} ${0.5 * body_width} 0.0" rpy="0.0 0.0 0.0" />
-    <origin xyz="0.0 ${0.5 * (front_wing_width - aileron_width)} 0.0" rpy="0.0 0.0 0.0" />
-    <xacro:insert_block name="small_wing_inertia" />
-  </xacro:wing>
-  <xacro:wing
-    robot_namespace="${namespace}"
-    suffix="right_small"
-    parent="${namespace}/base_link_inertia"
-    mass_wing="${mass_small_wing}"
-    wing_length="${aileron_length}"
-    wing_width="${front_wing_width - aileron_width}"
-    wing_height="${front_wing_height}"
-    color="${body_color}"
-    use_mesh="false"
-    mesh="">
-    <origin xyz="${0.5 * (1 - root_chord - aileron_length)} ${-0.5 * body_width} 0.0" rpy="0.0 0.0 0.0" />
-    <origin xyz="0.0 ${-0.5 * (front_wing_width - aileron_width)} 0.0" rpy="0.0 0.0 0.0" />
-    <xacro:insert_block name="small_wing_inertia" />
-  </xacro:wing>
+  </xacro:aero_surface>
   <!-- Instantiate the tail -->
   <xacro:tail
@@ -294,36 +278,50 @@
   </xacro:tail>
   <!-- Instantiate the rear wings-->
-  <xacro:wing
-    robot_namespace="${namespace}"
-    suffix="rear_left"
+  <xacro:aero_surface
+    robot_namespace="${namespace}"
+    surface_name="rear_left_wing"
+    surface_type="wing"
     parent="${namespace}/tail"
-    mass_wing="${mass_rear_wing}"
-    wing_length="${tail_length - elevator_length}"
-    wing_width="${rear_wing_width}"
-    wing_height="${rear_wing_height}"
-    color="${body_color}"
-    use_mesh="false"
-    mesh="">
+    mass_surface="${mass_rear_wing}"
+    joint_gain="0.0"
+    positive_direction="cw"
+    channel="0"
+    min_angle="0.0"
+    max_angle="0.0"
+    surface_length="${tail_length - elevator_length}"
+    surface_width="${rear_wing_width}"
+    surface_height="${rear_wing_height}"
+    color="${body_color}"
+    use_mesh="false"
+    mesh="">
+    <axis xyz="1 0 0" />
     <origin xyz="${0.5 * elevator_length} ${0.5 * tail_width} ${0.5 * (tail_height - rear_wing_height)}" rpy="0.0 0.0 0.0" />
     <origin xyz="0.0 ${0.5 * rear_wing_width} 0.0" rpy="0.0 0.0 0.0" />
     <xacro:insert_block name="rear_wing_inertia" />
-  </xacro:wing>
-  <xacro:wing
-    robot_namespace="${namespace}"
-    suffix="rear_right"
+  </xacro:aero_surface>
+  <xacro:aero_surface
+    robot_namespace="${namespace}"
+    surface_name="rear_right"
+    surface_type="wing"
     parent="${namespace}/tail"
-    mass_wing="${mass_rear_wing}"
-    wing_length="${tail_length - elevator_length}"
-    wing_width="${rear_wing_width}"
-    wing_height="${rear_wing_height}"
-    color="${body_color}"
-    use_mesh="false"
-    mesh="">
+    mass_surface="${mass_rear_wing}"
+    joint_gain="0.0"
+    positive_direction="cw"
+    channel="0"
+    min_angle="0.0"
+    max_angle="0.0"
+    surface_length="${tail_length - elevator_length}"
+    surface_width="${rear_wing_width}"
+    surface_height="${rear_wing_height}"
+    color="${body_color}"
+    use_mesh="false"
+    mesh="">
+    <axis xyz="1 0 0" />
     <origin xyz="${0.5 * elevator_length} ${-0.5 * tail_width} ${0.5 * (tail_height - rear_wing_height)}" rpy="0.0 0.0 0.0" />
     <origin xyz="0.0 ${-0.5 * rear_wing_width} 0.0" rpy="0.0 0.0 0.0" />
     <xacro:insert_block name="rear_wing_inertia" />
-  </xacro:wing>
+  </xacro:aero_surface>
   <!-- Instantiate the control surfaces -->
-  <xacro:control_surface
+<!--  <xacro:control_surface
     robot_namespace="${namespace}"
     surface_name="aileron_left"
@@ -429,4 +427,4 @@
     <origin xyz="${-0.5 * rudder_length} 0.0 0.0" rpy="0.0 0.0 0.0" />
     <xacro:insert_block name="rudder_inertia" />
-  </xacro:control_surface>
+  </xacro:control_surface>-->
 </robot>

File: rotors_description/urdf/fixed_wing_base.xacro (robot description, xacro)
@@ -117,5 +117,5 @@
   </xacro:macro>
   <!-- Wing joint and link -->
-  <xacro:macro name="wing"
+<!--  <xacro:macro name="wing"
     params="robot_namespace suffix parent mass_wing wing_length wing_width wing_height
       color use_mesh mesh *joint_origin *link_origin *inertia">
@@ -130,23 +130,23 @@
       <inertial>
         <xacro:insert_block name="link_origin" />
-        <mass value="${mass_wing}" /> <!-- [kg] -->
-        <xacro:insert_block name="inertia" />
-      </inertial>
-      <visual>
-        <xacro:insert_block name="link_origin" />
-        <geometry>
-          <xacro:if value="${use_mesh}">
-            <mesh filename="${mesh}"
-              scale="1 1 1" />
-          </xacro:if>
-          <xacro:unless value="${use_mesh}">
-            <box size="${wing_length} ${wing_width} ${wing_height}"/> <!-- [m] [m] [m] -->
-          </xacro:unless>
-        </geometry>
-      </visual>
-      <collision>
-        <xacro:insert_block name="link_origin" />
-        <geometry>
-          <box size="${wing_length - 0.01} ${wing_width - 0.01} ${wing_height - 0.01}"/> <!-- [m] [m] [m] -->
+        <mass value="${mass_wing}" />
+        <xacro:insert_block name="inertia" />
+      </inertial>
+      <visual>
+        <xacro:insert_block name="link_origin" />
+        <geometry>
+          <xacro:if value="${use_mesh}">
+            <mesh filename="${mesh}"
+              scale="1 1 1" />
+          </xacro:if>
+          <xacro:unless value="${use_mesh}">
+            <box size="${wing_length} ${wing_width} ${wing_height}"/>
+          </xacro:unless>
+        </geometry>
+      </visual>
+      <collision>
+        <xacro:insert_block name="link_origin" />
+        <geometry>
+          <box size="${wing_length - 0.01} ${wing_width - 0.01} ${wing_height - 0.01}"/>
         </geometry>
       </collision>
@@ -155,5 +155,5 @@
       <material>Gazebo/${color}</material>
     </gazebo>
-  </xacro:macro>
+  </xacro:macro>-->
   <!-- Tail joint and link -->
   <xacro:macro name="tail"
@@ -253,5 +253,5 @@
   </xacro:macro>
   <!-- Control surface joint and link -->
-  <xacro:macro name="control_surface"
+<!--  <xacro:macro name="control_surface"
     params="robot_namespace surface_name parent mass_surface gain
       positive_direction min_angle max_angle channel color use_mesh mesh
@@ -270,23 +270,23 @@
       <inertial>
         <xacro:insert_block name="link_origin" />
-        <mass value="${mass_surface}" /> <!-- [kg] -->
-        <xacro:insert_block name="inertia" />
-      </inertial>
-      <visual>
-        <xacro:insert_block name="link_origin" />
-        <geometry>
-          <xacro:if value="${use_mesh}">
-            <mesh filename="${mesh}"
-              scale="1 1 1" />
-          </xacro:if>
-          <xacro:unless value="${use_mesh}">
-            <box size="${surface_length} ${surface_width} ${surface_height}"/> <!-- [m] [m] [m] -->
-          </xacro:unless>
-        </geometry>
-      </visual>
-      <collision>
-        <xacro:insert_block name="link_origin" />
-        <geometry>
-          <box size="${surface_length - 0.01} ${surface_width - 0.01} ${surface_height - 0.01}"/> <!-- [m] [m] [m] -->
+        <mass value="${mass_surface}" />
+        <xacro:insert_block name="inertia" />
+      </inertial>
+      <visual>
+        <xacro:insert_block name="link_origin" />
+        <geometry>
+          <xacro:if value="${use_mesh}">
+            <mesh filename="${mesh}"
+              scale="1 1 1" />
+          </xacro:if>
+          <xacro:unless value="${use_mesh}">
+            <box size="${surface_length} ${surface_width} ${surface_height}"/>
+          </xacro:unless>
+        </geometry>
+      </visual>
+      <collision>
+        <xacro:insert_block name="link_origin" />
+        <geometry>
+          <box size="${surface_length - 0.01} ${surface_width - 0.01} ${surface_height - 0.01}"/>
         </geometry>
       </collision>
@@ -308,4 +308,60 @@
       <material>Gazebo/${color}</material>
     </gazebo>
+  </xacro:macro>-->
+  <!-- Aerodynamic surface joint and link -->
+  <xacro:macro name="aero_surface"
+    params="robot_namespace surface_name surface_type parent mass_surface joint_gain
+      positive_direction channel min_angle max_angle color use_mesh mesh surface_length
+      surface_width surface_height *axis *joint_origin *link_origin *inertia">
+    <joint name="${robot_namespace}/${surface_name}_joint" type="revolute">
+      <xacro:insert_block name="joint_origin" />
+      <xacro:insert_block name="axis" />
+      <parent link="${parent}" />
+      <child link="${robot_namespace}/${surface_name}" />
+      <limit upper="${max_angle}" lower="${min_angle}" effort="200.0" velocity="3.0" />
+      <dynamics friction="${9.8 * mass_surface}" damping="${9.8 * mass_surface}" />
+    </joint>
+    <link name="${robot_namespace}/${surface_name}">
+      <inertial>
+        <xacro:insert_block name="link_origin" />
+        <mass value="${mass_surface}" />
+        <xacro:insert_block name="inertia" />
+      </inertial>
+      <visual>
+        <xacro:insert_block name="link_origin" />
+        <geometry>
+          <xacro:if value="${use_mesh}">
+            <mesh filename="${mesh}"
+              scale="1 1 1" />
+          </xacro:if>
+          <xacro:unless value="${use_mesh}">
+            <box size="${surface_length} ${surface_width} ${surface_height}"/>
+          </xacro:unless>
+        </geometry>
+      </visual>
+      <collision>
+        <xacro:insert_block name="link_origin" />
+        <geometry>
+          <box size="${surface_length - 0.01} ${surface_width - 0.01} ${surface_height - 0.01}"/>
+        </geometry>
+      </collision>
+    </link>
+    <gazebo>
+      <plugin name="${robot_namespace}_${surface_name}" filename="librotors_gazebo_aero_surface_plugin.so">
+        <robotNamespace>${robot_namespace}</robotNamespace>
+        <jointName>${robot_namespace}/${surface_name}_joint</jointName>
+        <surfaceType>${surface_type}</surfaceType>
+        <positiveDirection>${positive_direction}</positiveDirection>
+        <commandSubTopic>gazebo/command/motor_speed</commandSubTopic>
+	<surfaceArea>${surface_length * surface_width}</surfaceArea>
+        <gain>${joint_gain}</gain>
+        <channel>${channel}</channel>
+        <minAngle>${min_angle}</minAngle>
+        <maxAngle>${max_angle}</maxAngle>
+      </plugin>
+    </gazebo>
+    <gazebo reference="${robot_namespace}/${surface_name}">
+      <material>Gazebo/${color}</material>
+    </gazebo>
   </xacro:macro>
 </robot>
