Commit message: Some minor clean-up

File: rotors_description/urdf/atlantik_solar.xacro (robot description, xacro)
@@ -23,14 +23,13 @@
   <xacro:property name="mesh_file" value="" />
   <!-- Component masses -->
-  <xacro:property name="mass_fuselage" value="3.0" /> <!-- [kg] -->
+  <xacro:property name="mass_fuselage" value="2.0" /> <!-- [kg] -->
   <xacro:property name="mass_wheel" value="0.05" /> <!-- [kg] -->
-  <xacro:property name="mass_front_wing" value="1.0" /> <!-- [kg] -->
-  <xacro:property name="mass_small_wing" value="0.3" /> <!-- [kg] -->
+  <xacro:property name="mass_wing" value="0.5" /> <!-- [kg] -->
+  <xacro:property name="mass_vertical_stabilizer" value="0.2" /> <!-- [kg] -->
   <xacro:property name="mass_tail" value="0.25" /> <!-- [kg] -->
-  <xacro:property name="mass_rear_wing" value="0.25" /> <!-- [kg] -->
   <xacro:property name="mass_propeller" value="0.01" /> <!-- [kg] -->
-  <xacro:property name="mass_aileron" value="0.3" /> <!-- [kg] -->
-  <xacro:property name="mass_elevator" value="0.2" /> <!-- [kg] -->
-  <xacro:property name="mass_rudder" value="0.2" /> <!-- [kg] -->
+  <xacro:property name="mass_aileron" value="0.2" /> <!-- [kg] -->
+  <xacro:property name="mass_elevator" value="0.1" /> <!-- [kg] -->
+  <xacro:property name="mass_rudder" value="0.1" /> <!-- [kg] -->
   <!-- Fuselage properties -->
   <xacro:property name="body_length" value="3.0" /> <!-- [m] -->
@@ -44,5 +43,5 @@
   <xacro:property name="propeller_offset" value="0.025" /> <!-- [m] -->
   <xacro:property name="radius_propeller" value="0.15" /> <!-- [m] -->
-  <xacro:property name="motor_constant" value="6.14858e-04" /> <!-- [kg m/s^2] -->
+  <xacro:property name="motor_constant" value="2.14858e-04" /> <!-- [kg m/s^2] -->
   <xacro:property name="moment_constant" value="0.016" /> <!-- [m] -->
   <xacro:property name="time_constant_up" value="0.0125" /> <!-- [s] -->
@@ -54,7 +53,7 @@
   <xacro:property name="wingspan" value="4.0" /> <!-- [m] -->
   <xacro:property name="root_chord" value="0.3" /> <!-- [m] -->
-  <xacro:property name="front_wing_height" value="0.02" /> <!-- [m] -->
-  <xacro:property name="rear_wingspan" value="1.0" /> <!-- [m] -->
-  <xacro:property name="rear_wing_height" value="0.02" /> <!-- [m] -->
+  <xacro:property name="wing_height" value="0.02" /> <!-- [m] -->
+  <xacro:property name="tail_wingspan" value="1.0" /> <!-- [m] -->
+  <xacro:property name="tail_height" value="0.02" /> <!-- [m] -->
   <xacro:property name="alpha_0" value="0.01" /> <!-- [rad] -->
   <xacro:property name="alpha_stall" value="0.2" /> <!-- [rad] -->
@@ -62,10 +61,10 @@
   <xacro:property name="air_density" value="1.225" /> <!-- [kg/m^3] -->
   <!-- Tail properties -->
-  <xacro:property name="tail_length" value="0.4" /> <!-- [m] -->
-  <xacro:property name="tail_width" value="0.05" /> <!-- [m] -->
-  <xacro:property name="tail_height" value="0.2" /> <!-- [m] -->
+  <xacro:property name="vertical_stabilizer_length" value="0.4" /> <!-- [m] -->
+  <xacro:property name="vertical_stabilizer_width" value="0.05" /> <!-- [m] -->
+  <xacro:property name="vertical_stabilizer_height" value="0.2" /> <!-- [m] -->
   <!-- Aileron properties -->
   <xacro:property name="aileron_length" value="${0.5 * root_chord}" /> <!-- [m] -->
-  <xacro:property name="aileron_width" value="${0.5 * front_wing_width}" /> <!-- [m] -->
+  <xacro:property name="aileron_width" value="${0.5 * wing_width}" /> <!-- [m] -->
   <xacro:property name="aileron_height" value="0.02" /> <!-- [m] -->
   <xacro:property name="aileron_gain" value="2.0" />
@@ -75,5 +74,5 @@
   <!-- Elevator properties -->
   <xacro:property name="elevator_length" value="0.15" /> <!-- [m] -->
-  <xacro:property name="elevator_width" value="${rear_wing_width}" /> <!-- [m] -->
+  <xacro:property name="elevator_width" value="${tail_width}" /> <!-- [m] -->
   <xacro:property name="elevator_height" value="0.02" /> <!-- [m] -->
   <xacro:property name="elevator_gain" value="2.0" />
@@ -83,6 +82,6 @@
   <!-- Rudder properties -->
   <xacro:property name="rudder_length" value="0.1" /> <!-- [m] -->
-  <xacro:property name="rudder_width" value="${tail_width}" /> <!-- [m] -->
-  <xacro:property name="rudder_height" value="${tail_height}" /> <!-- [m] -->
+  <xacro:property name="rudder_width" value="${vertical_stabilizer_width}" /> <!-- [m] -->
+  <xacro:property name="rudder_height" value="${vertical_stabilizer_height}" /> <!-- [m] -->
   <xacro:property name="rudder_gain" value="2.0" />
   <xacro:property name="rudder_min_angle" value="-0.55" /> <!-- [rad] -->
@@ -92,11 +91,7 @@
   <xacro:property name="PI" value="3.1415926535897931" />
   <!-- Front wing length -->
-  <xacro:property name="front_wing_width" value="${0.5 * (wingspan - body_width)}" />
+  <xacro:property name="wing_width" value="${0.5 * (wingspan - body_width)}" />
   <!-- Rear wing length -->
-  <xacro:property name="rear_wing_width" value="${0.5 * (rear_wingspan - tail_width)}" />
-  <!-- Total area of the wings -->
-  <xacro:property name="total_wing_area"
-    value="${2.0 * (front_wing_width * root_chord + (front_wing_width - aileron_width) * aileron_length)}" >
-  </xacro:property>
+  <xacro:property name="tail_width" value="${0.5 * (tail_wingspan - vertical_stabilizer_width)}" />
   <!-- Inertia of the fuselage -->
   <xacro:property name="body_inertia">
@@ -108,18 +103,14 @@
   </xacro:property>
   <!-- Inertia of a single front wing, assuming it is a cuboid -->
-  <xacro:property name="front_wing_inertia">
-    <xacro:box_inertia x="${root_chord}" y="${front_wing_width}" z="${front_wing_height}" mass="${mass_front_wing}" />
-  </xacro:property>
-  <!-- Inertia of a single small front wing, assuming it is a cuboid -->
-  <xacro:property name="small_wing_inertia">
-    <xacro:box_inertia x="${aileron_length}" y="${front_wing_width - aileron_width}" z="${front_wing_height}" mass="${mass_small_wing}" />
-  </xacro:property>
-  <!-- Inertia of the tail, assuming it is a cuboid -->
+  <xacro:property name="wing_inertia">
+    <xacro:box_inertia x="${root_chord}" y="${wing_width}" z="${wing_height}" mass="${mass_wing}" />
+  </xacro:property>
+  <!-- Inertia of the vertical_stabilizer, assuming it is a cuboid -->
+  <xacro:property name="vertical_stabilizer_inertia">
+    <xacro:box_inertia x="${vertical_stabilizer_length}" y="${vertical_stabilizer_width}" z="${vertical_stabilizer_height}" mass="${mass_vertical_stabilizer}" />
+  </xacro:property>
+  <!-- Inertia of a single tail wing, assuming it is a cuboid -->
   <xacro:property name="tail_inertia">
-    <xacro:box_inertia x="${tail_length}" y="${tail_width}" z="${tail_height}" mass="${mass_tail}" />
-  </xacro:property>
-  <!-- Inertia of a single rear wing, assuming it is a cuboid -->
-  <xacro:property name="rear_wing_inertia">
-    <xacro:box_inertia x="${tail_length - elevator_length}" y="${rear_wing_width}" z="${rear_wing_height}" mass="${mass_rear_wing}" />
+    <xacro:box_inertia x="${vertical_stabilizer_length - elevator_length}" y="${tail_width}" z="${tail_height}" mass="${mass_tail}" />
   </xacro:property>
   <!-- Inertia of the propeller, assuming it is a cuboid. Height=3mm, width=40mm -->
@@ -145,12 +136,11 @@
     robot_namespace="${namespace}"
     mass="${mass_fuselage}"
-    body_length="${body_length}"
-    body_width="${body_width}"
-    body_height="${body_height}"
+    length="${body_length}"
+    width="${body_width}"
+    height="${body_height}"
     color="${body_color}"
     use_mesh_file="${use_mesh_file}"
     mesh_file="${mesh_file}"
     reset_topic="reset"
-    total_wing_area="${total_wing_area}"
     air_density="${air_density}"
     alpha_stall="${alpha_stall}">
@@ -164,6 +154,6 @@
     moment_constant="${moment_constant}"
     parent="${namespace}/base_link_inertia"
-    mass_propeller="${mass_propeller}"
-    radius_propeller="${radius_propeller}"
+    mass="${mass_propeller}"
+    radius="${radius_propeller}"
     time_constant_up="${time_constant_up}"
     time_constant_down="${time_constant_down}"
@@ -183,10 +173,10 @@
     suffix="front_left"
     parent="${namespace}/base_link_inertia"
-    mass_wheel="${mass_wheel}"
-    color="${body_color}"
-    use_mesh="false"
-    mesh=""
-    wheel_radius="${wheel_radius}"
-    wheel_width="${wheel_width}">
+    mass="${mass_wheel}"
+    color="${body_color}"
+    use_mesh="false"
+    mesh=""
+    radius="${wheel_radius}"
+    width="${wheel_width}">
     <origin xyz="0.75 0.1 -0.1" rpy="${0.5 * PI} 0.0 0.0" />
     <xacro:insert_block name="wheel_inertia" />
@@ -196,10 +186,10 @@
     suffix="front_right"
     parent="${namespace}/base_link_inertia"
-    mass_wheel="${mass_wheel}"
-    color="${body_color}"
-    use_mesh="false"
-    mesh=""
-    wheel_radius="${wheel_radius}"
-    wheel_width="${wheel_width}">
+    mass="${mass_wheel}"
+    color="${body_color}"
+    use_mesh="false"
+    mesh=""
+    radius="${wheel_radius}"
+    width="${wheel_width}">
     <origin xyz="0.75 -0.1 -0.1" rpy="${0.5 * PI} 0.0 0.0" />
     <xacro:insert_block name="wheel_inertia" />
@@ -209,10 +199,10 @@
     suffix="back"
     parent="${namespace}/base_link_inertia"
-    mass_wheel="${mass_wheel}"
-    color="${body_color}"
-    use_mesh="false"
-    mesh=""
-    wheel_radius="${wheel_radius}"
-    wheel_width="${wheel_width}">
+    mass="${mass_wheel}"
+    color="${body_color}"
+    use_mesh="false"
+    mesh=""
+    radius="${wheel_radius}"
+    width="${wheel_width}">
     <origin xyz="-1.0 0.0 -0.1" rpy="${0.5 * PI} 0.0 0.0" />
     <xacro:insert_block name="wheel_inertia" />
@@ -224,5 +214,5 @@
     surface_type="wing"
     parent="${namespace}/base_link_inertia"
-    mass_surface="${mass_front_wing}"
+    mass_surface="${mass_wing}"
     joint_gain="0.0"
     positive_direction="cw"
@@ -231,6 +221,6 @@
     max_angle="0.0"
     surface_length="${root_chord}"
-    surface_width="${front_wing_width}"
-    surface_height="${front_wing_height}"
+    surface_width="${wing_width}"
+    surface_height="${wing_height}"
     color="${body_color}"
     use_mesh="false"
@@ -238,6 +228,6 @@
     <axis xyz="1 0 0" />
     <origin xyz="0.5 ${0.5 * body_width} 0.0" rpy="0.0 0.0 0.0" />
-    <origin xyz="0.0 ${0.5 * front_wing_width} 0.0" rpy="0.0 0.0 0.0" />
-    <xacro:insert_block name="front_wing_inertia" />
+    <origin xyz="0.0 ${0.5 * wing_width} 0.0" rpy="0.0 0.0 0.0" />
+    <xacro:insert_block name="wing_inertia" />
   </xacro:aero_surface>
   <xacro:aero_surface
@@ -246,5 +236,5 @@
     surface_type="wing"
     parent="${namespace}/base_link_inertia"
-    mass_surface="${mass_front_wing}"
+    mass_surface="${mass_wing}"
     joint_gain="0.0"
     positive_direction="cw"
@@ -253,6 +243,6 @@
     max_angle="0.0"
     surface_length="${root_chord}"
-    surface_width="${front_wing_width}"
-    surface_height="${front_wing_height}"
+    surface_width="${wing_width}"
+    surface_height="${wing_height}"
     color="${body_color}"
     use_mesh="false"
@@ -260,28 +250,28 @@
     <axis xyz="1 0 0" />
     <origin xyz="0.5 ${-0.5 * body_width} 0.0" rpy="0.0 0.0 0.0" />
-    <origin xyz="0.0 ${-0.5 * front_wing_width} 0.0" rpy="0.0 0.0 0.0" />
-    <xacro:insert_block name="front_wing_inertia" />
-  </xacro:aero_surface>
-  <!-- Instantiate the tail -->
-  <xacro:tail
-    robot_namespace="${namespace}"
-    parent="${namespace}/base_link_inertia"
-    mass_tail="${mass_tail}"
-    tail_length="${tail_length}"
-    tail_width="${tail_width}"
-    tail_height="${tail_height}"
-    color="${body_color}"
-    use_mesh="false"
-    mesh="">
-    <origin xyz="${-0.5*body_length + 0.5*tail_length} 0.0 ${0.5*body_height + 0.5*tail_height}" rpy="0.0 0.0 0.0" />
-    <xacro:insert_block name="tail_inertia" />
-  </xacro:tail>
+    <origin xyz="0.0 ${-0.5 * wing_width} 0.0" rpy="0.0 0.0 0.0" />
+    <xacro:insert_block name="wing_inertia" />
+  </xacro:aero_surface>
+  <!-- Instantiate the vertical stabilizer -->
+  <xacro:vertical_stabilizer
+    robot_namespace="${namespace}"
+    parent="${namespace}/base_link_inertia"
+    mass="${mass_vertical_stabilizer}"
+    length="${vertical_stabilizer_length}"
+    width="${vertical_stabilizer_width}"
+    height="${vertical_stabilizer_height}"
+    color="${body_color}"
+    use_mesh="false"
+    mesh="">
+    <origin xyz="${-0.5*body_length + 0.5*vertical_stabilizer_length} 0.0 ${0.5*body_height + 0.5*vertical_stabilizer_height}" rpy="0.0 0.0 0.0" />
+    <xacro:insert_block name="vertical_stabilizer_inertia" />
+  </xacro:vertical_stabilizer>
   <!-- Instantiate the rear wings-->
   <xacro:aero_surface
     robot_namespace="${namespace}"
-    surface_name="rear_wing_left"
-    surface_type="wing"
-    parent="${namespace}/tail"
-    mass_surface="${mass_rear_wing}"
+    surface_name="tail_left"
+    surface_type="tail"
+    parent="${namespace}/vertical_stabilizer"
+    mass_surface="${mass_tail}"
     joint_gain="0.0"
     positive_direction="cw"
@@ -289,21 +279,21 @@
     min_angle="0.0"
     max_angle="0.0"
-    surface_length="${tail_length - elevator_length}"
-    surface_width="${rear_wing_width}"
-    surface_height="${rear_wing_height}"
+    surface_length="${vertical_stabilizer_length - elevator_length}"
+    surface_width="${tail_width}"
+    surface_height="${tail_height}"
     color="${body_color}"
     use_mesh="false"
     mesh="">
     <axis xyz="1 0 0" />
-    <origin xyz="${0.5 * elevator_length} ${0.5 * tail_width} ${0.5 * (tail_height - rear_wing_height)}" rpy="0.0 0.0 0.0" />
-    <origin xyz="0.0 ${0.5 * rear_wing_width} 0.0" rpy="0.0 0.0 0.0" />
-    <xacro:insert_block name="rear_wing_inertia" />
-  </xacro:aero_surface>
-  <xacro:aero_surface
-    robot_namespace="${namespace}"
-    surface_name="rear_wing_right"
-    surface_type="wing"
-    parent="${namespace}/tail"
-    mass_surface="${mass_rear_wing}"
+    <origin xyz="${0.5 * elevator_length} ${0.5 * vertical_stabilizer_width} ${0.5 * (vertical_stabilizer_height - tail_height)}" rpy="0.0 0.0 0.0" />
+    <origin xyz="0.0 ${0.5 * tail_width} 0.0" rpy="0.0 0.0 0.0" />
+    <xacro:insert_block name="tail_inertia" />
+  </xacro:aero_surface>
+  <xacro:aero_surface
+    robot_namespace="${namespace}"
+    surface_name="tail_right"
+    surface_type="tail"
+    parent="${namespace}/vertical_stabilizer"
+    mass_surface="${mass_tail}"
     joint_gain="0.0"
     positive_direction="cw"
@@ -311,17 +301,17 @@
     min_angle="0.0"
     max_angle="0.0"
-    surface_length="${tail_length - elevator_length}"
-    surface_width="${rear_wing_width}"
-    surface_height="${rear_wing_height}"
+    surface_length="${vertical_stabilizer_length - elevator_length}"
+    surface_width="${tail_width}"
+    surface_height="${tail_height}"
     color="${body_color}"
     use_mesh="false"
     mesh="">
     <axis xyz="1 0 0" />
-    <origin xyz="${0.5 * elevator_length} ${-0.5 * tail_width} ${0.5 * (tail_height - rear_wing_height)}" rpy="0.0 0.0 0.0" />
-    <origin xyz="0.0 ${-0.5 * rear_wing_width} 0.0" rpy="0.0 0.0 0.0" />
-    <xacro:insert_block name="rear_wing_inertia" />
+    <origin xyz="${0.5 * elevator_length} ${-0.5 * vertical_stabilizer_width} ${0.5 * (vertical_stabilizer_height - tail_height)}" rpy="0.0 0.0 0.0" />
+    <origin xyz="0.0 ${-0.5 * tail_width} 0.0" rpy="0.0 0.0 0.0" />
+    <xacro:insert_block name="tail_inertia" />
   </xacro:aero_surface>
   <!-- Instantiate the ailerons -->
-  <xacro:aero_surface
+<!--  <xacro:aero_surface
     robot_namespace="${namespace}"
     surface_name="aileron_left"
@@ -341,5 +331,5 @@
     surface_height="${aileron_height}">
     <axis xyz="0 1 0" />
-    <origin xyz="${-0.5 * root_chord} ${front_wing_width - 0.5 * aileron_width} 0.0" rpy="0.0 0.0 0.0" />
+    <origin xyz="${-0.5 * root_chord} ${wing_width - 0.5 * aileron_width} 0.0" rpy="0.0 0.0 0.0" />
     <origin xyz="${-0.5 * aileron_length} 0.0 0.0" rpy="0.0 0.0 0.0" />
     <xacro:insert_block name="aileron_inertia" />
@@ -363,14 +353,14 @@
     surface_height="${aileron_height}">
     <axis xyz="0 1 0" />
-    <origin xyz="${-0.5 * root_chord} ${-(front_wing_width - 0.5 * aileron_width)} 0.0" rpy="0.0 0.0 0.0" />
+    <origin xyz="${-0.5 * root_chord} ${-(wing_width - 0.5 * aileron_width)} 0.0" rpy="0.0 0.0 0.0" />
     <origin xyz="${-0.5 * aileron_length} 0.0 0.0" rpy="0.0 0.0 0.0" />
     <xacro:insert_block name="aileron_inertia" />
-  </xacro:aero_surface>
+  </xacro:aero_surface>-->
   <!-- Instantiate the elevators -->
-  <xacro:aero_surface
+<!--  <xacro:aero_surface
     robot_namespace="${namespace}"
     surface_name="elevator_left"
     surface_type="elevator"
-    parent="${namespace}/rear_wing_left"
+    parent="${namespace}/tail_left"
     mass_surface="${mass_elevator}"
     joint_gain="${elevator_gain}"
@@ -386,5 +376,5 @@
     surface_height="${elevator_height}">
     <axis xyz="0 1 0" />
-    <origin xyz="${-0.5 * (tail_length - elevator_length)} ${0.5 * rear_wing_width} 0.0" rpy="0.0 0.0 0.0" />
+    <origin xyz="${-0.5 * (vertical_stabilizer_length - elevator_length)} ${0.5 * tail_width} 0.0" rpy="0.0 0.0 0.0" />
     <origin xyz="${-0.5 * elevator_length} 0.0 0.0" rpy="0.0 0.0 0.0" />
     <xacro:insert_block name="elevator_inertia" />
@@ -394,5 +384,5 @@
     surface_name="elevator_right"
     surface_type="elevator"
-    parent="${namespace}/rear_wing_right"
+    parent="${namespace}/tail_right"
     mass_surface="${mass_elevator}"
     joint_gain="${elevator_gain}"
@@ -408,14 +398,14 @@
     surface_height="${elevator_height}">
     <axis xyz="0 1 0" />
-    <origin xyz="${-0.5 * (tail_length - elevator_length)} ${-0.5 * rear_wing_width} 0.0" rpy="0.0 0.0 0.0" />
+    <origin xyz="${-0.5 * (vertical_stabilizer_length - elevator_length)} ${-0.5 * tail_width} 0.0" rpy="0.0 0.0 0.0" />
     <origin xyz="${-0.5 * elevator_length} 0.0 0.0" rpy="0.0 0.0 0.0" />
     <xacro:insert_block name="elevator_inertia" />
-  </xacro:aero_surface>
+  </xacro:aero_surface>-->
   <!-- Instantiate the rudder -->
-  <xacro:aero_surface
+<!--  <xacro:aero_surface
     robot_namespace="${namespace}"
     surface_name="rudder"
     surface_type="rudder"
-    parent="${namespace}/tail"
+    parent="${namespace}/vertical_stabilizer"
     mass_surface="${mass_rudder}"
     joint_gain="${rudder_gain}"
@@ -431,7 +421,7 @@
     surface_height="${rudder_height}">
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
File: rotors_description/urdf/atlantik_solar_base.xacro (robot description, xacro)
@@ -31,5 +31,5 @@
   <xacro:default_pressure_sensor namespace="${namespace}" parent_link="${namespace}/base_link_inertia" />
   <!-- Mount a downward-looking camera. -->
-  <xacro:camera_macro
+<!--  <xacro:camera_macro
     namespace="${namespace}"
     parent_link="${namespace}/base_link_inertia"
@@ -47,5 +47,5 @@
     <mesh filename="package://rotors_description/meshes/vi_camera.dae" scale="1 1 1" />
     <origin xyz="0 0 -0.05" rpy="0 1.5707 0" />
-  </xacro:camera_macro>
+  </xacro:camera_macro>-->
   <xacro:if value="$(arg enable_ground_truth)">
     <xacro:ground_truth_imu_and_odometry namespace="${namespace}" parent_link="${namespace}/base_link_inertia" />
