Commit message: Some minor clean-up

File: rotors_description/urdf/fixed_wing_base.xacro (robot description, xacro)
@@ -31,17 +31,17 @@
   <!-- Fixed-wing fuselage link -->
   <xacro:macro name="fixed_wing_base_macro"
-    params="robot_namespace mass body_length body_width body_height color
-      use_mesh_file mesh_file reset_topic total_wing_area air_density
-      alpha_stall *inertia">
-    <link name="${robot_namespace}/base_link"></link>
+    params="robot_namespace mass length width height color use_mesh_file
+      mesh_file reset_topic air_density alpha_stall *inertia">
+<!--    <link name="${robot_namespace}/base_link"></link>
     <joint name="${robot_namespace}/base_joint" type="fixed">
       <origin xyz="0 0 0.1" rpy="0 0 0" />
       <parent link="${robot_namespace}/base_link" />
       <child link="${robot_namespace}/base_link_inertia" />
-    </joint>
+    </joint>-->
     <link name="${robot_namespace}/base_link_inertia">
-      <inertial>
-        <mass value="${mass}" />  <!-- [kg] -->
-        <origin xyz="0.7 0 0" rpy="0 0 0" />
+      <pose>0 0 0 0 0 0</pose>
+      <inertial>
+        <mass value="${mass}" />
+        <origin xyz="0.0 0 0" rpy="0 0 0" />
         <xacro:insert_block name="inertia" />
       </inertial>
@@ -53,5 +53,5 @@
           </xacro:if>
           <xacro:unless value="${use_mesh_file}">
-            <box size="${body_length} ${body_width} ${body_height}"/> <!-- [m] [m] [m] -->
+            <box size="${length} ${width} ${height}" />
           </xacro:unless>
         </geometry>
@@ -60,5 +60,5 @@
         <origin xyz="0 0 0" rpy="0 0 0" />
         <geometry>
-          <box size="${body_length} ${body_width} ${body_height}" /> <!-- [m] [m] [m] -->
+          <box size="${length} ${width} ${height}" />
         </geometry>
       </collision>
@@ -67,6 +67,5 @@
       <plugin name="${robot_namespace}_base" filename="librotors_gazebo_fixedwing_base_plugin.so">
         <robotNamespace>${robot_namespace}</robotNamespace>
-        <linkName>${robot_namespace}/base_link</linkName>
-	<totalWingArea>${total_wing_area}</totalWingArea>
+        <linkName>${robot_namespace}/base_link_inertia</linkName>
 	<resetTopic>${reset_topic}</resetTopic>
 	<airDensity>${air_density}</airDensity>
@@ -74,5 +73,5 @@
       </plugin>
     </gazebo>
-    <gazebo reference="${robot_namespace}/base_link">
+    <gazebo reference="${robot_namespace}/base_link_inertia">
       <material>Gazebo/${color}</material>
     </gazebo>
@@ -80,6 +79,5 @@
   <!-- Wheel joint and link -->
   <xacro:macro name="wheel"
-    params="robot_namespace suffix parent mass_wheel color use_mesh mesh
-      wheel_radius wheel_width *origin *inertia">
+    params="robot_namespace suffix parent mass color use_mesh mesh radius width *origin *inertia">
     <joint name="${robot_namespace}/wheel_${suffix}_joint" type="fixed">
       <xacro:insert_block name="origin" />
@@ -92,5 +90,5 @@
       <inertial>
         <origin xyz="0.0 0.0 0.0" rpy="0.0 0.0 0.0" />
-        <mass value="${mass_wheel}" /> <!-- [kg] -->
+        <mass value="${mass}" />
         <xacro:insert_block name="inertia" />
       </inertial>
@@ -102,11 +100,11 @@
           </xacro:if>
           <xacro:unless value="${use_mesh}">
-            <cylinder length="${wheel_width}" radius="${wheel_radius}" /> <!-- [m] -->
-          </xacro:unless>
-        </geometry>
-      </visual>
-      <collision>
-        <geometry>
-          <cylinder length="${wheel_width}" radius="${wheel_radius}" /> <!-- [m] -->
+            <cylinder length="${width}" radius="${radius}" />
+          </xacro:unless>
+        </geometry>
+      </visual>
+      <collision>
+        <geometry>
+          <cylinder length="${width}" radius="${radius}" />
         </geometry>
       </collision>
@@ -116,59 +114,18 @@
     </gazebo>
   </xacro:macro>
-  <!-- Wing joint and link -->
-<!--  <xacro:macro name="wing"
-    params="robot_namespace suffix parent mass_wing wing_length wing_width wing_height
-      color use_mesh mesh *joint_origin *link_origin *inertia">
-    <joint name="${robot_namespace}/wing_${suffix}_joint" type="revolute">
-      <xacro:insert_block name="joint_origin" />
-      <axis xyz="1 0 0" />
-      <parent link="${parent}" />
-      <child link="${robot_namespace}/wing_${suffix}" />
-      <limit upper="0" lower="0" effort="0" velocity="0" />
-    </joint>
-    <link name="${robot_namespace}/wing_${suffix}">
-      <inertial>
-        <xacro:insert_block name="link_origin" />
-        <mass value="${mass_wing}" />
-        <xacro:insert_block name="inertia" />
-      </inertial>
-      <visual>
-        <xacro:insert_block name="link_origin" />
-        <geometry>
-          <xacro:if value="${use_mesh}">
-            <mesh filename="${mesh}"
-              scale="1 1 1" />
-          </xacro:if>
-          <xacro:unless value="${use_mesh}">
-            <box size="${wing_length} ${wing_width} ${wing_height}"/>
-          </xacro:unless>
-        </geometry>
-      </visual>
-      <collision>
-        <xacro:insert_block name="link_origin" />
-        <geometry>
-          <box size="${wing_length - 0.01} ${wing_width - 0.01} ${wing_height - 0.01}"/>
-        </geometry>
-      </collision>
-    </link>
-    <gazebo reference="${robot_namespace}/wing_${suffix}">
-      <material>Gazebo/${color}</material>
-    </gazebo>
-  </xacro:macro>-->
-  <!-- Tail joint and link -->
-  <xacro:macro name="tail"
-    params="robot_namespace parent mass_tail tail_length tail_width tail_height
-      color use_mesh mesh *origin *inertia">
-    <joint name="${robot_namespace}/tail_joint" type="revolute">
+  <!-- Vertical stabilizer joint and link -->
+  <xacro:macro name="vertical_stabilizer"
+    params="robot_namespace parent mass length width height color use_mesh mesh *origin *inertia">
+    <joint name="${robot_namespace}/vertical_stabilizer_joint" type="fixed">
       <xacro:insert_block name="origin" />
       <axis xyz="0 0 1" />
       <parent link="${parent}" />
-      <child link="${robot_namespace}/tail" />
+      <child link="${robot_namespace}/vertical_stabilizer" />
       <limit upper="0" lower="0" effort="0" velocity="0" />
     </joint>
-    <link name="${robot_namespace}/tail">
+    <link name="${robot_namespace}/vertical_stabilizer">
       <inertial>
         <origin xyz="0.0 0.0 0.0" rpy="0.0 0.0 0.0" />
-        <mass value="${mass_tail}" /> <!-- [kg] -->
+        <mass value="${mass}" />
         <xacro:insert_block name="inertia" />
       </inertial>
@@ -180,15 +137,15 @@
           </xacro:if>
           <xacro:unless value="${use_mesh}">
-            <box size="${tail_length} ${tail_width} ${tail_height}"/> <!-- [m] [m] [m] -->
-          </xacro:unless>
-        </geometry>
-      </visual>
-      <collision>
-        <geometry>
-          <box size="${tail_length} ${tail_width} ${tail_height}"/> <!-- [m] [m] [m] -->
-        </geometry>
-      </collision>
-    </link>
-    <gazebo reference="${robot_namespace}/tail">
+            <box size="${length} ${width} ${height}" />
+          </xacro:unless>
+        </geometry>
+      </visual>
+      <collision>
+        <geometry>
+          <box size="${length} ${width} ${height}" />
+        </geometry>
+      </collision>
+    </link>
+    <gazebo reference="${robot_namespace}/vertical_stabilizer">
       <material>Gazebo/${color}</material>
     </gazebo>
@@ -196,6 +153,6 @@
   <!-- Propeller joint and link -->
   <xacro:macro name="propeller"
-    params="robot_namespace direction motor_constant moment_constant parent mass_propeller
-      radius_propeller time_constant_up time_constant_down max_propeller_velocity motor_number
+    params="robot_namespace direction motor_constant moment_constant parent mass radius
+      time_constant_up time_constant_down max_propeller_velocity motor_number
       rotor_drag_coefficient rolling_moment_coefficient use_own_mesh mesh color *origin *inertia">
     <joint name="${robot_namespace}/propeller_joint" type="continuous">
@@ -208,5 +165,5 @@
       <inertial>
         <origin xyz="0.0 0.0 0.0" rpy="0.0 0.0 0.0" />
-        <mass value="${mass_propeller}" /> <!-- [kg] -->
+        <mass value="${mass_propeller}" />
         <xacro:insert_block name="inertia" />
       </inertial>
@@ -219,11 +176,11 @@
           <xacro:unless value="${use_own_mesh}">
             <mesh filename="package://rotors_description/meshes/propeller_${direction}.dae"
-              scale="${radius_propeller} ${radius_propeller} ${radius_propeller}" /> <!-- The propeller meshes have a radius of 1m -->
-          </xacro:unless>
-        </geometry>
-      </visual>
-      <collision>
-        <geometry>
-          <cylinder length="0.005" radius="0.1" /> <!-- [m] -->
+              scale="${radius_propeller} ${radius_propeller} ${radius_propeller}" />
+          </xacro:unless>
+        </geometry>
+      </visual>
+      <collision>
+        <geometry>
+          <cylinder length="0.005" radius="0.1" />
         </geometry>
       </collision>
@@ -252,61 +209,4 @@
     </gazebo>
   </xacro:macro>
-  <!-- Control surface joint and link -->
-<!--  <xacro:macro name="control_surface"
-    params="robot_namespace surface_name parent mass_surface gain
-      positive_direction min_angle max_angle channel color use_mesh mesh
-      surface_length surface_width surface_height *axis *joint_origin
-      *link_origin *inertia">
-    <joint name="${robot_namespace}/${surface_name}_joint" type="revolute">
-      <xacro:insert_block name="joint_origin" />
-      <xacro:insert_block name="axis" />
-      <parent link="${parent}" />
-      <child link="${robot_namespace}/${surface_name}" />
-      <limit upper="${max_angle}" lower="${min_angle}" effort="200.0" velocity="3.0" />
-      <dynamics friction="${9.8 * mass_surface}" damping="${9.8 * mass_surface}" />
-    </joint>
-    <link name="${robot_namespace}/${surface_name}">
-      <gravity>0</gravity>
-      <inertial>
-        <xacro:insert_block name="link_origin" />
-        <mass value="${mass_surface}" />
-        <xacro:insert_block name="inertia" />
-      </inertial>
-      <visual>
-        <xacro:insert_block name="link_origin" />
-        <geometry>
-          <xacro:if value="${use_mesh}">
-            <mesh filename="${mesh}"
-              scale="1 1 1" />
-          </xacro:if>
-          <xacro:unless value="${use_mesh}">
-            <box size="${surface_length} ${surface_width} ${surface_height}"/>
-          </xacro:unless>
-        </geometry>
-      </visual>
-      <collision>
-        <xacro:insert_block name="link_origin" />
-        <geometry>
-          <box size="${surface_length - 0.01} ${surface_width - 0.01} ${surface_height - 0.01}"/>
-        </geometry>
-      </collision>
-    </link>
-    <gazebo>
-      <plugin name="${robot_namespace}_${surface_name}_servo" filename="librotors_gazebo_servo_plugin.so">
-        <robotNamespace>${robot_namespace}</robotNamespace>
-        <jointName>${robot_namespace}/${surface_name}_joint</jointName>
-        <childLinkName>${robot_namespace}/${surface_name}</childLinkName>
-        <commandSubTopic>gazebo/command/motor_speed</commandSubTopic>
-        <positiveDirection>${positive_direction}</positiveDirection>
-        <gain>${gain}</gain>
-        <minAngle>${min_angle}</minAngle>
-        <maxAngle>${max_angle}</maxAngle>
-        <channel>${channel}</channel>
-      </plugin>
-    </gazebo>
-    <gazebo reference="${robot_namespace}/${surface_name}">
-      <material>Gazebo/${color}</material>
-    </gazebo>
-  </xacro:macro>-->
   <!-- Aerodynamic surface joint and link -->
   <xacro:macro name="aero_surface"
@@ -319,5 +219,5 @@
       <parent link="${parent}" />
       <child link="${robot_namespace}/${surface_name}" />
-      <limit upper="${max_angle}" lower="${min_angle}" effort="200.0" velocity="3.0" />
+      <limit upper="${max_angle}" lower="${min_angle}" effort="200.0" velocity="1.0" />
       <dynamics friction="${9.8 * mass_surface}" damping="${9.8 * mass_surface}" />
     </joint>
@@ -336,5 +236,5 @@
           </xacro:if>
           <xacro:unless value="${use_mesh}">
-            <box size="${surface_length} ${surface_width} ${surface_height}"/>
+            <box size="${surface_length} ${surface_width} ${surface_height}" />
           </xacro:unless>
         </geometry>
@@ -343,5 +243,5 @@
         <xacro:insert_block name="link_origin" />
         <geometry>
-          <box size="${surface_length - 0.01} ${surface_width - 0.01} ${surface_height - 0.01}"/>
+          <box size="${surface_length - 0.01} ${surface_width - 0.01} ${surface_height - 0.01}" />
         </geometry>
       </collision>

Commit message: Implementing the aerodynamics model

File: rotors_description/urdf/atlantik_solar.xacro (robot description, xacro)
@@ -22,4 +22,6 @@
   <xacro:property name="use_mesh_file" value="false" />
   <xacro:property name="mesh_file" value="" />
+  <!-- Constants -->
+  <xacro:property name="PI" value="3.1415926535897931" />
   <!-- Component masses -->
   <xacro:property name="mass_fuselage" value="2.0" /> <!-- [kg] -->
@@ -69,6 +71,6 @@
   <xacro:property name="aileron_height" value="0.02" /> <!-- [m] -->
   <xacro:property name="aileron_gain" value="2.0" />
-  <xacro:property name="aileron_min_angle" value="-0.55" /> <!-- [rad] -->
-  <xacro:property name="aileron_max_angle" value="0.55" /> <!-- [rad] -->
+  <xacro:property name="aileron_min_angle" value="-0.349066" /> <!-- [rad] -->
+  <xacro:property name="aileron_max_angle" value="0.349066" /> <!-- [rad] -->
   <xacro:property name="aileron_channel" value="0" />
   <!-- Elevator properties -->
@@ -77,6 +79,6 @@
   <xacro:property name="elevator_height" value="0.02" /> <!-- [m] -->
   <xacro:property name="elevator_gain" value="2.0" />
-  <xacro:property name="elevator_min_angle" value="-0.55" /> <!-- [rad] -->
-  <xacro:property name="elevator_max_angle" value="0.55" /> <!-- [rad] -->
+  <xacro:property name="elevator_min_angle" value="-0.349066" /> <!-- [rad] -->
+  <xacro:property name="elevator_max_angle" value="0.349066" /> <!-- [rad] -->
   <xacro:property name="elevator_channel" value="1" />
   <!-- Rudder properties -->
@@ -85,9 +87,7 @@
   <xacro:property name="rudder_height" value="${vertical_stabilizer_height}" /> <!-- [m] -->
   <xacro:property name="rudder_gain" value="2.0" />
-  <xacro:property name="rudder_min_angle" value="-0.55" /> <!-- [rad] -->
-  <xacro:property name="rudder_max_angle" value="0.55" /> <!-- [rad] -->
+  <xacro:property name="rudder_min_angle" value="-0.349066" /> <!-- [rad] -->
+  <xacro:property name="rudder_max_angle" value="0.349066" /> <!-- [rad] -->
   <xacro:property name="rudder_channel" value="2" />
-  <!-- Constants -->
-  <xacro:property name="PI" value="3.1415926535897931" />
   <!-- Front wing length -->
   <xacro:property name="wing_width" value="${0.5 * (wingspan - body_width)}" />
@@ -313,5 +313,5 @@
   </xacro:aero_surface>
   <!-- Instantiate the ailerons -->
-<!--  <xacro:aero_surface
+  <xacro:aero_surface
     robot_namespace="${namespace}"
     surface_name="aileron_left"
@@ -356,7 +356,7 @@
     <origin xyz="${-0.5 * aileron_length} 0.0 0.0" rpy="0.0 0.0 0.0" />
     <xacro:insert_block name="aileron_inertia" />
-  </xacro:aero_surface>-->
+  </xacro:aero_surface>
   <!-- Instantiate the elevators -->
-<!--  <xacro:aero_surface
+  <xacro:aero_surface
     robot_namespace="${namespace}"
     surface_name="elevator_left"
@@ -401,7 +401,7 @@
     <origin xyz="${-0.5 * elevator_length} 0.0 0.0" rpy="0.0 0.0 0.0" />
     <xacro:insert_block name="elevator_inertia" />
-  </xacro:aero_surface>-->
+  </xacro:aero_surface>
   <!-- Instantiate the rudder -->
-<!--  <xacro:aero_surface
+  <xacro:aero_surface
     robot_namespace="${namespace}"
     surface_name="rudder"
@@ -424,4 +424,4 @@
     <origin xyz="${-0.5 * rudder_length} 0.0 0.0" rpy="0.0 0.0 0.0" />
     <xacro:insert_block name="rudder_inertia" />
-  </xacro:aero_surface>-->
+  </xacro:aero_surface>
 </robot>
