Commit message: Implementing publishing of ground speed from GPS and wind speed from wind plugin

File: rotors_description/urdf/atlantik_solar.xacro (robot description, xacro)
@@ -25,9 +25,9 @@
   <xacro:property name="PI" value="3.1415926535897931" />
   <!-- Component masses -->
-  <xacro:property name="mass_fuselage" value="2.0" /> <!-- [kg] -->
+  <xacro:property name="mass_fuselage" value="1.2" /> <!-- [kg] -->
   <xacro:property name="mass_wheel" value="0.05" /> <!-- [kg] -->
-  <xacro:property name="mass_wing" value="0.5" /> <!-- [kg] -->
+  <xacro:property name="mass_wing" value="0.4" /> <!-- [kg] -->
   <xacro:property name="mass_vertical_stabilizer" value="0.2" /> <!-- [kg] -->
-  <xacro:property name="mass_tail" value="0.25" /> <!-- [kg] -->
+  <xacro:property name="mass_tail" value="0.15" /> <!-- [kg] -->
   <xacro:property name="mass_propeller" value="0.01" /> <!-- [kg] -->
   <xacro:property name="mass_aileron" value="0.2" /> <!-- [kg] -->
@@ -35,5 +35,5 @@
   <xacro:property name="mass_rudder" value="0.1" /> <!-- [kg] -->
   <!-- Fuselage properties -->
-  <xacro:property name="body_length" value="3.0" /> <!-- [m] -->
+  <xacro:property name="body_length" value="2.0" /> <!-- [m] -->
   <xacro:property name="body_width" value="0.1" /> <!-- [m] -->
   <xacro:property name="body_height" value="0.1" /> <!-- [m] -->
@@ -53,6 +53,6 @@
   <xacro:property name="rolling_moment_coefficient" value="0.000001" />
   <!-- Wing properties -->
-  <xacro:property name="wingspan" value="4.0" /> <!-- [m] -->
-  <xacro:property name="root_chord" value="0.3" /> <!-- [m] -->
+  <xacro:property name="wingspan" value="2.59" /> <!-- [m] -->
+  <xacro:property name="root_chord" value="0.18" /> <!-- [m] -->
   <xacro:property name="wing_height" value="0.02" /> <!-- [m] -->
   <xacro:property name="tail_wingspan" value="1.0" /> <!-- [m] -->
@@ -61,7 +61,7 @@
   <xacro:property name="alpha_stall" value="0.2" /> <!-- [rad] -->
   <xacro:property name="c_L_alpha" value="3.0" />
-  <xacro:property name="air_density" value="1.225" /> <!-- [kg/m^3] -->
+  <xacro:property name="air_density" value="1.18" /> <!-- [kg/m^3] -->
   <!-- Tail properties -->
-  <xacro:property name="vertical_stabilizer_length" value="0.4" /> <!-- [m] -->
+  <xacro:property name="vertical_stabilizer_length" value="0.3" /> <!-- [m] -->
   <xacro:property name="vertical_stabilizer_width" value="0.05" /> <!-- [m] -->
   <xacro:property name="vertical_stabilizer_height" value="0.2" /> <!-- [m] -->
@@ -145,5 +145,7 @@
     air_density="${air_density}"
     alpha_stall="${alpha_stall}">
-    <xacro:insert_block name="body_inertia" />
+    <origin xyz="0.45 0 0" rpy="0 0 0" />
+    <inertia ixx="${0.1512 * 1.1}" ixy="0.0" ixz="0.0755" iyy="${0.2785 * 1.4}" iyz="0.0" izz="${0.3745 * 1.4}" />
+    <!--<xacro:insert_block name="body_inertia" />-->
   </xacro:fixed_wing_base_macro>
   <!-- Instantiate the propeller -->
@@ -153,5 +155,5 @@
     motor_constant="${motor_constant}"
     moment_constant="${moment_constant}"
-    parent="${namespace}/base_link_inertia"
+    parent="${namespace}/base_link"
     mass="${mass_propeller}"
     radius="${radius_propeller}"
@@ -172,5 +174,5 @@
     robot_namespace="${namespace}"
     suffix="front_left"
-    parent="${namespace}/base_link_inertia"
+    parent="${namespace}/base_link"
     mass="${mass_wheel}"
     color="${body_color}"
@@ -185,5 +187,5 @@
     robot_namespace="${namespace}"
     suffix="front_right"
-    parent="${namespace}/base_link_inertia"
+    parent="${namespace}/base_link"
     mass="${mass_wheel}"
     color="${body_color}"
@@ -198,5 +200,5 @@
     robot_namespace="${namespace}"
     suffix="back"
-    parent="${namespace}/base_link_inertia"
+    parent="${namespace}/base_link"
     mass="${mass_wheel}"
     color="${body_color}"
@@ -205,5 +207,5 @@
     radius="${wheel_radius}"
     width="${wheel_width}">
-    <origin xyz="-1.0 0.0 -0.1" rpy="${0.5 * PI} 0.0 0.0" />
+    <origin xyz="-0.5 0.0 -0.1" rpy="${0.5 * PI} 0.0 0.0" />
     <xacro:insert_block name="wheel_inertia" />
   </xacro:wheel>
@@ -213,5 +215,5 @@
     surface_name="wing_left"
     surface_type="wing"
-    parent="${namespace}/base_link_inertia"
+    parent="${namespace}/base_link"
     mass_surface="${mass_wing}"
     joint_gain="0.0"
@@ -235,5 +237,5 @@
     surface_name="wing_right"
     surface_type="wing"
-    parent="${namespace}/base_link_inertia"
+    parent="${namespace}/base_link"
     mass_surface="${mass_wing}"
     joint_gain="0.0"
@@ -256,5 +258,5 @@
   <xacro:vertical_stabilizer
     robot_namespace="${namespace}"
-    parent="${namespace}/base_link_inertia"
+    parent="${namespace}/base_link"
     mass="${mass_vertical_stabilizer}"
     length="${vertical_stabilizer_length}"
@@ -267,5 +269,5 @@
     <xacro:insert_block name="vertical_stabilizer_inertia" />
   </xacro:vertical_stabilizer>
-  <!-- Instantiate the rear wings-->
+  <!-- Instantiate the tail -->
   <xacro:aero_surface
     robot_namespace="${namespace}"
@@ -313,5 +315,5 @@
   </xacro:aero_surface>
   <!-- Instantiate the ailerons -->
-  <xacro:aero_surface
+<!--  <xacro:aero_surface
     robot_namespace="${namespace}"
     surface_name="aileron_left"
@@ -356,7 +358,7 @@
     <origin xyz="${-0.5 * aileron_length} 0.0 0.0" rpy="0.0 0.0 0.0" />
     <xacro:insert_block name="aileron_inertia" />
-  </xacro:aero_surface>
+  </xacro:aero_surface>-->
   <!-- Instantiate the elevators -->
-  <xacro:aero_surface
+<!--  <xacro:aero_surface
     robot_namespace="${namespace}"
     surface_name="elevator_left"
@@ -401,7 +403,7 @@
     <origin xyz="${-0.5 * elevator_length} 0.0 0.0" rpy="0.0 0.0 0.0" />
     <xacro:insert_block name="elevator_inertia" />
-  </xacro:aero_surface>
+  </xacro:aero_surface>-->
   <!-- Instantiate the rudder -->
-  <xacro:aero_surface
+<!--  <xacro:aero_surface
     robot_namespace="${namespace}"
     surface_name="rudder"
@@ -424,4 +426,4 @@
     <origin xyz="${-0.5 * rudder_length} 0.0 0.0" rpy="0.0 0.0 0.0" />
     <xacro:insert_block name="rudder_inertia" />
-  </xacro:aero_surface>
+  </xacro:aero_surface>-->
 </robot>

File: rotors_description/urdf/component_snippets.xacro (robot description, xacro)
@@ -345,5 +345,5 @@
     params="namespace xyz_offset wind_direction wind_force_mean
       wind_gust_direction wind_gust_duration wind_gust_start
-      wind_gust_force_mean">
+      wind_gust_force_mean object_drag_coefficient">
     <gazebo>
       <plugin filename="librotors_gazebo_wind_plugin.so" name="wind_plugin">
@@ -358,4 +358,5 @@
         <windGustStart>${wind_gust_start}</windGustStart> <!-- [s] -->
         <windGustForceMean>${wind_gust_force_mean}</windGustForceMean> <!-- [N] -->
+        <objectDragCoefficient>${object_drag_coefficient}</objectDragCoefficient>
       </plugin>
     </gazebo>
@@ -363,6 +364,6 @@
   <!-- Macro to add a GPS sensor. -->
   <xacro:macro name="gps_plugin_macro"
-    params="namespace gps_suffix parent_link gps_topic mass_gps_sensor
-      reference_latitude reference_longitude reference_altitude
+    params="namespace gps_suffix parent_link gps_topic ground_speed_topic
+      mass_gps_sensor reference_latitude reference_longitude reference_altitude
       reference_heading noise_normal_position noise_uniform_position
       *inertia *origin">
@@ -387,4 +388,5 @@
       <linkName>${namespace}/gps${gps_suffix}_link</linkName> <!-- (string, required): name of the body which holds the GPS sensor -->
       <gpsTopic>${gps_topic}</gpsTopic> <!-- (string): name of the sensor output topic and prefix of service names (defaults to 'gps') -->
+      <groundSpeedTopic>${ground_speed_topic}</groundSpeedTopic> <!-- (string): name of the ground speed output topic (defaults to 'ground_speed') -->
       <referenceLatitude>${reference_latitude}</referenceLatitude> <!-- the initial latitude [degrees [-90, 90]] -->
       <referenceLongitude>${reference_longitude}</referenceLongitude> <!-- the initial longitude [degrees [-180, 180]] -->
@@ -748,4 +750,5 @@
       parent_link="${parent_link}"
       gps_topic="gps"
+      ground_speed_topic="ground_speed"
       mass_gps_sensor="0.015"
       reference_latitude="47.3667"

File: rotors_description/urdf/fixed_wing_base.xacro (robot description, xacro)
@@ -32,16 +32,15 @@
   <xacro:macro name="fixed_wing_base_macro"
     params="robot_namespace mass length width height color use_mesh_file
-      mesh_file reset_topic air_density alpha_stall *inertia">
-<!--    <link name="${robot_namespace}/base_link"></link>
+      mesh_file reset_topic air_density alpha_stall *cog *inertia">
+    <link name="${robot_namespace}/base_link"></link>
     <joint name="${robot_namespace}/base_joint" type="fixed">
-      <origin xyz="0 0 0.1" rpy="0 0 0" />
+      <origin xyz="0 0 0.0" rpy="0 0 0" />
       <parent link="${robot_namespace}/base_link" />
       <child link="${robot_namespace}/base_link_inertia" />
     </joint>-->
     <link name="${robot_namespace}/base_link_inertia">
-      <pose>0 0 0 0 0 0</pose>
       <inertial>
         <mass value="${mass}" />
-        <origin xyz="0.0 0 0" rpy="0 0 0" />
+        <xacro:insert_block name="cog" />
         <xacro:insert_block name="inertia" />
       </inertial>
@@ -67,5 +66,5 @@
       <plugin name="${robot_namespace}_base" filename="librotors_gazebo_fixedwing_base_plugin.so">
         <robotNamespace>${robot_namespace}</robotNamespace>
-        <linkName>${robot_namespace}/base_link_inertia</linkName>
+        <linkName>${robot_namespace}/base_link</linkName>
 	<resetTopic>${reset_topic}</resetTopic>
 	<airDensity>${air_density}</airDensity>
@@ -73,5 +72,5 @@
       </plugin>
     </gazebo>
-    <gazebo reference="${robot_namespace}/base_link_inertia">
+    <gazebo reference="${robot_namespace}/base_link">
       <material>Gazebo/${color}</material>
     </gazebo>
@@ -214,10 +213,11 @@
       positive_direction channel min_angle max_angle color use_mesh mesh surface_length
       surface_width surface_height *axis *joint_origin *link_origin *inertia">
-    <joint name="${robot_namespace}/${surface_name}_joint" type="revolute">
+    <joint name="${robot_namespace}/${surface_name}_joint" type="fixed">
       <xacro:insert_block name="joint_origin" />
       <xacro:insert_block name="axis" />
       <parent link="${parent}" />
       <child link="${robot_namespace}/${surface_name}" />
-      <limit upper="${max_angle}" lower="${min_angle}" effort="200.0" velocity="1.0" />
+      <limit upper="0" lower="0" effort="0" velocity="0" />
+      <!--<limit upper="${max_angle}" lower="${min_angle}" effort="200.0" velocity="1.0" />-->
       <dynamics friction="${9.8 * mass_surface}" damping="${9.8 * mass_surface}" />
     </joint>
@@ -247,5 +247,5 @@
       </collision>
     </link>
-    <gazebo>
+<!--    <gazebo>
       <plugin name="${robot_namespace}_${surface_name}" filename="librotors_gazebo_aero_surface_plugin.so">
         <robotNamespace>${robot_namespace}</robotNamespace>
@@ -260,5 +260,5 @@
         <maxAngle>${max_angle}</maxAngle>
       </plugin>
-    </gazebo>
+    </gazebo>-->
     <gazebo reference="${robot_namespace}/${surface_name}">
       <material>Gazebo/${color}</material>

Commit message: Adding air speed to the fixed wing base plugin

File: rotors_description/urdf/atlantik_solar.xacro (robot description, xacro)
@@ -25,7 +25,7 @@
   <xacro:property name="PI" value="3.1415926535897931" />
   <!-- Component masses -->
-  <xacro:property name="mass_fuselage" value="1.2" /> <!-- [kg] -->
+  <xacro:property name="mass_fuselage" value="2.0" /> <!-- [kg] -->
   <xacro:property name="mass_wheel" value="0.05" /> <!-- [kg] -->
-  <xacro:property name="mass_wing" value="0.4" /> <!-- [kg] -->
+  <xacro:property name="mass_wing" value="0.5" /> <!-- [kg] -->
   <xacro:property name="mass_vertical_stabilizer" value="0.2" /> <!-- [kg] -->
   <xacro:property name="mass_tail" value="0.15" /> <!-- [kg] -->
@@ -63,5 +63,5 @@
   <xacro:property name="air_density" value="1.18" /> <!-- [kg/m^3] -->
   <!-- Tail properties -->
-  <xacro:property name="vertical_stabilizer_length" value="0.3" /> <!-- [m] -->
+  <xacro:property name="vertical_stabilizer_length" value="0.2" /> <!-- [m] -->
   <xacro:property name="vertical_stabilizer_width" value="0.05" /> <!-- [m] -->
   <xacro:property name="vertical_stabilizer_height" value="0.2" /> <!-- [m] -->
@@ -75,5 +75,5 @@
   <xacro:property name="aileron_channel" value="0" />
   <!-- Elevator properties -->
-  <xacro:property name="elevator_length" value="0.15" /> <!-- [m] -->
+  <xacro:property name="elevator_length" value="0.0" /> <!-- [m] -->
   <xacro:property name="elevator_width" value="${tail_width}" /> <!-- [m] -->
   <xacro:property name="elevator_height" value="0.02" /> <!-- [m] -->
@@ -145,10 +145,10 @@
     air_density="${air_density}"
     alpha_stall="${alpha_stall}">
-    <origin xyz="0.45 0 0" rpy="0 0 0" />
+    <origin xyz="0 0 0" rpy="0 0 0" />
     <inertia ixx="${0.1512 * 1.1}" ixy="0.0" ixz="0.0755" iyy="${0.2785 * 1.4}" iyz="0.0" izz="${0.3745 * 1.4}" />
     <!--<xacro:insert_block name="body_inertia" />-->
   </xacro:fixed_wing_base_macro>
   <!-- Instantiate the propeller -->
-  <xacro:propeller
+<!--  <xacro:propeller
     robot_namespace="${namespace}"
     direction="cw"
@@ -169,7 +169,7 @@
     <origin xyz="${0.5 * body_length + propeller_offset} 0.0 0.0" rpy="0.0 ${0.5 * PI} 0.0" />
     <xacro:insert_block name="propeller_inertia" />
-  </xacro:propeller>
+  </xacro:propeller>-->
   <!-- Instantiate wheels -->
-  <xacro:wheel
+<!--  <xacro:wheel
     robot_namespace="${namespace}"
     suffix="front_left"
@@ -209,5 +209,5 @@
     <origin xyz="-0.5 0.0 -0.1" rpy="${0.5 * PI} 0.0 0.0" />
     <xacro:insert_block name="wheel_inertia" />
-  </xacro:wheel>
+  </xacro:wheel>-->
   <!-- Instantiate wings -->
   <xacro:aero_surface

Commit message: Stable straight flight code

File: rotors_description/urdf/atlantik_solar.xacro (robot description, xacro)
@@ -229,6 +229,6 @@
     mesh="">
     <axis xyz="1 0 0" />
-    <origin xyz="0.5 ${0.5 * body_width} 0.0" rpy="0.0 0.0 0.0" />
-    <origin xyz="0.0 ${0.5 * wing_width} 0.0" rpy="0.0 0.0 0.0" />
+    <origin xyz="0.5 ${-0.5 * body_width} 0.0" rpy="0.0 0.0 0.0" />
+    <origin xyz="0.0 ${-0.5 * wing_width} 0.0" rpy="0.0 0.0 0.0" />
     <xacro:insert_block name="wing_inertia" />
   </xacro:aero_surface>
@@ -251,6 +251,6 @@
     mesh="">
     <axis xyz="1 0 0" />
-    <origin xyz="0.5 ${-0.5 * body_width} 0.0" rpy="0.0 0.0 0.0" />
-    <origin xyz="0.0 ${-0.5 * wing_width} 0.0" rpy="0.0 0.0 0.0" />
+    <origin xyz="0.5 ${0.5 * body_width} 0.0" rpy="0.0 0.0 0.0" />
+    <origin xyz="0.0 ${0.5 * wing_width} 0.0" rpy="0.0 0.0 0.0" />
     <xacro:insert_block name="wing_inertia" />
   </xacro:aero_surface>
@@ -266,5 +266,5 @@
     use_mesh="false"
     mesh="">
-    <origin xyz="${-0.5*body_length + 0.5*vertical_stabilizer_length} 0.0 ${0.5*body_height + 0.5*vertical_stabilizer_height}" rpy="0.0 0.0 0.0" />
+    <origin xyz="${-0.5 * body_length + 0.5 * vertical_stabilizer_length} 0.0 ${-0.5 * (body_height + vertical_stabilizer_height)}" rpy="0.0 0.0 0.0" />
     <xacro:insert_block name="vertical_stabilizer_inertia" />
   </xacro:vertical_stabilizer>
@@ -288,6 +288,6 @@
     mesh="">
     <axis xyz="1 0 0" />
-    <origin xyz="${0.5 * elevator_length} ${0.5 * vertical_stabilizer_width} ${0.5 * (vertical_stabilizer_height - tail_height)}" rpy="0.0 0.0 0.0" />
-    <origin xyz="0.0 ${0.5 * tail_width} 0.0" rpy="0.0 0.0 0.0" />
+    <origin xyz="${0.5 * elevator_length} ${-0.5 * vertical_stabilizer_width} ${-0.5 * (vertical_stabilizer_height - tail_height)}" rpy="0.0 0.0 0.0" />
+    <origin xyz="0.0 ${-0.5 * tail_width} 0.0" rpy="0.0 0.0 0.0" />
     <xacro:insert_block name="tail_inertia" />
   </xacro:aero_surface>
@@ -310,6 +310,6 @@
     mesh="">
     <axis xyz="1 0 0" />
-    <origin xyz="${0.5 * elevator_length} ${-0.5 * vertical_stabilizer_width} ${0.5 * (vertical_stabilizer_height - tail_height)}" rpy="0.0 0.0 0.0" />
-    <origin xyz="0.0 ${-0.5 * tail_width} 0.0" rpy="0.0 0.0 0.0" />
+    <origin xyz="${0.5 * elevator_length} ${0.5 * vertical_stabilizer_width} ${-0.5 * (vertical_stabilizer_height - tail_height)}" rpy="0.0 0.0 0.0" />
+    <origin xyz="0.0 ${0.5 * tail_width} 0.0" rpy="0.0 0.0 0.0" />
     <xacro:insert_block name="tail_inertia" />
   </xacro:aero_surface>

File: rotors_description/urdf/fixed_wing_base.xacro (robot description, xacro)
@@ -38,5 +38,5 @@
       <parent link="${robot_namespace}/base_link" />
       <child link="${robot_namespace}/base_link_inertia" />
-    </joint>-->
+    </joint>
     <link name="${robot_namespace}/base_link_inertia">
       <inertial>
