Commit message: Renaming fixed_wing model to Techpod and adding parameter files

File: rotors_description/urdf/techpod.xacro (robot description, xacro)
@@ -16,7 +16,7 @@
   limitations under the License.
 -->
-<robot name="atlantik_solar" xmlns:xacro="http://ros.org/wiki/xacro">
+<robot name="techpod" xmlns:xacro="http://ros.org/wiki/xacro">
   <!-- Global properties -->
-  <xacro:property name="namespace" value="$(arg mav_name)" />
+  <xacro:property name="namespace" value="$(arg uav_name)" />
   <xacro:property name="propeller_velocity_slowdown_sim" value="10" />
   <xacro:property name="use_mesh_file" value="false" />

File: rotors_description/urdf/techpod_base.xacro (robot description, xacro)
@@ -16,8 +16,8 @@
   limitations under the License.
 -->
-<robot name="atlantik_solar" xmlns:xacro="http://ros.org/wiki/xacro">
+<robot name="techpod" xmlns:xacro="http://ros.org/wiki/xacro">
   <xacro:include filename="$(find rotors_description)/urdf/component_snippets.xacro" />
   <!-- Instantiate fixed wing "mechanics" -->
-  <xacro:include filename="$(find rotors_description)/urdf/atlantik_solar.xacro" />
+  <xacro:include filename="$(find rotors_description)/urdf/techpod.xacro" />
   <!-- Instantiate a controller. -->
   <xacro:controller_plugin_macro namespace="${namespace}" imu_sub_topic="imu" />

Commit message: Adding the functionality of rebooting the autopilot to the GUI

File: rotors_description/urdf/techpod.xacro (robot description, xacro)
@@ -145,5 +145,5 @@
     use_mesh_file="${use_mesh_file}"
     mesh_file="${mesh_file}"
-    reset_topic="reset"
+    reset_topic="reset_model"
     air_density="${air_density}"
     alpha_stall="${alpha_stall}">

File: rotors_description/urdf/techpod_base.xacro (robot description, xacro)
@@ -33,9 +33,9 @@
   <xacro:default_air_speed_sensor namespace="${namespace}" parent_link="${namespace}/base_link" />
   <!-- Mount a downward-looking camera. -->
-<!--  <xacro:camera_macro
+  <xacro:camera_macro
     namespace="${namespace}"
     parent_link="${namespace}/base_link_inertia"
     camera_suffix="downward"
-    frame_rate="10.0"
+    frame_rate="35.0"
     horizontal_fov="1.3962634"
     image_width="752"
@@ -48,6 +48,6 @@
     enable_visual="false">
     <mesh filename="package://rotors_description/meshes/vi_camera.dae" scale="1 1 1" />
-    <origin xyz="0 0 -0.05" rpy="0 1.5707 0" />
-  </xacro:camera_macro>-->
+    <origin xyz="0 0 0" rpy="0 1.5707 0" />
+  </xacro:camera_macro>
   <xacro:if value="$(arg enable_ground_truth)">
     <xacro:ground_truth_imu_and_odometry namespace="${namespace}" parent_link="${namespace}/base_link_inertia" />

Commit message: Adding a test environment for kiki

File: rotors_description/urdf/techpod.xacro (robot description, xacro)
@@ -15,5 +15,5 @@
   <!-- Global properties -->
   <xacro:property name="namespace" value="$(arg uav_name)" />
-  <!--<xacro:property name="propeller_velocity_slowdown_sim" value="10" />-->
+  <xacro:property name="propeller_velocity_slowdown_sim" value="10" />
   <xacro:property name="use_mesh" value="true" />
   <!-- Constants -->
@@ -30,9 +30,6 @@
   <xacro:property name="mass_rudder" value="0.1" /> <!-- [kg] -->
   <!-- Fuselage properties -->
-  <xacro:property name="body_length" value="2.0" /> <!-- [m] -->
-  <xacro:property name="body_width" value="0.1" /> <!-- [m] -->
-  <xacro:property name="body_height" value="0.1" /> <!-- [m] -->
   <xacro:property name="body_length" value="1.33" /> <!-- [m] -->
-  <xacro:property name="body_width" value="0.85" /> <!-- [m] -->
+  <xacro:property name="body_width" value="2.65" /> <!-- [m] -->
   <xacro:property name="body_height" value="0.25" /> <!-- [m] -->
   <xacro:property name="body_color" value="Gray" />
@@ -48,5 +45,5 @@
   <xacro:property name="rolling_moment_coefficient" value="0.000001" />
   <!-- Aileron properties -->
-  <!--<xacro:property name="aileron_length" value="${0.5 * root_chord}" />
+  <xacro:property name="aileron_length" value="${0.5 * root_chord}" />
   <xacro:property name="aileron_width" value="${0.5 * wing_width}" />
   <xacro:property name="aileron_height" value="0.02" />
@@ -54,5 +51,5 @@
   <xacro:property name="aileron_min_angle" value="-0.349066" />
   <xacro:property name="aileron_max_angle" value="0.349066" />
-  <xacro:property name="aileron_channel" value="0" />-->
+  <xacro:property name="aileron_channel" value="0" />
   <!-- Elevator properties -->
   <xacro:property name="elevator_length" value="0.1" />
@@ -175,5 +172,5 @@
   </xacro:aero_surface>-->
   <!-- Instantiate the elevators -->
-  <xacro:aero_surface
+  <!--<xacro:aero_surface
     robot_namespace="${namespace}"
     surface_name="elevator"
@@ -196,5 +193,5 @@
     <origin xyz="0.0 0.0 0.0" rpy="${PI} 0.0 0.0" />
     <xacro:insert_block name="elevator_inertia" />
-  </xacro:aero_surface>
+  </xacro:aero_surface>-->
   <!-- Instantiate the rudder -->
   <!--<xacro:aero_surface

Commit message: Fixing the new aerodynamic model

File: rotors_description/urdf/techpod.xacro (robot description, xacro)
@@ -20,5 +20,5 @@
   <xacro:property name="PI" value="3.1415926535897931" />
   <!-- Component masses -->
-  <xacro:property name="mass_fuselage" value="1.25" /> <!-- [kg] -->
+  <xacro:property name="mass_fuselage" value="1.85" /> <!-- [kg] -->
   <xacro:property name="mass_aileron" value="0.1" /> <!-- [kg] -->
   <xacro:property name="mass_flap" value="0.1" /> <!-- [kg] -->
@@ -66,6 +66,6 @@
   <!-- Inertia of the main body -->
   <xacro:property name="body_inertia">
-    <!--<inertia ixx="0.16632" ixy="0.0" ixz="0.0755" iyy="0.3899" iyz="0.0" izz="0.5243" />-->
-    <inertia ixx="0.1512" ixy="0.0" ixz="0.0755" iyy="0.2785" iyz="0.0" izz="0.3745" />
+    <inertia ixx="0.16632" ixy="0.0" ixz="0.0755" iyy="0.3899" iyz="0.0" izz="0.5243" />
+    <!--<inertia ixx="0.1512" ixy="0.0" ixz="0.0755" iyy="0.2785" iyz="0.0" izz="0.3745" />-->
   </xacro:property>
   <!-- Inertia of the aileron, assuming it is a cuboid -->
