Commit message: Adding a GPS plug-in

File: rotors_description/urdf/component_snippets.xacro (robot description, xacro)
@@ -369,4 +369,39 @@
       </plugin>
     </gazebo>
+  </xacro:macro>
+  <!-- Macro to add a GPS sensor. -->
+  <xacro:macro name="gps_plugin_macro"
+    params="namespace gps_suffix parent_link gps_topic mass_gps_sensor
+      reference_latitude reference_longitude reference_altitude
+      reference_heading noise_normal_position noise_uniform_position
+      *inertia *origin">
+  <!-- GPS link -->
+  <link name="${namespace}/gps${gps_suffix}_link">
+    <inertial>
+      <xacro:insert_block name="inertia" />
+      <mass value="${mass_gps_sensor}" />  <!-- [kg] -->
+      <origin xyz="0 0 0" rpy="0 0 0" />
+    </inertial>
+  </link>
+  <!-- GPS joint -->
+  <joint name="${namespace}/gps${gps_suffix}_link" type="revolute">
+    <xacro:insert_block name="origin" />
+    <parent link="${parent_link}" />
+    <child link="${namespace}/gps${gps_suffix}_link" />
+    <limit upper="0" lower="0" effort="0" velocity="0" />
+  </joint>
+  <gazebo>
+    <plugin filename="librotors_gazebo_gps_plugin.so" name="rotors_gazebo_gps${gps_suffix}_plugin">
+      <robotNamespace>${namespace}</robotNamespace> <!-- (string, required): ros namespace in which the messages are published -->
+      <linkName>${namespace}/gps${gps_suffix}_link</linkName> <!-- (string, required): name of the body which holds the GPS sensor -->
+      <gpsTopic>${gps_topic}</gpsTopic> <!-- (string): name of the sensor output topic and prefix of service names (defaults to 'gps') -->
+      <referenceLatitude>${reference_latitude}</referenceLatitude> <!-- the initial latitude [degrees [-90, 90]] -->
+      <referenceLongitude>${reference_longitude}</referenceLongitude> <!-- the initial longitude [degrees [-180, 180]] -->
+      <referenceAltitude>${reference_altitude}</referenceAltitude> <!-- the initial altitude [m] -->
+      <referenceHeading>${reference_heading}</referenceHeading> <!-- the initial degrees, measured from North [deg] -->
+      <noiseNormalPosition>${noise_normal_position}</noiseNormalPosition> <!-- standard deviation of additive white gaussian noise [m] -->
+      <noiseUniformPosition>${noise_uniform_position}</noiseUniformPosition> <!-- symmetric bounds of uniform noise [m] -->
+    </plugin>
+  </gazebo>
   </xacro:macro>
   <!-- VI sensor macros -->
@@ -650,3 +685,20 @@
     </xacro:imu_plugin_macro>
   </xacro:macro>
+  <xacro:macro name="default_gps" params="namespace parent_link">
+    <xacro:gps_plugin_macro
+      namespace="${namespace}"
+      gps_suffix=""
+      parent_link="${parent_link}"
+      gps_topic="gps"
+      mass_gps_sensor="0.015"
+      reference_latitude="47.3667"
+      reference_longitude="8.5500"
+      reference_altitude="500.0"
+      reference_heading="0.0"
+      noise_normal_position="0 0 0"
+      noise_uniform_position="0 0 0">
+      <inertia ixx="0.00001" ixy="0.0" ixz="0.0" iyy="0.00001" iyz="0.0" izz="0.00001" />
+      <origin xyz="0 0 0" rpy="0 0 0" />
+    </xacro:gps_plugin_macro>
+  </xacro:macro>
 </robot>

Commit message: Adding a magnetometer plugin and removing the mavlink plugin

File: rotors_description/urdf/component_snippets.xacro (robot description, xacro)
@@ -245,14 +245,4 @@
     </gazebo>
   </xacro:macro>
-  <!-- Macro to add the mavlink interface. -->
-  <xacro:macro name="mavlink_interface_macro" params="namespace imu_sub_topic">
-    <gazebo>
-      <plugin name="mavlink_interface" filename="librotors_gazebo_mavlink_interface.so">
-        <robotNamespace>${namespace}</robotNamespace>
-        <imuSubTopic>${imu_sub_topic}</imuSubTopic>
-        <motorSpeedCommandPubTopic>gazebo/command/motor_speed</motorSpeedCommandPubTopic>
-      </plugin>
-    </gazebo>
-  </xacro:macro>
   <!-- Macro to add an IMU. -->
   <xacro:macro name="imu_plugin_macro"
@@ -402,4 +392,39 @@
       <noiseNormalPosition>${noise_normal_position}</noiseNormalPosition> <!-- standard deviation of additive white gaussian noise [m] -->
       <noiseUniformPosition>${noise_uniform_position}</noiseUniformPosition> <!-- symmetric bounds of uniform noise [m] -->
+    </plugin>
+  </gazebo>
+  </xacro:macro>
+  <!-- Macro to add a magnetometer sensor. -->
+  <xacro:macro name="magnetometer_plugin_macro"
+    params="namespace magnetometer_suffix parent_link magnetometer_topic mass_magnetometer
+      reference_magnetic_field_north reference_magnetic_field_east reference_magnetic_field_down
+      *inertia *origin">
+  <!-- Magnetometer link -->
+  <link name="${namespace}/magnetometer${magnetometer_suffix}_link">
+    <inertial>
+      <xacro:insert_block name="inertia" />
+      <mass value="${mass_magnetometer}" />  <!-- [kg] -->
+      <origin xyz="0 0 0" rpy="0 0 0" />
+    </inertial>
+  </link>
+  <!-- Magnetometer joint -->
+  <joint name="${namespace}/magnetometer${magnetometer_suffix}_link" type="revolute">
+    <xacro:insert_block name="origin" />
+    <parent link="${parent_link}" />
+    <child link="${namespace}/magnetometer${magnetometer_suffix}_link" />
+    <limit upper="0" lower="0" effort="0" velocity="0" />
+  </joint>
+  <gazebo>
+    <plugin filename="librotors_gazebo_magnetometer_plugin.so" name="rotors_gazebo_magnetometer${magnetometer_suffix}_plugin">
+      <robotNamespace>${namespace}</robotNamespace> <!-- (string, required): ros namespace in which the messages are published -->
+      <linkName>${namespace}/magnetometer${magnetometer_suffix}_link</linkName> <!-- (string, required): name of the body which holds the magnetometer -->
+      <magnetometerTopic>${magnetometer_topic}</magnetometerTopic> <!-- (string): name of the sensor output topic and prefix of service names (defaults to 'magnetic_field') -->
+      <!-- [Tesla] Below are the North, East, and Down components of the Earth's magnetic field at the reference location.
+           The default reference location is Zurich (lat=+47.3667degN, lon=+8.5500degE, h=+500m, WGS84).
+	   You can obtain the magnetic field strength for your location using the World Magnetic Model:
+           https://www.ngdc.noaa.gov/geomag/WMM/calculators.shtml -->
+      <referenceMagNorth>${reference_magnetic_field_north}</referenceMagNorth>
+      <referenceMagEast>${reference_magnetic_field_east}</referenceMagEast>
+      <referenceMagDown>${reference_magnetic_field_down}</referenceMagDown>
     </plugin>
   </gazebo>
@@ -702,3 +727,17 @@
     </xacro:gps_plugin_macro>
   </xacro:macro>
+  <xacro:macro name="default_magnetometer" params="namespace parent_link">
+    <xacro:magnetometer_plugin_macro
+      namespace="${namespace}"
+      magnetometer_suffix=""
+      parent_link="${parent_link}"
+      magnetometer_topic="magnetic_field"
+      mass_magnetometer="0.015"
+      reference_magnetic_field_north="0.000021475"
+      reference_magnetic_field_east="0.000000797"
+      reference_magnetic_field_down="0.000042817">
+      <inertia ixx="0.00001" ixy="0.0" ixz="0.0" iyy="0.00001" iyz="0.0" izz="0.00001" />
+      <origin xyz="0 0 0" rpy="0 0 0" />
+    </xacro:magnetometer_plugin_macro>
+  </xacro:macro>
 </robot>

Commit message: Adding a single-ray laser sensor for measuring height from ground

File: rotors_description/urdf/component_snippets.xacro (robot description, xacro)
@@ -493,4 +493,49 @@
         <windSpeedTopic>${wind_speed_topic}</windSpeedTopic> <!-- (string): name of the topic for receiving wind speed data -->
       </plugin>
+    </gazebo>
+  </xacro:macro>
+  <!-- Macro to add a laser sensor. -->
+  <xacro:macro name="laser_sensor_plugin_macro"
+    params="namespace parent_link laser_suffix *origin">
+    <!-- Laser sensor link -->
+    <link name="${namespace}/laser_${laser_suffix}_link">
+      <inertial>
+        <mass value="1e-5" />
+        <origin xyz="0 0 0" rpy="0 0 0" />
+        <inertia ixx="1e-6" ixy="0" ixz="0" iyy="1e-6" iyz="0" izz="1e-6" />
+      </inertial>
+    </link>
+    <!-- Laser sensor joint -->
+    <joint name="${namespace}/laser_${laser_suffix}_joint" type="revolute">
+      <xacro:insert_block name="origin" />
+      <parent link="${parent_link}" />
+      <child link="${namespace}/laser_${laser_suffix}_link" />
+      <limit upper="0" lower="0" effort="0" velocity="0" />
+    </joint>
+    <gazebo reference="${namespace}/laser_${laser_suffix}_link">
+      <sensor type="ray" name="laser_1">
+	<pose>0 0 0 0 0 0</pose>
+        <update_rate>30.0</update_rate>
+	<visualize>false</visualize>
+        <ray>
+          <scan>
+            <horizontal>
+              <samples>1</samples>
+              <resolution>1</resolution>
+              <min_angle>0</min_angle>
+              <max_angle>0</max_angle>
+            </horizontal>
+          </scan>
+          <range>
+            <min>0.3</min>
+            <max>300.0</max>
+            <resolution>0.1</resolution>
+          </range>
+        </ray>
+        <plugin name="laser_scan_controller" filename="libgazebo_ros_laser.so">
+          <frameName>${namespace}/${parent_link}</frameName>
+          <topicName>depth_scan</topicName>
+        </plugin>
+      </sensor>
     </gazebo>
   </xacro:macro>

File: rotors_description/urdf/techpod_base.xacro (robot description, xacro)
@@ -35,5 +35,5 @@
   <xacro:camera_macro
     namespace="${namespace}"
-    parent_link="${namespace}/base_link_inertia"
+    parent_link="${namespace}/base_link"
     camera_suffix="downward"
     frame_rate="35.0"
@@ -41,5 +41,5 @@
     image_width="752"
     image_height="480"
-    image_format="R8G8B8"
+    image_format="L8"
     min_distance="0.1"
     max_distance="100.0"
@@ -48,6 +48,13 @@
     enable_visual="false">
     <mesh filename="package://rotors_description/meshes/vi_camera.dae" scale="1 1 1" />
-    <origin xyz="0 0 0" rpy="0 1.5707 0" />
+    <origin xyz="0 0 0" rpy="0 1.5707 1.5707" />
   </xacro:camera_macro>
+  <!-- Mount a downward-looking laser sensor. -->
+  <xacro:laser_sensor_plugin_macro
+    namespace="${namespace}"
+    parent_link="${namespace}/base_link"
+    laser_suffix="downward">
+    <origin xyz="0 0 0" rpy="0 1.5707 1.5707" />
+  </xacro:laser_sensor_plugin_macro>
   <xacro:if value="$(arg enable_ground_truth)">
     <xacro:ground_truth_imu_and_odometry namespace="${namespace}" parent_link="${namespace}/base_link_inertia" />

Commit message: Adding a gps plugin with gaussian noise

File: rotors_description/urdf/component_snippets.xacro (robot description, xacro)
@@ -314,5 +314,5 @@
     </gazebo>
   </xacro:macro>
-<!-- Macro to add a generic odometry sensor. -->
+  <!-- Macro to add a generic odometry sensor. -->
   <xacro:macro name="odometry_plugin_macro"
     params="
@@ -366,4 +366,75 @@
         </xacro:if>
       </plugin>
+    </gazebo>
+  </xacro:macro>
+  <!-- Macro to add a GPS sensor with gaussian noise. -->
+  <xacro:macro name="gps_gaussian_plugin_macro"
+    params="namespace gps_suffix parent_link gps_topic mass_gps_sensor *inertia
+      *origin">
+    <!-- GPS link -->
+    <link name="${namespace}/gps${gps_suffix}_link">
+      <inertial>
+        <xacro:insert_block name="inertia" />
+        <mass value="${mass_gps_sensor}" />  <!-- [kg] -->
+        <origin xyz="0 0 0" rpy="0 0 0" />
+      </inertial>
+    </link>
+    <!-- GPS joint -->
+    <joint name="${namespace}/gps${gps_suffix}_joint" type="revolute">
+      <xacro:insert_block name="origin" />
+      <parent link="${parent_link}" />
+      <child link="${namespace}/gps${gps_suffix}_link" />
+      <limit upper="0" lower="0" effort="0" velocity="0" />
+    </joint>
+    <gazebo reference="${namespace}/gps${gps_suffix}_link">
+      <sensor type="gps" name="${namespace}_gps${gps_suffix}">
+        <pose>0 0 0 0 0 0</pose>
+        <visualize>0</visualize>
+        <always_on>1</always_on>
+        <update_rate>5</update_rate>
+        <gps>
+          <position_sensing>
+            <horizontal>
+              <noise type="gaussian">
+                <mean>0.0</mean>
+                <stddev>3.000</stddev>
+                <bias_mean>0.0</bias_mean>
+                <bias_stddev>0.0</bias_stddev>
+              </noise>
+            </horizontal>
+            <vertical>
+              <noise type="gaussian">
+                <mean>0.0</mean>
+                <stddev>6.000</stddev>
+                <bias_mean>0.0</bias_mean>
+                <bias_stddev>0.0</bias_stddev>
+              </noise>
+            </vertical>
+          </position_sensing>
+          <velocity_sensing>
+            <horizontal>
+              <noise type="gaussian">
+                <mean>0.0</mean>
+                <stddev>0.03</stddev>
+                <bias_mean>0.0</bias_mean>
+                <bias_stddev>0.0</bias_stddev>
+              </noise>
+            </horizontal>
+            <vertical>
+              <noise type="gaussian">
+                <mean>0.0</mean>
+                <stddev>0.100</stddev>
+                <bias_mean>0.0</bias_mean>
+                <bias_stddev>0.0</bias_stddev>
+              </noise>
+            </vertical>
+          </velocity_sensing>
+        </gps>
+        <plugin filename="librotors_gazebo_gps_plugin.so" name="rotors_gazebo_gps${gps_suffix}_plugin">
+          <robotNamespace>${namespace}</robotNamespace> <!-- (string, required): ros namespace in which the messages are published -->
+          <linkName>${namespace}/gps${gps_suffix}_link</linkName> <!-- (string, required): name of the body which holds the GPS sensor -->
+          <gpsTopic>${gps_topic}</gpsTopic> <!-- (string): name of the sensor output topic and prefix of service names (defaults to gps) -->
+        </plugin>
+      </sensor>
     </gazebo>
   </xacro:macro>
@@ -668,4 +739,16 @@
     </xacro:imu_plugin_macro>
   </xacro:macro>
+  <xacro:macro name="default_gps_gaussian" params="namespace parent_link">
+    <!-- Default GPS. -->
+    <xacro:gps_gaussian_plugin_macro
+      namespace="${namespace}"
+      gps_suffix=""
+      parent_link="${parent_link}"
+      gps_topic="gps"
+      mass_gps_sensor="0.015">
+      <inertia ixx="0.00001" ixy="0.0" ixz="0.0" iyy="0.00001" iyz="0.0" izz="0.00001" />
+      <origin xyz="0 0 0" rpy="0 0 0" />
+    </xacro:gps_gaussian_plugin_macro>
+  </xacro:macro>
   <xacro:macro name="default_mavlink_interface" params="namespace imu_sub_topic rotor_count">
     <xacro:mavlink_interface_macro

File: rotors_description/urdf/firefly_base.xacro (robot description, xacro)
@@ -28,4 +28,6 @@
   <!-- Mount an ADIS16448 IMU. -->
   <xacro:default_imu namespace="${namespace}" parent_link="${namespace}/base_link" />
+  <!-- Mount a GPS sensor. -->
+  <xacro:default_gps_gaussian namespace="${namespace}" parent_link="${namespace}/base_link" />
   <xacro:if value="$(arg enable_ground_truth)">
     <xacro:ground_truth_imu_and_odometry namespace="${namespace}" parent_link="${namespace}/base_link" />

Commit message: Adding parameters for whether to mount a GPS and which noise model to use.

File: rotors_description/urdf/component_snippets.xacro (robot description, xacro)
@@ -368,8 +368,9 @@
     </gazebo>
   </xacro:macro>
-  <!-- Macro to add a GPS sensor with gaussian noise. -->
-  <xacro:macro name="gps_gaussian_plugin_macro"
-    params="namespace gps_suffix parent_link gps_topic mass_gps_sensor *inertia
-      *origin">
+  <!-- Macro to add a GPS sensor. -->
+  <xacro:macro name="gps_plugin_macro"
+    params="namespace gps_suffix parent_link gps_topic mass_gps_sensor
+      use_advanced_noise horizontal_pos_std_dev vertical_pos_std_dev
+      horizontal_vel_std_dev vertical_vel_std_dev *inertia *origin">
     <!-- GPS link -->
     <link name="${namespace}/gps${gps_suffix}_link">
@@ -393,42 +394,47 @@
         <always_on>1</always_on>
         <update_rate>5</update_rate>
-        <gps>
-          <position_sensing>
-            <horizontal>
-              <noise type="gaussian">
-                <mean>0.0</mean>
-                <stddev>3.000</stddev>
-                <bias_mean>0.0</bias_mean>
-                <bias_stddev>0.0</bias_stddev>
-              </noise>
-            </horizontal>
-            <vertical>
-              <noise type="gaussian">
-                <mean>0.0</mean>
-                <stddev>6.000</stddev>
-                <bias_mean>0.0</bias_mean>
-                <bias_stddev>0.0</bias_stddev>
-              </noise>
-            </vertical>
-          </position_sensing>
-          <velocity_sensing>
-            <horizontal>
-              <noise type="gaussian">
-                <mean>0.0</mean>
-                <stddev>0.03</stddev>
-                <bias_mean>0.0</bias_mean>
-                <bias_stddev>0.0</bias_stddev>
-              </noise>
-            </horizontal>
-            <vertical>
-              <noise type="gaussian">
-                <mean>0.0</mean>
-                <stddev>0.100</stddev>
-                <bias_mean>0.0</bias_mean>
-                <bias_stddev>0.0</bias_stddev>
-              </noise>
-            </vertical>
-          </velocity_sensing>
-        </gps>
+        <xacro:if value="${use_advanced_noise}">
+          <gps></gps>
+        </xacro:if>
+        <xacro:unless value="${use_advanced_noise}">
+          <gps>
+            <position_sensing>
+              <horizontal>
+                <noise type="gaussian">
+                  <mean>0.0</mean>
+                  <stddev>${horizontal_pos_std_dev}</stddev>
+                  <bias_mean>0.0</bias_mean>
+                  <bias_stddev>0.0</bias_stddev>
+                </noise>
+              </horizontal>
+              <vertical>
+                <noise type="gaussian">
+                  <mean>0.0</mean>
+                  <stddev>${vertical_pos_std_dev}</stddev>
+                  <bias_mean>0.0</bias_mean>
+                  <bias_stddev>0.0</bias_stddev>
+                </noise>
+              </vertical>
+            </position_sensing>
+            <velocity_sensing>
+              <horizontal>
+                <noise type="gaussian">
+                  <mean>0.0</mean>
+                  <stddev>${horizontal_vel_std_dev}</stddev>
+                  <bias_mean>0.0</bias_mean>
+                  <bias_stddev>0.0</bias_stddev>
+                </noise>
+              </horizontal>
+              <vertical>
+                <noise type="gaussian">
+                  <mean>0.0</mean>
+                  <stddev>${vertical_vel_std_dev}</stddev>
+                  <bias_mean>0.0</bias_mean>
+                  <bias_stddev>0.0</bias_stddev>
+                </noise>
+              </vertical>
+            </velocity_sensing>
+          </gps>
+        </xacro:unless>
         <plugin filename="librotors_gazebo_gps_plugin.so" name="rotors_gazebo_gps${gps_suffix}_plugin">
           <robotNamespace>${namespace}</robotNamespace> <!-- (string, required): ros namespace in which the messages are published -->
@@ -739,15 +745,20 @@
     </xacro:imu_plugin_macro>
   </xacro:macro>
-  <xacro:macro name="default_gps_gaussian" params="namespace parent_link">
+  <xacro:macro name="default_gps" params="namespace parent_link use_advanced_noise">
     <!-- Default GPS. -->
-    <xacro:gps_gaussian_plugin_macro
+    <xacro:gps_plugin_macro
       namespace="${namespace}"
-      gps_suffix=""
+      gps_suffix="gaussian"
       parent_link="${parent_link}"
       gps_topic="gps"
-      mass_gps_sensor="0.015">
+      mass_gps_sensor="0.015"
+      use_advanced_noise="${use_advanced_noise}"
+      horizontal_pos_std_dev="3.0"
+      vertical_pos_std_dev="6.0"
+      horizontal_vel_std_dev="0.03"
+      vertical_vel_std_dev="0.1">
       <inertia ixx="0.00001" ixy="0.0" ixz="0.0" iyy="0.00001" iyz="0.0" izz="0.00001" />
       <origin xyz="0 0 0" rpy="0 0 0" />
-    </xacro:gps_gaussian_plugin_macro>
+    </xacro:gps_plugin_macro>
   </xacro:macro>
   <xacro:macro name="default_mavlink_interface" params="namespace imu_sub_topic rotor_count">

File: rotors_description/urdf/firefly_base.xacro (robot description, xacro)
@@ -28,6 +28,10 @@
   <!-- Mount an ADIS16448 IMU. -->
   <xacro:default_imu namespace="${namespace}" parent_link="${namespace}/base_link" />
-  <!-- Mount a GPS sensor. -->
-  <xacro:default_gps_gaussian namespace="${namespace}" parent_link="${namespace}/base_link" />
+  <xacro:if value="$(arg mount_gps)">
+    <!-- Mount a GPS sensor. -->
+    <xacro:default_gps namespace="${namespace}" parent_link="${namespace}/base_link"
+      use_advanced_noise="$(arg use_advanced_gps_noise)">
+    </xacro:default_gps>
+  </xacro:if>
   <xacro:if value="$(arg enable_ground_truth)">
     <xacro:ground_truth_imu_and_odometry namespace="${namespace}" parent_link="${namespace}/base_link" />

Commit message: Small changes for uav orientation

File: rotors_description/urdf/component_snippets.xacro (robot description, xacro)
@@ -817,5 +817,5 @@
       accelerometer_turn_on_bias_sigma="0.1960">
       <inertia ixx="0.00001" ixy="0.0" ixz="0.0" iyy="0.00001" iyz="0.0" izz="0.00001" />
-      <origin xyz="0 0 0" rpy="0 0 0" />
+      <origin xyz="0 0 0" rpy="3.1415926535897931 0 0" />
     </xacro:imu_plugin_macro>
   </xacro:macro>

File: rotors_description/urdf/techpod_base.xacro (robot description, xacro)
@@ -33,5 +33,5 @@
   <xacro:default_air_speed_sensor namespace="${namespace}" parent_link="${namespace}/base_link" />
   <!-- Mount a downward-looking camera. -->
-  <xacro:camera_macro
+  <!--<xacro:camera_macro
     namespace="${namespace}"
     parent_link="${namespace}/base_link"
@@ -49,12 +49,12 @@
     <mesh filename="package://rotors_description/meshes/vi_camera.dae" scale="1 1 1" />
     <origin xyz="0 0 0" rpy="0 1.5707 1.5707" />
-  </xacro:camera_macro>
+  </xacro:camera_macro>-->
   <!-- Mount a downward-looking laser sensor. -->
-  <xacro:laser_sensor_plugin_macro
+  <!--<xacro:laser_sensor_plugin_macro
     namespace="${namespace}"
     parent_link="${namespace}/base_link"
     laser_suffix="downward">
     <origin xyz="0 0 0" rpy="0 1.5707 1.5707" />
-  </xacro:laser_sensor_plugin_macro>
+  </xacro:laser_sensor_plugin_macro>-->
   <xacro:if value="$(arg enable_ground_truth)">
     <xacro:ground_truth_imu_and_odometry namespace="${namespace}" parent_link="${namespace}/base_link_inertia" />
