Commit message: Adding magnetometer and sdf api wrapper from master branch

File: rotors_description/urdf/component_snippets.xacro (robot description, xacro)
@@ -401,14 +401,14 @@
     </gazebo>
   </xacro:macro>
-  <!-- Macro to add a magnetometer sensor. -->
+  <!-- Macro to add a magnetometer. -->
   <xacro:macro name="magnetometer_plugin_macro"
-    params="namespace magnetometer_suffix parent_link magnetometer_topic mass_magnetometer
-      reference_magnetic_field_north reference_magnetic_field_east reference_magnetic_field_down
-      noise_normal noise_uniform *inertia *origin">
+    params="namespace magnetometer_suffix parent_link magnetometer_topic
+      mass_magnetometer_sensor ref_mag_north ref_mag_east ref_mag_down
+      noise_normal noise_uniform_initial_bias *inertia *origin">
     <!-- Magnetometer link -->
     <link name="${namespace}/magnetometer${magnetometer_suffix}_link">
       <inertial>
         <xacro:insert_block name="inertia" />
-        <mass value="${mass_magnetometer}" />  <!-- [kg] -->
+        <mass value="${mass_magnetometer_sensor}" />  <!-- [kg] -->
         <origin xyz="0 0 0" rpy="0 0 0" />
       </inertial>
@@ -426,13 +426,13 @@
         <linkName>${namespace}/magnetometer${magnetometer_suffix}_link</linkName> <!-- (string, required): name of the body which holds the magnetometer -->
         <magnetometerTopic>${magnetometer_topic}</magnetometerTopic> <!-- (string): name of the sensor output topic and prefix of service names (defaults to 'magnetic_field') -->
-        <!-- [Tesla] Below are the North, East, and Down components of the Earth's magnetic field at the reference location.
+        <!-- [Tesla] Below is the reference Earth's magnetic field at the reference location in NED frame.
              The default reference location is Zurich (lat=+47.3667degN, lon=+8.5500degE, h=+500m, WGS84).
 	     You can obtain the magnetic field strength for your location using the World Magnetic Model:
-             https://www.ngdc.noaa.gov/geomag/WMM/calculators.shtml -->
-        <referenceMagNorth>${reference_magnetic_field_north}</referenceMagNorth>
-        <referenceMagEast>${reference_magnetic_field_east}</referenceMagEast>
-        <referenceMagDown>${reference_magnetic_field_down}</referenceMagDown>
-        <noiseNormal>${noise_normal}</noiseNormal> <!-- standard deviation of additive white gaussian noise [rad] -->
-        <noiseUniform>${noise_uniform}</noiseUniform> <!-- symmetric bounds of uniform noise [rad] -->
+             http://www.ngdc.noaa.gov/geomag-web/#igrfwmm -->
+        <refMagNorth>${ref_mag_north}</refMagNorth>
+        <refMagEast>${ref_mag_east}</refMagEast>
+        <refMagDown>${ref_mag_down}</refMagDown>
+        <noiseNormal>${noise_normal}</noiseNormal> <!-- standard deviation of additive white gaussian noise [Tesla] -->
+        <noiseUniformInitialBias>${noise_uniform_initial_bias}</noiseUniformInitialBias> <!-- symmetric bounds of uniform noise for initial sensor bias [Tesla] -->
       </plugin>
     </gazebo>
@@ -813,7 +813,7 @@
       gyroscope_turn_on_bias_sigma="0.0087"
       accelerometer_noise_density="0.004"
-      accelerometer_random_walk="0.006"
+      accelerometer_random_walk="0.0"
       accelerometer_bias_correlation_time="300.0"
-      accelerometer_turn_on_bias_sigma="0.1960">
+      accelerometer_turn_on_bias_sigma="0.0">
       <inertia ixx="0.00001" ixy="0.0" ixz="0.0" iyy="0.00001" iyz="0.0" izz="0.00001" />
       <origin xyz="0 0 0" rpy="3.1415926535897931 0 0" />
@@ -839,4 +839,5 @@
   </xacro:macro>
   <xacro:macro name="default_magnetometer" params="namespace parent_link">
+    <!-- ADIS16448 Magnetometer. -->
     <xacro:magnetometer_plugin_macro
       namespace="${namespace}"
@@ -844,12 +845,12 @@
       parent_link="${parent_link}"
       magnetometer_topic="magnetic_field"
-      mass_magnetometer="0.015"
-      reference_magnetic_field_north="0.000021475"
-      reference_magnetic_field_east="0.000000797"
-      reference_magnetic_field_down="0.000042817"
-      noise_normal="0 0 0"
-      noise_uniform="0 0 0">
+      mass_magnetometer_sensor="0.015"
+      ref_mag_north="0.000021493"
+      ref_mag_east="0.000000815"
+      ref_mag_down="0.000042795"
+      noise_normal="0.000000080 0.000000080 0.000000080"
+      noise_uniform_initial_bias="0.000000400 0.000000400 0.000000400">
       <inertia ixx="0.00001" ixy="0.0" ixz="0.0" iyy="0.00001" iyz="0.0" izz="0.00001" />
-      <origin xyz="0 0 0" rpy="0 0 0" />
+      <origin xyz="0 0 0" rpy="3.1415926535897931 0 0" />
     </xacro:magnetometer_plugin_macro>
   </xacro:macro>

Commit message: Changing the orientation of the airplane back to north, west, up

File: rotors_description/urdf/component_snippets.xacro (robot description, xacro)
@@ -817,5 +817,5 @@
       accelerometer_turn_on_bias_sigma="0.0">
       <inertia ixx="0.00001" ixy="0.0" ixz="0.0" iyy="0.00001" iyz="0.0" izz="0.00001" />
-      <origin xyz="0 0 0" rpy="3.1415926535897931 0 0" />
+      <origin xyz="0 0 0" rpy="0 0 0" />
     </xacro:imu_plugin_macro>
   </xacro:macro>
@@ -852,5 +852,5 @@
       noise_uniform_initial_bias="0.000000400 0.000000400 0.000000400">
       <inertia ixx="0.00001" ixy="0.0" ixz="0.0" iyy="0.00001" iyz="0.0" izz="0.00001" />
-      <origin xyz="0 0 0" rpy="3.1415926535897931 0 0" />
+      <origin xyz="0 0 0" rpy="0 0 0" />
     </xacro:magnetometer_plugin_macro>
   </xacro:macro>

File: rotors_description/urdf/techpod.xacro (robot description, xacro)
@@ -100,5 +100,5 @@
     use_mesh_file="${use_mesh}"
     mesh_file="package://rotors_description/meshes/techpod/techpod_body.dae">
-    <origin xyz="0 0 0" rpy="${PI} 0 0" />
+    <origin xyz="0 0 0" rpy="0 0 0" />
     <xacro:insert_block name="body_inertia" />
   </xacro:fixed_wing_base_macro>
@@ -118,7 +118,7 @@
     surface_width="${aileron_width}"
     surface_height="${aileron_height}">
-    <axis xyz="0 1 0" />
-    <origin xyz="0.1095 -0.99245 -0.115" rpy="0.0 0.0 0.0" />
-    <origin xyz="0.0 0.0 0.0" rpy="${PI} 0.0 0.0" />
+    <axis xyz="0 -1 0" />
+    <origin xyz="0.1095 0.99245 0.115" rpy="0 0 0" />
+    <origin xyz="0 0 0" rpy="0 0 0" />
     <xacro:insert_block name="aileron_inertia" />
   </xacro:control_surface>
@@ -137,7 +137,7 @@
     surface_width="${aileron_width}"
     surface_height="${aileron_height}">
-    <axis xyz="0 -1 0" />
-    <origin xyz="0.1095 0.99245 -0.115" rpy="0.0 0.0 0.0" />
-    <origin xyz="0.0 0.0 0.0" rpy="${PI} 0.0 0.0" />
+    <axis xyz="0 1 0" />
+    <origin xyz="0.1095 -0.99245 0.115" rpy="0 0 0" />
+    <origin xyz="0 0 0" rpy="0 0 0" />
     <xacro:insert_block name="aileron_inertia" />
   </xacro:control_surface>
@@ -158,6 +158,6 @@
     surface_height="${flap_height}">
     <axis xyz="0 -1 0" />
-    <origin xyz="0.101 -0.382 -0.1185" rpy="0.0 0.0 0.0" />
-    <origin xyz="0.0 0.0 0.0" rpy="${PI} 0.0 0.0" />
+    <origin xyz="0.101 0.382 0.1185" rpy="0 0 0" />
+    <origin xyz="0 0 0" rpy="0 0 0" />
     <xacro:insert_block name="flap_inertia" />
   </xacro:control_surface>
@@ -177,6 +177,6 @@
     surface_height="${flap_height}">
     <axis xyz="0 1 0" />
-    <origin xyz="0.101 0.382 -0.1185" rpy="0.0 0.0 0.0" />
-    <origin xyz="0.0 0.0 0.0" rpy="${PI} 0.0 0.0" />
+    <origin xyz="0.101 -0.382 0.1185" rpy="0 0 0" />
+    <origin xyz="0 0 0" rpy="0 0 0" />
     <xacro:insert_block name="flap_inertia" />
   </xacro:control_surface>
@@ -196,7 +196,7 @@
     surface_width="${elevator_width}"
     surface_height="${elevator_height}">
-    <axis xyz="0 1 0" />
-    <origin xyz="-0.555 0.0 -0.26" rpy="0.0 0.0 0.0" />
-    <origin xyz="0.0 0.0 0.0" rpy="${PI} 0.0 0.0" />
+    <axis xyz="0 -1 0" />
+    <origin xyz="-0.555 0.0 0.26" rpy="0 0 0" />
+    <origin xyz="0 0 0" rpy="0 0 0" />
     <xacro:insert_block name="elevator_inertia" />
   </xacro:control_surface>
@@ -216,11 +216,11 @@
     surface_width="${rudder_width}"
     surface_height="${rudder_height}">
-    <axis xyz="0 0 -1" />
-    <origin xyz="-0.428 0.0 0.0" rpy="0.0 0.25 0.0" />
-    <origin xyz="0.0 0.0 0.0" rpy="${PI} -0.25 0.0" />
+    <axis xyz="0 0 1" />
+    <origin xyz="-0.428 0.0 0.0" rpy="0 0.25 0" />
+    <origin xyz="0 0 0" rpy="0 -0.25 0" />
     <xacro:insert_block name="rudder_inertia" />
   </xacro:control_surface>
   <!-- Instantiate the propeller -->
-  <xacro:propeller
+  <!--<xacro:propeller
     robot_namespace="${namespace}"
     suffix=""
@@ -231,6 +231,6 @@
     use_mesh_file="${use_mesh}"
     mesh_file="package://rotors_description/meshes/propeller_${propeller_direction}.dae">
-    <origin xyz="-0.025 0.0 -0.15" rpy="0.0 ${-0.5*PI} 0.0" />
+    <origin xyz="-0.025 0 -0.15" rpy="0 ${-0.5*PI} 0" />
     <xacro:insert_block name="propeller_inertia" />
-  </xacro:propeller>
+  </xacro:propeller>-->
 </robot>

File: rotors_description/urdf/techpod_base.xacro (robot description, xacro)
@@ -48,13 +48,13 @@
     enable_visual="false">
     <mesh filename="package://rotors_description/meshes/vi_camera.dae" scale="1 1 1" />
-    <origin xyz="0 0 0" rpy="0 -1.5707 1.5707" />
+    <origin xyz="0 0 0" rpy="0 1.5707 1.5707" />
   </xacro:camera_macro>
   <!-- Mount a downward-looking laser sensor. -->
-  <xacro:laser_sensor_plugin_macro
+  <!--<xacro:laser_sensor_plugin_macro
     namespace="${namespace}"
     parent_link="${namespace}/base_link"
     laser_suffix="downward">
     <origin xyz="0 0 0" rpy="0 -1.5707 -1.5707" />
-  </xacro:laser_sensor_plugin_macro>
+  </xacro:laser_sensor_plugin_macro>-->
   <xacro:if value="$(arg enable_ground_truth)">
     <xacro:ground_truth_imu_and_odometry namespace="${namespace}" parent_link="${namespace}/base_link_inertia" />

Commit message: Adding new GPS and rosbag plugins code

File: rotors_description/urdf/component_snippets.xacro (robot description, xacro)
@@ -20,5 +20,5 @@
   <!-- Macro to add logging to a bag file. -->
   <xacro:macro name="bag_plugin_macro"
-    params="namespace bag_file rotor_velocity_slowdown_sim">
+    params="namespace bag_file rotor_velocity_slowdown_sim wait_to_record_bag">
     <gazebo>
       <plugin filename="librotors_gazebo_bag_plugin.so" name="rosbag">
@@ -28,4 +28,5 @@
         <frameId>${namespace}/base_link</frameId>
         <rotorVelocitySlowdownSim>${rotor_velocity_slowdown_sim}</rotorVelocitySlowdownSim>
+        <waitToRecordBag>${wait_to_record_bag}</waitToRecordBag>
       </plugin>
     </gazebo>
@@ -368,7 +369,6 @@
   <xacro:macro name="gps_plugin_macro"
     params="namespace gps_suffix parent_link gps_topic ground_speed_topic
-      mass_gps_sensor reference_latitude reference_longitude reference_altitude
-      reference_heading noise_normal_position noise_uniform_position
-      *inertia *origin">
+      mass_gps_sensor horizontal_pos_std_dev vertical_pos_std_dev
+      horizontal_vel_std_dev vertical_vel_std_dev *inertia *origin">
     <!-- GPS link -->
     <link name="${namespace}/gps${gps_suffix}_link">
@@ -386,17 +386,59 @@
       <limit upper="0" lower="0" effort="0" velocity="0" />
     </joint>
-    <gazebo>
-      <plugin filename="librotors_gazebo_gps_plugin.so" name="rotors_gazebo_gps${gps_suffix}_plugin">
-        <robotNamespace>${namespace}</robotNamespace> <!-- (string, required): ros namespace in which the messages are published -->
-        <linkName>${namespace}/gps${gps_suffix}_link</linkName> <!-- (string, required): name of the body which holds the GPS sensor -->
-        <gpsTopic>${gps_topic}</gpsTopic> <!-- (string): name of the sensor output topic and prefix of service names (defaults to 'gps') -->
-        <groundSpeedTopic>${ground_speed_topic}</groundSpeedTopic> <!-- (string): name of the ground speed output topic (defaults to 'ground_speed') -->
-        <referenceLatitude>${reference_latitude}</referenceLatitude> <!-- the initial latitude [degrees [-90, 90]] -->
-        <referenceLongitude>${reference_longitude}</referenceLongitude> <!-- the initial longitude [degrees [-180, 180]] -->
-        <referenceAltitude>${reference_altitude}</referenceAltitude> <!-- the initial altitude [m] -->
-        <referenceHeading>${reference_heading}</referenceHeading> <!-- the initial degrees, measured from North [deg] -->
-        <noiseNormalPosition>${noise_normal_position}</noiseNormalPosition> <!-- standard deviation of additive white gaussian noise [m] -->
-        <noiseUniformPosition>${noise_uniform_position}</noiseUniformPosition> <!-- symmetric bounds of uniform noise [m] -->
-      </plugin>
+    <gazebo reference="${namespace}/gps${gps_suffix}_link">
+      <sensor type="gps" name="${namespace}_gps${gps_suffix}">
+        <pose>0 0 0 0 0 0</pose>
+        <visualize>0</visualize>
+        <always_on>1</always_on>
+        <update_rate>5</update_rate>
+        <gps>
+          <position_sensing>
+            <horizontal>
+              <noise type="gaussian">
+                <mean>0.0</mean>
+                <stddev>${horizontal_pos_std_dev}</stddev>
+                <bias_mean>0.0</bias_mean>
+                <bias_stddev>0.0</bias_stddev>
+              </noise>
+            </horizontal>
+            <vertical>
+              <noise type="gaussian">
+                <mean>0.0</mean>
+                <stddev>${vertical_pos_std_dev}</stddev>
+                <bias_mean>0.0</bias_mean>
+                <bias_stddev>0.0</bias_stddev>
+              </noise>
+            </vertical>
+          </position_sensing>
+          <velocity_sensing>
+            <horizontal>
+              <noise type="gaussian">
+                <mean>0.0</mean>
+                <stddev>${horizontal_vel_std_dev}</stddev>
+                <bias_mean>0.0</bias_mean>
+                <bias_stddev>0.0</bias_stddev>
+              </noise>
+            </horizontal>
+            <vertical>
+              <noise type="gaussian">
+                <mean>0.0</mean>
+                <stddev>${vertical_vel_std_dev}</stddev>
+                <bias_mean>0.0</bias_mean>
+                <bias_stddev>0.0</bias_stddev>
+              </noise>
+            </vertical>
+          </velocity_sensing>
+        </gps>
+        <plugin filename="librotors_gazebo_gps_plugin.so" name="rotors_gazebo_gps${gps_suffix}_plugin">
+          <robotNamespace>${namespace}</robotNamespace> <!-- (string, required): ros namespace in which the messages are published -->
+          <linkName>${namespace}/gps${gps_suffix}_link</linkName> <!-- (string, required): name of the body which holds the GPS sensor -->
+          <gpsTopic>${gps_topic}</gpsTopic> <!-- (string): name of the sensor output topic and prefix of service names (defaults to 'gps') -->
+          <groundSpeedTopic>${ground_speed_topic}</groundSpeedTopic> <!-- (string): name of the ground speed output topic (defaults to 'ground_speed') -->
+          <horPosStdDev>${horizontal_pos_std_dev}</horPosStdDev> <!-- standard deviation for horizontal position noise [m] -->
+          <verPosStdDev>${vertical_pos_std_dev}</verPosStdDev> <!-- standard deviation for vertical position noise [m] -->
+          <horVelStdDev>${horizontal_vel_std_dev}</horVelStdDev> <!-- standard deviation for horizontal speed noise [m/s] -->
+          <verVelStdDev>${vertical_vel_std_dev}</verVelStdDev> <!-- standard deviation for vertical speed noise [m/s] -->
+        </plugin>
+      </sensor>
     </gazebo>
   </xacro:macro>
@@ -813,7 +855,7 @@
       gyroscope_turn_on_bias_sigma="0.0087"
       accelerometer_noise_density="0.004"
-      accelerometer_random_walk="0.0"
+      accelerometer_random_walk="0.006"
       accelerometer_bias_correlation_time="300.0"
-      accelerometer_turn_on_bias_sigma="0.0">
+      accelerometer_turn_on_bias_sigma="0.1960">
       <inertia ixx="0.00001" ixy="0.0" ixz="0.0" iyy="0.00001" iyz="0.0" izz="0.00001" />
       <origin xyz="0 0 0" rpy="0 0 0" />
@@ -821,4 +863,5 @@
   </xacro:macro>
   <xacro:macro name="default_gps" params="namespace parent_link">
+    <!-- Default GPS. -->
     <xacro:gps_plugin_macro
       namespace="${namespace}"
@@ -828,10 +871,8 @@
       ground_speed_topic="ground_speed"
       mass_gps_sensor="0.015"
-      reference_latitude="47.3667"
-      reference_longitude="8.5500"
-      reference_altitude="500.0"
-      reference_heading="0.0"
-      noise_normal_position="0 0 0"
-      noise_uniform_position="0 0 0">
+      horizontal_pos_std_dev="3.0"
+      vertical_pos_std_dev="6.0"
+      horizontal_vel_std_dev="0.1"
+      vertical_vel_std_dev="0.1">
       <inertia ixx="0.00001" ixy="0.0" ixz="0.0" iyy="0.00001" iyz="0.0" izz="0.00001" />
       <origin xyz="0 0 0" rpy="0 0 0" />

File: rotors_description/urdf/techpod_base.xacro (robot description, xacro)
@@ -37,5 +37,5 @@
     parent_link="${namespace}/base_link"
     camera_suffix="downward"
-    frame_rate="35.0"
+    frame_rate="20.0"
     horizontal_fov="1.3962634"
     image_width="752"
@@ -43,10 +43,10 @@
     image_format="L8"
     min_distance="0.1"
-    max_distance="100.0"
+    max_distance="150.0"
     noise_mean="0.0"
     noise_stddev="0.007"
     enable_visual="false">
     <mesh filename="package://rotors_description/meshes/vi_camera.dae" scale="1 1 1" />
-    <origin xyz="0 0 0" rpy="0 1.5707 1.5707" />
+    <origin xyz="5 0 2.5" rpy="0 1.5707 1.5707" />
   </xacro:camera_macro>
   <!-- Mount a downward-looking laser sensor. -->
@@ -65,5 +65,6 @@
       namespace="${namespace}"
       bag_file="$(arg log_file)"
-      rotor_velocity_slowdown_sim="${rotor_velocity_slowdown_sim}" />
+      rotor_velocity_slowdown_sim="${rotor_velocity_slowdown_sim}"
+      wait_to_record_bag="$(arg wait_to_record_bag)" />
   </xacro:if>
 </robot>

Commit message: Adding a simple camera plugin

File: rotors_description/urdf/component_snippets.xacro (robot description, xacro)
@@ -107,4 +107,72 @@
           <distortionT1>0.0</distortionT1>
           <distortionT2>0.0</distortionT2>
+        </plugin>
+      </sensor>
+    </gazebo>
+  </xacro:macro>
+  <!-- Macro to add a raw camera. -->
+  <xacro:macro name="raw_camera_macro"
+    params="namespace parent_link camera_suffix frame_rate
+      horizontal_fov image_width image_height image_format min_distance
+      max_distance noise_mean noise_stddev enable_visual *geometry *origin">
+    <link name="${namespace}/camera_${camera_suffix}_link">
+      <collision>
+        <origin xyz="0 0 0" rpy="0 0 0" />
+        <geometry>
+          <xacro:insert_block name="geometry" />
+        </geometry>
+      </collision>
+      <xacro:if value="${enable_visual}">
+        <visual>
+          <origin xyz="0 0 0" rpy="0 ${pi/2} 0" />
+          <geometry>
+            <xacro:insert_block name="geometry" />
+          </geometry>
+          <material name="red" />
+        </visual>
+      </xacro:if>
+      <inertial>
+        <mass value="1e-5" />
+        <origin xyz="0 0 0" rpy="0 0 0" />
+        <inertia ixx="1e-6" ixy="0" ixz="0" iyy="1e-6" iyz="0" izz="1e-6" />
+      </inertial>
+    </link>
+    <joint name="${namespace}/camera_${camera_suffix}_joint" type="fixed">
+      <xacro:insert_block name="origin" />
+      <parent link="${parent_link}" />
+      <child link="${namespace}/camera_${camera_suffix}_link" />
+    </joint>
+    <link name="${namespace}/camera_${camera_suffix}_optical_link" />
+    <joint name="${namespace}/camera_${camera_suffix}_optical_joint" type="fixed" >
+      <origin xyz="0 0 0" rpy="${-pi/2} 0 ${-pi/2}" />
+      <parent link="${namespace}/camera_${camera_suffix}_link" />
+      <child link="${namespace}/camera_${camera_suffix}_optical_link" />
+    </joint>
+    <gazebo reference="${namespace}/camera_${camera_suffix}_link">
+      <sensor type="camera" name="${namespace}_camera_${camera_suffix}">
+        <update_rate>${frame_rate}</update_rate>
+        <camera name="head">
+          <horizontal_fov>${horizontal_fov}</horizontal_fov>
+          <image>
+            <width>${image_width}</width>
+            <height>${image_height}</height>
+            <format>${image_format}</format>
+          </image>
+          <clip>
+            <near>${min_distance}</near>
+            <far>${max_distance}</far>
+          </clip>
+          <noise>
+            <type>gaussian</type>
+            <!-- Noise is sampled independently per pixel on each frame.
+                 That pixel's noise value is added to each of its color
+                 channels, which at that point lie in the range [0,1]. -->
+            <mean>${noise_mean}</mean>
+            <stddev>${noise_stddev}</stddev>
+          </noise>
+        </camera>
+        <plugin name="${namespace}_camera_${camera_suffix}_controller" filename="librotors_gazebo_camera_plugin.so">
+          <robotNamespace>${namespace}</robotNamespace>
+          <linkName>${namespace}/camera_${camera_suffix}_link</linkName>
         </plugin>
       </sensor>
@@ -850,5 +918,13 @@
       imu_topic="imu"
       mass_imu_sensor="0.015"
-      gyroscope_noise_density="0.0003394"
+      gyroscope_noise_density="0.0"
+      gyroscopoe_random_walk="0.0"
+      gyroscope_bias_correlation_time="10.0"
+      gyroscope_turn_on_bias_sigma="0.0"
+      accelerometer_noise_density="0.0"
+      accelerometer_random_walk="0.0"
+      accelerometer_bias_correlation_time="10.0"
+      accelerometer_turn_on_bias_sigma="0.0">
+      <!--gyroscope_noise_density="0.0003394"
       gyroscopoe_random_walk="0.000038785"
       gyroscope_bias_correlation_time="1000.0"
@@ -857,5 +933,5 @@
       accelerometer_random_walk="0.006"
       accelerometer_bias_correlation_time="300.0"
-      accelerometer_turn_on_bias_sigma="0.1960">
+      accelerometer_turn_on_bias_sigma="0.1960">-->
       <inertia ixx="0.00001" ixy="0.0" ixz="0.0" iyy="0.00001" iyz="0.0" izz="0.00001" />
       <origin xyz="0 0 0" rpy="0 0 0" />

File: rotors_description/urdf/techpod_base.xacro (robot description, xacro)
@@ -33,5 +33,5 @@
   <xacro:default_air_speed_sensor namespace="${namespace}" parent_link="${namespace}/base_link" />
   <!-- Mount a downward-looking camera. -->
-  <xacro:camera_macro
+  <xacro:raw_camera_macro
     namespace="${namespace}"
     parent_link="${namespace}/base_link"
@@ -48,6 +48,6 @@
     enable_visual="false">
     <mesh filename="package://rotors_description/meshes/vi_camera.dae" scale="1 1 1" />
-    <origin xyz="5 0 2.5" rpy="0 1.5707 1.5707" />
-  </xacro:camera_macro>
+    <origin xyz="15 0 7.5" rpy="0 1.5707 1.5707" />
+  </xacro:raw_camera_macro>
   <!-- Mount a downward-looking laser sensor. -->
   <!--<xacro:laser_sensor_plugin_macro
