Commit message: Clean-up and re-adding old GPS plugin and way to pass air/wind speed

File: rotors_description/urdf/component_snippets.xacro (robot description, xacro)
@@ -437,15 +437,49 @@
   <xacro:macro name="gps_plugin_macro"
     params="namespace gps_suffix parent_link gps_topic ground_speed_topic
+      mass_gps_sensor reference_latitude reference_longitude reference_altitude
+      reference_heading noise_normal_position noise_uniform_position
+      *inertia *origin">
+  <!-- GPS link -->
+  <link name="${namespace}/gps${gps_suffix}_link">
+    <inertial>
+      <xacro:insert_block name="inertia" />
+      <mass value="${mass_gps_sensor}" />  <!-- [kg] -->
+      <origin xyz="0 0 0" rpy="0 0 0" />
+    </inertial>
+  </link>
+  <!-- GPS joint -->
+  <joint name="${namespace}/gps${gps_suffix}_joint" type="revolute">
+    <xacro:insert_block name="origin" />
+    <parent link="${parent_link}" />
+    <child link="${namespace}/gps${gps_suffix}_link" />
+    <limit upper="0" lower="0" effort="0" velocity="0" />
+  </joint>
+  <gazebo>
+    <plugin filename="librotors_gazebo_gps_plugin.so" name="rotors_gazebo_gps${gps_suffix}_plugin">
+      <robotNamespace>${namespace}</robotNamespace> <!-- (string, required): ros namespace in which the messages are published -->
+      <linkName>${namespace}/gps${gps_suffix}_link</linkName> <!-- (string, required): name of the body which holds the GPS sensor -->
+      <gpsTopic>${gps_topic}</gpsTopic> <!-- (string): name of the sensor output topic and prefix of service names (defaults to 'gps') -->
+      <groundSpeedTopic>${ground_speed_topic}</groundSpeedTopic> <!-- (string): name of the ground speed output topic (defaults to 'ground_speed') -->
+      <referenceLatitude>${reference_latitude}</referenceLatitude> <!-- the initial latitude [degrees [-90, 90]] -->
+      <referenceLongitude>${reference_longitude}</referenceLongitude> <!-- the initial longitude [degrees [-180, 180]] -->
+      <referenceAltitude>${reference_altitude}</referenceAltitude> <!-- the initial altitude [m] -->
+      <referenceHeading>${reference_heading}</referenceHeading> <!-- the initial degrees, measured from North [deg] -->
+      <noiseNormalPosition>${noise_normal_position}</noiseNormalPosition> <!-- standard deviation of additive white gaussian noise [m] -->
+      <noiseUniformPosition>${noise_uniform_position}</noiseUniformPosition> <!-- symmetric bounds of uniform noise [m] -->
+    </plugin>
+  </gazebo>
+  </xacro:macro>
+  <!-- Macro to add a GPS sensor. -->
+  <!--<xacro:macro name="gps_plugin_macro"
+    params="namespace gps_suffix parent_link gps_topic ground_speed_topic
       mass_gps_sensor horizontal_pos_std_dev vertical_pos_std_dev
       horizontal_vel_std_dev vertical_vel_std_dev *inertia *origin">
-    <!-- GPS link -->
     <link name="${namespace}/gps${gps_suffix}_link">
       <inertial>
         <xacro:insert_block name="inertia" />
-        <mass value="${mass_gps_sensor}" />  <!-- [kg] -->
-        <origin xyz="0 0 0" rpy="0 0 0" />
-      </inertial>
-    </link>
-    <!-- GPS joint -->
+        <mass value="${mass_gps_sensor}" />
+        <origin xyz="0 0 0" rpy="0 0 0" />
+      </inertial>
+    </link>
     <joint name="${namespace}/gps${gps_suffix}_joint" type="revolute">
       <xacro:insert_block name="origin" />
@@ -459,5 +493,5 @@
         <visualize>0</visualize>
         <always_on>1</always_on>
-        <update_rate>5</update_rate>
+        <update_rate>5ROS</update_rate>
         <gps>
           <position_sensing>
@@ -499,16 +533,16 @@
         </gps>
         <plugin filename="librotors_gazebo_gps_plugin.so" name="rotors_gazebo_gps${gps_suffix}_plugin">
-          <robotNamespace>${namespace}</robotNamespace> <!-- (string, required): ros namespace in which the messages are published -->
-          <linkName>${namespace}/gps${gps_suffix}_link</linkName> <!-- (string, required): name of the body which holds the GPS sensor -->
-          <gpsTopic>${gps_topic}</gpsTopic> <!-- (string): name of the sensor output topic and prefix of service names (defaults to 'gps') -->
-          <groundSpeedTopic>${ground_speed_topic}</groundSpeedTopic> <!-- (string): name of the ground speed output topic (defaults to 'ground_speed') -->
-          <horPosStdDev>${horizontal_pos_std_dev}</horPosStdDev> <!-- standard deviation for horizontal position noise [m] -->
-          <verPosStdDev>${vertical_pos_std_dev}</verPosStdDev> <!-- standard deviation for vertical position noise [m] -->
-          <horVelStdDev>${horizontal_vel_std_dev}</horVelStdDev> <!-- standard deviation for horizontal speed noise [m/s] -->
-          <verVelStdDev>${vertical_vel_std_dev}</verVelStdDev> <!-- standard deviation for vertical speed noise [m/s] -->
+          <robotNamespace>${namespace}</robotNamespace>
+          <linkName>${namespace}/gps${gps_suffix}_link</linkName>
+          <gpsTopic>${gps_topic}</gpsTopic>
+          <groundSpeedTopic>${ground_speed_topic}</groundSpeedTopic>
+          <horPosStdDev>${horizontal_pos_std_dev}</horPosStdDev>
+          <verPosStdDev>${vertical_pos_std_dev}</verPosStdDev>
+          <horVelStdDev>${horizontal_vel_std_dev}</horVelStdDev>
+          <verVelStdDev>${vertical_vel_std_dev}</verVelStdDev>
         </plugin>
       </sensor>
     </gazebo>
-  </xacro:macro>
+  </xacro:macro>-->
   <!-- Macro to add a magnetometer. -->
   <xacro:macro name="magnetometer_plugin_macro"
@@ -918,5 +952,13 @@
       imu_topic="imu"
       mass_imu_sensor="0.015"
-      gyroscope_noise_density="0.0"
+      gyroscope_noise_density="0.0003394"
+      gyroscopoe_random_walk="0.000038785"
+      gyroscope_bias_correlation_time="1000.0"
+      gyroscope_turn_on_bias_sigma="0.0087"
+      accelerometer_noise_density="0.004"
+      accelerometer_random_walk="0.006"
+      accelerometer_bias_correlation_time="300.0"
+      accelerometer_turn_on_bias_sigma="0.1960">
+      <!--gyroscope_noise_density="0.0"
       gyroscopoe_random_walk="0.0"
       gyroscope_bias_correlation_time="10.0"
@@ -925,19 +967,31 @@
       accelerometer_random_walk="0.0"
       accelerometer_bias_correlation_time="10.0"
-      accelerometer_turn_on_bias_sigma="0.0">
-      <!--gyroscope_noise_density="0.0003394"
-      gyroscopoe_random_walk="0.000038785"
-      gyroscope_bias_correlation_time="1000.0"
-      gyroscope_turn_on_bias_sigma="0.0087"
-      accelerometer_noise_density="0.004"
-      accelerometer_random_walk="0.006"
-      accelerometer_bias_correlation_time="300.0"
-      accelerometer_turn_on_bias_sigma="0.1960">-->
+      accelerometer_turn_on_bias_sigma="0.0">-->
       <inertia ixx="0.00001" ixy="0.0" ixz="0.0" iyy="0.00001" iyz="0.0" izz="0.00001" />
       <origin xyz="0 0 0" rpy="0 0 0" />
     </xacro:imu_plugin_macro>
   </xacro:macro>
+  <!--<xacro:macro name="default_gps" params="namespace parent_link">-->
+    <!-- Default GPS. -->
+    <!--<xacro:gps_plugin_macro
+      namespace="${namespace}"
+      gps_suffix=""
+      parent_link="${parent_link}"
+      gps_topic="gps"
+      ground_speed_topic="ground_speed"
+      mass_gps_sensor="0.015"
+      horizontal_pos_std_dev="0.0"
+      vertical_pos_std_dev="0.0"
+      horizontal_vel_std_dev="0.0"
+      vertical_vel_std_dev="0.0">-->
+      <!--horizontal_pos_std_dev="3.0"
+      vertical_pos_std_dev="6.0"
+      horizontal_vel_std_dev="0.1"
+      vertical_vel_std_dev="0.1">-->
+      <!--<inertia ixx="0.00001" ixy="0.0" ixz="0.0" iyy="0.00001" iyz="0.0" izz="0.00001" />
+      <origin xyz="0 0 0" rpy="0 0 0" />
+    </xacro:gps_plugin_macro>
+  </xacro:macro>-->
   <xacro:macro name="default_gps" params="namespace parent_link">
-    <!-- Default GPS. -->
     <xacro:gps_plugin_macro
       namespace="${namespace}"
@@ -947,8 +1001,10 @@
       ground_speed_topic="ground_speed"
       mass_gps_sensor="0.015"
-      horizontal_pos_std_dev="3.0"
-      vertical_pos_std_dev="6.0"
-      horizontal_vel_std_dev="0.1"
-      vertical_vel_std_dev="0.1">
+      reference_latitude="47.3667"
+      reference_longitude="8.5500"
+      reference_altitude="500.0"
+      reference_heading="0.0"
+      noise_normal_position="0 0 0"
+      noise_uniform_position="0 0 0">
       <inertia ixx="0.00001" ixy="0.0" ixz="0.0" iyy="0.00001" iyz="0.0" izz="0.00001" />
       <origin xyz="0 0 0" rpy="0 0 0" />

File: rotors_description/urdf/techpod_base.xacro (robot description, xacro)
@@ -48,13 +48,6 @@
     enable_visual="false">
     <mesh filename="package://rotors_description/meshes/vi_camera.dae" scale="1 1 1" />
-    <origin xyz="15 0 7.5" rpy="0 1.5707 1.5707" />
+    <origin xyz="0 0 0" rpy="0 1.5707 1.5707" />
   </xacro:raw_camera_macro>
-  <!-- Mount a downward-looking laser sensor. -->
-  <!--<xacro:laser_sensor_plugin_macro
-    namespace="${namespace}"
-    parent_link="${namespace}/base_link"
-    laser_suffix="downward">
-    <origin xyz="0 0 0" rpy="0 -1.5707 -1.5707" />
-  </xacro:laser_sensor_plugin_macro>-->
   <xacro:if value="$(arg enable_ground_truth)">
     <xacro:ground_truth_imu_and_odometry namespace="${namespace}" parent_link="${namespace}/base_link_inertia" />

Commit message: Adding flap actuation and some other small changes

File: rotors_description/urdf/component_snippets.xacro (robot description, xacro)
@@ -960,12 +960,4 @@
       accelerometer_bias_correlation_time="300.0"
       accelerometer_turn_on_bias_sigma="0.1960">
-      <!--gyroscope_noise_density="0.0"
-      gyroscopoe_random_walk="0.0"
-      gyroscope_bias_correlation_time="10.0"
-      gyroscope_turn_on_bias_sigma="0.0"
-      accelerometer_noise_density="0.0"
-      accelerometer_random_walk="0.0"
-      accelerometer_bias_correlation_time="10.0"
-      accelerometer_turn_on_bias_sigma="0.0">-->
       <inertia ixx="0.00001" ixy="0.0" ixz="0.0" iyy="0.00001" iyz="0.0" izz="0.00001" />
       <origin xyz="0 0 0" rpy="0 0 0" />
@@ -1019,7 +1011,7 @@
       magnetometer_topic="magnetic_field"
       mass_magnetometer_sensor="0.015"
-      ref_mag_north="0.000021493"
-      ref_mag_east="0.000000815"
-      ref_mag_down="0.000042795"
+      ref_mag_north="0.000021517759"
+      ref_mag_east="0.000000794477"
+      ref_mag_down="0.00004274884"
       noise_normal="0.000000080 0.000000080 0.000000080"
       noise_uniform_initial_bias="0.000000400 0.000000400 0.000000400">

File: rotors_description/urdf/fixed_wing_base.xacro (robot description, xacro)
@@ -60,5 +60,6 @@
     </link>
     <gazebo>
-      <plugin name="${robot_namespace}_base" filename="librotors_gazebo_fixedwing_base_plugin.so">
+      <!--<plugin name="${robot_namespace}_base" filename="librotors_gazebo_fixedwing_base_plugin.so">-->
+      <plugin name="${robot_namespace}_base" filename="librotors_gazebo_aerodynamics_plugin.so">
         <robotNamespace>${robot_namespace}</robotNamespace>
         <linkName>${robot_namespace}/base_link</linkName>
@@ -71,5 +72,5 @@
   <!-- Control surface joint and link -->
   <xacro:macro name="control_surface"
-    params="robot_namespace surface_name parent mass_surface surface_type
+    params="robot_namespace surface_name parent mass_surface surface_type surface_side
       min_angle max_angle color use_mesh_file mesh_file surface_length surface_width
       surface_height *axis *joint_origin *link_origin *inertia">
@@ -115,4 +116,6 @@
         <jointName>${robot_namespace}/${surface_name}_joint</jointName>
         <surfaceType>${surface_type}</surfaceType>
+        <surfaceSide>${surface_side}</surfaceSide>
+        <surfaceName>${surface_name}</surfaceName>
         <angleMin>${min_angle}</angleMin>
         <angleMax>${max_angle}</angleMax>

File: rotors_description/urdf/techpod.xacro (robot description, xacro)
@@ -20,5 +20,5 @@
   <xacro:property name="PI" value="3.1415926535897931" />
   <!-- Component masses -->
-  <xacro:property name="mass_fuselage" value="2.05" /> <!-- [kg] -->
+  <xacro:property name="mass_fuselage" value="1.25" /> <!-- [kg] -->
   <xacro:property name="mass_aileron" value="0.1" /> <!-- [kg] -->
   <xacro:property name="mass_flap" value="0.1" /> <!-- [kg] -->
@@ -42,6 +42,6 @@
   <xacro:property name="flap_width" value="0.459" /> <!-- [m] -->
   <xacro:property name="flap_height" value="0.016" /> <!-- [m] -->
-  <xacro:property name="flap_min_angle" value="0.0" /> <!-- [rad] -->
-  <xacro:property name="flap_max_angle" value="0.0" /> <!-- [rad] -->
+  <xacro:property name="flap_min_angle" value="-0.349066" /> <!-- [rad] -->
+  <xacro:property name="flap_max_angle" value="0.349066" /> <!-- [rad] -->
   <xacro:property name="flap_color" value="Yellow" />
   <!-- Elevator properties -->
@@ -66,5 +66,6 @@
   <!-- Inertia of the main body -->
   <xacro:property name="body_inertia">
-    <inertia ixx="0.16632" ixy="0.0" ixz="0.0755" iyy="0.3899" iyz="0.0" izz="0.5243" />
+    <!--<inertia ixx="0.16632" ixy="0.0" ixz="0.0755" iyy="0.3899" iyz="0.0" izz="0.5243" />-->
+    <inertia ixx="0.1512" ixy="0.0" ixz="0.0755" iyy="0.2785" iyz="0.0" izz="0.3745" />
   </xacro:property>
   <!-- Inertia of the aileron, assuming it is a cuboid -->
@@ -110,4 +111,5 @@
     mass_surface="${mass_aileron}"
     surface_type="aileron"
+    surface_side="left"
     min_angle="${aileron_min_angle}"
     max_angle="${aileron_max_angle}"
@@ -129,4 +131,5 @@
     mass_surface="${mass_aileron}"
     surface_type="aileron"
+    surface_side="right"
     min_angle="${aileron_min_angle}"
     max_angle="${aileron_max_angle}"
@@ -149,4 +152,5 @@
     mass_surface="${mass_flap}"
     surface_type="flap"
+    surface_side="left"
     min_angle="${flap_min_angle}"
     max_angle="${flap_max_angle}"
@@ -157,5 +161,5 @@
     surface_width="${flap_width}"
     surface_height="${flap_height}">
-    <axis xyz="0 -1 0" />
+    <axis xyz="0 1 0" />
     <origin xyz="0.101 0.382 0.1185" rpy="0 0 0" />
     <origin xyz="0 0 0" rpy="0 0 0" />
@@ -168,4 +172,5 @@
     mass_surface="${mass_flap}"
     surface_type="flap"
+    surface_side="right"
     min_angle="${flap_min_angle}"
     max_angle="${flap_max_angle}"
@@ -188,4 +193,5 @@
     mass_surface="${mass_elevator}"
     surface_type="elevator"
+    surface_side=""
     min_angle="${elevator_min_angle}"
     max_angle="${elevator_max_angle}"
@@ -208,4 +214,5 @@
     mass_surface="${mass_rudder}"
     surface_type="rudder"
+    surface_side=""
     min_angle="${rudder_min_angle}"
     max_angle="${rudder_max_angle}"
@@ -217,6 +224,6 @@
     surface_height="${rudder_height}">
     <axis xyz="0 0 1" />
-    <origin xyz="-0.428 0.0 0.0" rpy="0 0.25 0" />
-    <origin xyz="0 0 0" rpy="0 -0.25 0" />
+    <origin xyz="-0.428 0.0 0.0" rpy="0 -0.25 0" />
+    <origin xyz="0 0 0" rpy="0 0.25 0" />
     <xacro:insert_block name="rudder_inertia" />
   </xacro:control_surface>

Commit message: Adding temporary code for GPS testing

File: rotors_description/urdf/component_snippets.xacro (robot description, xacro)
@@ -440,36 +440,36 @@
       reference_heading noise_normal_position noise_uniform_position
       *inertia *origin">
-  <!-- GPS link -->
-  <link name="${namespace}/gps${gps_suffix}_link">
-    <inertial>
-      <xacro:insert_block name="inertia" />
-      <mass value="${mass_gps_sensor}" />  <!-- [kg] -->
-      <origin xyz="0 0 0" rpy="0 0 0" />
-    </inertial>
-  </link>
-  <!-- GPS joint -->
-  <joint name="${namespace}/gps${gps_suffix}_joint" type="revolute">
-    <xacro:insert_block name="origin" />
-    <parent link="${parent_link}" />
-    <child link="${namespace}/gps${gps_suffix}_link" />
-    <limit upper="0" lower="0" effort="0" velocity="0" />
-  </joint>
-  <gazebo>
-    <plugin filename="librotors_gazebo_gps_plugin.so" name="rotors_gazebo_gps${gps_suffix}_plugin">
-      <robotNamespace>${namespace}</robotNamespace> <!-- (string, required): ros namespace in which the messages are published -->
-      <linkName>${namespace}/gps${gps_suffix}_link</linkName> <!-- (string, required): name of the body which holds the GPS sensor -->
-      <gpsTopic>${gps_topic}</gpsTopic> <!-- (string): name of the sensor output topic and prefix of service names (defaults to 'gps') -->
-      <groundSpeedTopic>${ground_speed_topic}</groundSpeedTopic> <!-- (string): name of the ground speed output topic (defaults to 'ground_speed') -->
-      <referenceLatitude>${reference_latitude}</referenceLatitude> <!-- the initial latitude [degrees [-90, 90]] -->
-      <referenceLongitude>${reference_longitude}</referenceLongitude> <!-- the initial longitude [degrees [-180, 180]] -->
-      <referenceAltitude>${reference_altitude}</referenceAltitude> <!-- the initial altitude [m] -->
-      <referenceHeading>${reference_heading}</referenceHeading> <!-- the initial degrees, measured from North [deg] -->
-      <noiseNormalPosition>${noise_normal_position}</noiseNormalPosition> <!-- standard deviation of additive white gaussian noise [m] -->
-      <noiseUniformPosition>${noise_uniform_position}</noiseUniformPosition> <!-- symmetric bounds of uniform noise [m] -->
-    </plugin>
-  </gazebo>
+    <!-- GPS link -->
+    <link name="${namespace}/gps${gps_suffix}_link">
+      <inertial>
+        <xacro:insert_block name="inertia" />
+        <mass value="${mass_gps_sensor}" />  <!-- [kg] -->
+        <origin xyz="0 0 0" rpy="0 0 0" />
+      </inertial>
+    </link>
+    <!-- GPS joint -->
+    <joint name="${namespace}/gps${gps_suffix}_joint" type="revolute">
+      <xacro:insert_block name="origin" />
+      <parent link="${parent_link}" />
+      <child link="${namespace}/gps${gps_suffix}_link" />
+      <limit upper="0" lower="0" effort="0" velocity="0" />
+    </joint>
+    <gazebo>
+      <plugin filename="librotors_gazebo_gps_plugin.so" name="rotors_gazebo_gps${gps_suffix}_plugin">
+        <robotNamespace>${namespace}</robotNamespace> <!-- (string, required): ros namespace in which the messages are published -->
+        <linkName>${namespace}/gps${gps_suffix}_link</linkName> <!-- (string, required): name of the body which holds the GPS sensor -->
+        <gpsTopic>${gps_topic}</gpsTopic> <!-- (string): name of the sensor output topic and prefix of service names (defaults to 'gps') -->
+        <groundSpeedTopic>${ground_speed_topic}</groundSpeedTopic> <!-- (string): name of the ground speed output topic (defaults to 'ground_speed') -->
+        <referenceLatitude>${reference_latitude}</referenceLatitude> <!-- the initial latitude [degrees [-90, 90]] -->
+        <referenceLongitude>${reference_longitude}</referenceLongitude> <!-- the initial longitude [degrees [-180, 180]] -->
+        <referenceAltitude>${reference_altitude}</referenceAltitude> <!-- the initial altitude [m] -->
+        <referenceHeading>${reference_heading}</referenceHeading> <!-- the initial degrees, measured from North [deg] -->
+        <noiseNormalPosition>${noise_normal_position}</noiseNormalPosition> <!-- standard deviation of additive white gaussian noise [m] -->
+        <noiseUniformPosition>${noise_uniform_position}</noiseUniformPosition> <!-- symmetric bounds of uniform noise [m] -->
+      </plugin>
+    </gazebo>
   </xacro:macro>
   <!-- Macro to add a GPS sensor. -->
-  <!--<xacro:macro name="gps_plugin_macro"
+  <xacro:macro name="gps_gazebo_plugin_macro"
     params="namespace gps_suffix parent_link gps_topic ground_speed_topic
       mass_gps_sensor horizontal_pos_std_dev vertical_pos_std_dev
@@ -493,5 +493,5 @@
         <visualize>0</visualize>
         <always_on>1</always_on>
-        <update_rate>5ROS</update_rate>
+        <update_rate>5</update_rate>
         <gps>
           <position_sensing>
@@ -532,5 +532,5 @@
           </velocity_sensing>
         </gps>
-        <plugin filename="librotors_gazebo_gps_plugin.so" name="rotors_gazebo_gps${gps_suffix}_plugin">
+        <plugin filename="libgps_temp.so" name="rotors_gazebo_gps${gps_suffix}_plugin">
           <robotNamespace>${namespace}</robotNamespace>
           <linkName>${namespace}/gps${gps_suffix}_link</linkName>
@@ -544,5 +544,5 @@
       </sensor>
     </gazebo>
-  </xacro:macro>-->
+  </xacro:macro>
   <!-- Macro to add a magnetometer. -->
   <xacro:macro name="magnetometer_plugin_macro"
@@ -888,5 +888,5 @@
       accelerometer_noise_density="0.004"
       accelerometer_random_walk="0.006"
-      accelerometer_bias_correlation_time="300.0"
+      accelerometer_bias_correlation_time="30.0"
       accelerometer_turn_on_bias_sigma="0.1960">
       <inertia ixx="0.00001" ixy="0.0" ixz="0.0" iyy="0.00001" iyz="0.0" izz="0.00001" />
@@ -964,11 +964,11 @@
     </xacro:imu_plugin_macro>
   </xacro:macro>
-  <!--<xacro:macro name="default_gps" params="namespace parent_link">-->
+  <xacro:macro name="default_gps_gazebo" params="namespace parent_link">
     <!-- Default GPS. -->
-    <!--<xacro:gps_plugin_macro
+    <xacro:gps_gazebo_plugin_macro
       namespace="${namespace}"
-      gps_suffix=""
-      parent_link="${parent_link}"
-      gps_topic="gps"
+      gps_suffix="gazebo"
+      parent_link="${parent_link}"
+      gps_topic="gps_gazebo"
       ground_speed_topic="ground_speed"
       mass_gps_sensor="0.015"
@@ -976,13 +976,13 @@
       vertical_pos_std_dev="0.0"
       horizontal_vel_std_dev="0.0"
-      vertical_vel_std_dev="0.0">-->
+      vertical_vel_std_dev="0.0">
       <!--horizontal_pos_std_dev="3.0"
       vertical_pos_std_dev="6.0"
       horizontal_vel_std_dev="0.1"
       vertical_vel_std_dev="0.1">-->
-      <!--<inertia ixx="0.00001" ixy="0.0" ixz="0.0" iyy="0.00001" iyz="0.0" izz="0.00001" />
+      <inertia ixx="0.00001" ixy="0.0" ixz="0.0" iyy="0.00001" iyz="0.0" izz="0.00001" />
       <origin xyz="0 0 0" rpy="0 0 0" />
-    </xacro:gps_plugin_macro>
-  </xacro:macro>-->
+    </xacro:gps_gazebo_plugin_macro>
+  </xacro:macro>
   <xacro:macro name="default_gps" params="namespace parent_link">
     <xacro:gps_plugin_macro

File: rotors_description/urdf/fixed_wing_base.xacro (robot description, xacro)
@@ -65,4 +65,7 @@
         <linkName>${robot_namespace}/base_link</linkName>
       </plugin>
+      <!--<plugin name="${robot_namespace}_base" filename="libgps_test.so">
+        <linkName>${robot_namespace}/base_link</linkName>
+      </plugin>-->
     </gazebo>
     <gazebo reference="${robot_namespace}/base_link">
