Commit message: Fixing camera orientation and not using simulation time

File: rotors_description/urdf/techpod_base.xacro (robot description, xacro)
@@ -48,5 +48,5 @@
     enable_visual="false">
     <mesh filename="package://rotors_description/meshes/vi_camera.dae" scale="1 1 1" />
-    <origin xyz="0 0 0" rpy="0 1.5707 1.5707" />
+    <origin xyz="0 0 0" rpy="0 -1.5707 -1.5707" />
   </xacro:camera_macro>-->
   <!-- Mount a downward-looking laser sensor. -->

Commit message: Fixing camera and laser sensor orientations and removing tf broadcasting

File: rotors_description/urdf/techpod_base.xacro (robot description, xacro)
@@ -33,5 +33,5 @@
   <xacro:default_air_speed_sensor namespace="${namespace}" parent_link="${namespace}/base_link" />
   <!-- Mount a downward-looking camera. -->
-  <!--<xacro:camera_macro
+  <xacro:camera_macro
     namespace="${namespace}"
     parent_link="${namespace}/base_link"
@@ -48,13 +48,13 @@
     enable_visual="false">
     <mesh filename="package://rotors_description/meshes/vi_camera.dae" scale="1 1 1" />
-    <origin xyz="0 0 0" rpy="0 -1.5707 -1.5707" />
-  </xacro:camera_macro>-->
+    <origin xyz="0 0 0" rpy="0 -1.5707 1.5707" />
+  </xacro:camera_macro>
   <!-- Mount a downward-looking laser sensor. -->
-  <!--<xacro:laser_sensor_plugin_macro
+  <xacro:laser_sensor_plugin_macro
     namespace="${namespace}"
     parent_link="${namespace}/base_link"
     laser_suffix="downward">
-    <origin xyz="0 0 0" rpy="0 1.5707 1.5707" />
-  </xacro:laser_sensor_plugin_macro>-->
+    <origin xyz="0 0 0" rpy="0 -1.5707 -1.5707" />
+  </xacro:laser_sensor_plugin_macro>
   <xacro:if value="$(arg enable_ground_truth)">
     <xacro:ground_truth_imu_and_odometry namespace="${namespace}" parent_link="${namespace}/base_link_inertia" />

Commit message: Creating a camera controller for a video

File: rotors_description/urdf/techpod_base.xacro (robot description, xacro)
@@ -46,7 +46,7 @@
     noise_mean="0.0"
     noise_stddev="0.007"
-    enable_visual="false">
+    enable_visual="true">
     <mesh filename="package://rotors_description/meshes/vi_camera.dae" scale="1 1 1" />
-    <origin xyz="0 0 0" rpy="0 1.5707 1.5707" />
+    <origin xyz="0 0 -0.03" rpy="0 1.5707 1.5707" />
   </xacro:raw_camera_macro>
   <xacro:if value="$(arg enable_ground_truth)">
