Commit message: Adding a plugin for wing model and starting the fixed wing model

File: rotors_description/urdf/fixed_wing_base.xacro (robot description, xacro)
@@ -16,23 +16,92 @@
   limitations under the License.
 -->
-<robot name="fixed_wing" xmlns:xacro="http://ros.org/wiki/xacro">
-  <xacro:include filename="$(find rotors_description)/urdf/component_snippets.xacro" />
-  <!-- Instantiate fixed wing "mechanics" -->
-  <xacro:include filename="$(find rotors_description)/urdf/firefly.xacro" />
-  <!-- Instantiate a controller. -->
-  <xacro:controller_plugin_macro namespace="${namespace}" imu_sub_topic="imu" />
-  <!-- Mount an ADIS16448 IMU. -->
-  <xacro:default_imu namespace="${namespace}" parent_link="${namespace}/base_link" />
-  <!-- Mount a GPS. -->
-  <xacro:default_gps namespace="${namespace}" parent_link="${namespace}/base_link" />
-  <xacro:if value="$(arg enable_ground_truth)">
-    <xacro:ground_truth_imu_and_odometry namespace="${namespace}" parent_link="${namespace}/base_link" />
-  </xacro:if>
-  <xacro:if value="$(arg enable_logging)">
-    <!-- Instantiate a logger -->
-    <xacro:bag_plugin_macro
-      namespace="${namespace}"
-      bag_file="$(arg log_file)"
-      rotor_velocity_slowdown_sim="${rotor_velocity_slowdown_sim}" />
-  </xacro:if>
+<robot xmlns:xacro="http://ros.org/wiki/xacro">
+  <!-- Macro for the inertia of a box -->
+  <xacro:macro name="box_inertia" params="x y z mass">
+    <inertia ixx="${0.0833333 * mass * (y*y + z*z)}" ixy="0.0" ixz="0.0"
+      iyy="${0.0833333 * mass * (x*x + z*z)}" iyz="0.0"
+      izz="${0.0833333 * mass * (x*x + y*y)}" />
+  </xacro:macro>
+  <!-- Macro for the inertial properties of a box -->
+  <xacro:macro name="box_inertial" params="x y z mass *origin">
+    <inertial>
+      <mass value="${mass}" />
+      <xacro:insert_block name="origin" />
+      <xacro:box_inertia x="${x}" y="${y}" z="${z}" mass="${mass}" />
+    </inertial>
+  </xacro:macro>
+  <!-- Fixed-wing fuselage link -->
+  <xacro:macro name="fixed_wing_base_macro"
+    params="robot_namespace mass body_length body_width body_height use_mesh_file mesh_file *inertia">
+    <link name="${robot_namespace}/base_link"></link>
+    <joint name="${robot_namespace}/base_joint" type="fixed">
+      <origin xyz="0 0 0" rpy="0 0 0" />
+      <parent link="${robot_namespace}/base_link" />
+      <child link="${robot_namespace}/base_link_inertia" />
+    </joint>
+    <link name="${robot_namespace}/base_link_inertia">
+      <inertial>
+        <mass value="${mass}" />  <!-- [kg] -->
+        <origin xyz="0 0 0" />
+        <xacro:insert_block name="inertia" />
+      </inertial>
+      <visual>
+        <origin xyz="0 0 0" rpy="0 0 0" />
+        <geometry>
+          <xacro:if value="${use_mesh_file}">
+            <mesh filename="${mesh_file}" scale="1 1 1" />
+          </xacro:if>
+          <xacro:unless value="${use_mesh_file}">
+            <box size="${body_length} ${body_width} ${body_height}"/> <!-- [m] [m] [m] -->
+          </xacro:unless>
+        </geometry>
+      </visual>
+      <collision>
+        <origin xyz="0 0 0" rpy="0 0 0" />
+        <geometry>
+          <box size="${body_length} ${body_width} ${body_height}" /> <!-- [m] [m] [m] -->
+        </geometry>
+      </collision>
+    </link>
+  </xacro:macro>
+  <!-- Wing joint and link -->
+  <xacro:macro name="wing"
+    params="robot_namespace suffix parent mass_wing
+      wing_length wing_width wing_height use_mesh mesh *origin *inertia">
+    <joint name="${robot_namespace}/wing_${suffix}_joint" type="revolute">
+      <xacro:insert_block name="origin" />
+      <axis xyz="0 0 1" />
+      <parent link="${parent}" />
+      <child link="${robot_namespace}/wing_${suffix}" />
+      <limit upper="0" lower="0" effort="0" velocity="0" />
+    </joint>
+    <link name="${robot_namespace}/wing_${suffix}">
+      <inertial>
+        <mass value="${mass_wing}" /> <!-- [kg] -->
+        <xacro:insert_block name="inertia" />
+      </inertial>
+      <visual>
+        <geometry>
+          <xacro:if value="${use_mesh}">
+            <mesh filename="${mesh}"
+              scale="1 1 1" />
+          </xacro:if>
+          <xacro:unless value="${use_mesh}">
+            <box size="${wing_length} ${wing_width} ${wing_height}"/> <!-- [m] [m] [m] -->
+          </xacro:unless>
+        </geometry>
+      </visual>
+      <collision>
+        <geometry>
+          <box size="${wing_length} ${wing_width} ${wing_height}"/> <!-- [m] [m] [m] -->
+        </geometry>
+      </collision>
+    </link>
+    <gazebo>
+      <plugin name="${robot_namespace}_${suffix}_wing_model" filename="librotors_gazebo_wing_model.so">
+        <robotNamespace>${robot_namespace}</robotNamespace>
+        <linkName>${robot_namespace}/wing_${suffix}</linkName>
+      </plugin>
+    </gazebo>
+  </xacro:macro>
 </robot>

Commit message: First stable flying

File: rotors_description/urdf/fixed_wing_base.xacro (robot description, xacro)
@@ -35,9 +35,10 @@
     <link name="${robot_namespace}/base_link"></link>
     <joint name="${robot_namespace}/base_joint" type="fixed">
-      <origin xyz="0 0 0.0" rpy="0 0 0" />
+      <origin xyz="0 0 0" rpy="0 0 0" />
       <parent link="${robot_namespace}/base_link" />
       <child link="${robot_namespace}/base_link_inertia" />
     </joint>
     <link name="${robot_namespace}/base_link_inertia">
+<!--    <link name="${robot_namespace}/base_link">-->
       <inertial>
         <mass value="${mass}" />
@@ -48,10 +49,12 @@
         <origin xyz="0 0 0" rpy="0 0 0" />
         <geometry>
-          <xacro:if value="${use_mesh_file}">
+<!--          <xacro:if value="${use_mesh_file}">
             <mesh filename="${mesh_file}" scale="1 1 1" />
           </xacro:if>
           <xacro:unless value="${use_mesh_file}">
             <box size="${length} ${width} ${height}" />
-          </xacro:unless>
+          </xacro:unless>-->
+          <mesh filename="package://rotors_gazebo/models/body.dae"
+              scale="0.2 0.2 0.2" />
         </geometry>
       </visual>
@@ -72,7 +75,7 @@
       </plugin>
     </gazebo>
-    <gazebo reference="${robot_namespace}/base_link">
-      <material>Gazebo/${color}</material>
-    </gazebo>
+<!--    <gazebo reference="${robot_namespace}/base_link">
+      <material>Gazebo/${color}</material>
+    </gazebo>-->
   </xacro:macro>
   <!-- Wheel joint and link -->

File: rotors_description/urdf/techpod.xacro (robot description, xacro)
@@ -25,7 +25,7 @@
   <xacro:property name="PI" value="3.1415926535897931" />
   <!-- Component masses -->
-  <xacro:property name="mass_fuselage" value="2.0" /> <!-- [kg] -->
+  <xacro:property name="mass_fuselage" value="2.65" /> <!-- [kg] -->
   <xacro:property name="mass_wheel" value="0.05" /> <!-- [kg] -->
-  <xacro:property name="mass_wing" value="0.5" /> <!-- [kg] -->
+  <xacro:property name="mass_wing" value="0.25" /> <!-- [kg] -->
   <xacro:property name="mass_vertical_stabilizer" value="0.2" /> <!-- [kg] -->
   <xacro:property name="mass_tail" value="0.15" /> <!-- [kg] -->
@@ -35,7 +35,10 @@
   <xacro:property name="mass_rudder" value="0.1" /> <!-- [kg] -->
   <!-- Fuselage properties -->
-  <xacro:property name="body_length" value="2.0" /> <!-- [m] -->
-  <xacro:property name="body_width" value="0.1" /> <!-- [m] -->
-  <xacro:property name="body_height" value="0.1" /> <!-- [m] -->
+  <!--<xacro:property name="body_length" value="2.0" />
+  <xacro:property name="body_width" value="0.1" />
+  <xacro:property name="body_height" value="0.1" />-->
+  <xacro:property name="body_length" value="1.33" /> <!-- [m] -->
+  <xacro:property name="body_width" value="0.85" /> <!-- [m] -->
+  <xacro:property name="body_height" value="0.25" /> <!-- [m] -->
   <xacro:property name="body_color" value="Red" />
   <!-- Wheel properties -->
@@ -181,5 +184,5 @@
     radius="${wheel_radius}"
     width="${wheel_width}">
-    <origin xyz="0.75 0.1 -0.1" rpy="${0.5 * PI} 0.0 0.0" />
+    <origin xyz="0.5 0.2 -0.1" rpy="${0.5 * PI} 0.0 0.0" />
     <xacro:insert_block name="wheel_inertia" />
   </xacro:wheel>
@@ -194,5 +197,5 @@
     radius="${wheel_radius}"
     width="${wheel_width}">
-    <origin xyz="0.75 -0.1 -0.1" rpy="${0.5 * PI} 0.0 0.0" />
+    <origin xyz="0.5 -0.2 -0.1" rpy="${0.5 * PI} 0.0 0.0" />
     <xacro:insert_block name="wheel_inertia" />
   </xacro:wheel>
@@ -211,5 +214,5 @@
   </xacro:wheel>-->
   <!-- Instantiate wings -->
-  <xacro:aero_surface
+<!--  <xacro:aero_surface
     robot_namespace="${namespace}"
     surface_name="wing_left"
@@ -229,6 +232,6 @@
     mesh="">
     <axis xyz="1 0 0" />
-    <origin xyz="0.5 ${-0.5 * body_width} 0.0" rpy="0.0 0.0 0.0" />
-    <origin xyz="0.0 ${-0.5 * wing_width} 0.0" rpy="0.0 0.0 0.0" />
+    <origin xyz="0.5 ${0.5 * body_width} 0.0" rpy="0.0 0.0 0.0" />
+    <origin xyz="0.0 ${0.5 * wing_width} 0.0" rpy="0.0 0.0 0.0" />
     <xacro:insert_block name="wing_inertia" />
   </xacro:aero_surface>
@@ -251,10 +254,10 @@
     mesh="">
     <axis xyz="1 0 0" />
-    <origin xyz="0.5 ${0.5 * body_width} 0.0" rpy="0.0 0.0 0.0" />
-    <origin xyz="0.0 ${0.5 * wing_width} 0.0" rpy="0.0 0.0 0.0" />
+    <origin xyz="0.5 ${-0.5 * body_width} 0.0" rpy="0.0 0.0 0.0" />
+    <origin xyz="0.0 ${-0.5 * wing_width} 0.0" rpy="0.0 0.0 0.0" />
     <xacro:insert_block name="wing_inertia" />
-  </xacro:aero_surface>
+  </xacro:aero_surface>-->
   <!-- Instantiate the vertical stabilizer -->
-  <xacro:vertical_stabilizer
+<!--  <xacro:vertical_stabilizer
     robot_namespace="${namespace}"
     parent="${namespace}/base_link"
@@ -266,9 +269,9 @@
     use_mesh="false"
     mesh="">
-    <origin xyz="${-0.5 * body_length + 0.5 * vertical_stabilizer_length} 0.0 ${-0.5 * (body_height + vertical_stabilizer_height)}" rpy="0.0 0.0 0.0" />
+    <origin xyz="${-0.5 * body_length + 0.5 * vertical_stabilizer_length} 0.0 ${0.5 * (body_height + vertical_stabilizer_height)}" rpy="0.0 0.0 0.0" />
     <xacro:insert_block name="vertical_stabilizer_inertia" />
-  </xacro:vertical_stabilizer>
+  </xacro:vertical_stabilizer>-->
   <!-- Instantiate the tail -->
-  <xacro:aero_surface
+<!--  <xacro:aero_surface
     robot_namespace="${namespace}"
     surface_name="tail_left"
@@ -288,6 +291,6 @@
     mesh="">
     <axis xyz="1 0 0" />
-    <origin xyz="${0.5 * elevator_length} ${-0.5 * vertical_stabilizer_width} ${-0.5 * (vertical_stabilizer_height - tail_height)}" rpy="0.0 0.0 0.0" />
-    <origin xyz="0.0 ${-0.5 * tail_width} 0.0" rpy="0.0 0.0 0.0" />
+    <origin xyz="${0.5 * elevator_length} ${0.5 * vertical_stabilizer_width} ${0.5 * (vertical_stabilizer_height - tail_height)}" rpy="0.0 0.0 0.0" />
+    <origin xyz="0.0 ${0.5 * tail_width} 0.0" rpy="0.0 0.0 0.0" />
     <xacro:insert_block name="tail_inertia" />
   </xacro:aero_surface>
@@ -310,8 +313,8 @@
     mesh="">
     <axis xyz="1 0 0" />
-    <origin xyz="${0.5 * elevator_length} ${0.5 * vertical_stabilizer_width} ${-0.5 * (vertical_stabilizer_height - tail_height)}" rpy="0.0 0.0 0.0" />
-    <origin xyz="0.0 ${0.5 * tail_width} 0.0" rpy="0.0 0.0 0.0" />
+    <origin xyz="${0.5 * elevator_length} ${-0.5 * vertical_stabilizer_width} ${0.5 * (vertical_stabilizer_height - tail_height)}" rpy="0.0 0.0 0.0" />
+    <origin xyz="0.0 ${-0.5 * tail_width} 0.0" rpy="0.0 0.0 0.0" />
     <xacro:insert_block name="tail_inertia" />
-  </xacro:aero_surface>
+  </xacro:aero_surface>-->
   <!-- Instantiate the ailerons -->
 <!--  <xacro:aero_surface

Commit message: Adding view control and a gui for selecting view point

File: rotors_description/urdf/fixed_wing_base.xacro (robot description, xacro)
@@ -40,5 +40,4 @@
     </joint>
     <link name="${robot_namespace}/base_link_inertia">
-<!--    <link name="${robot_namespace}/base_link">-->
       <inertial>
         <mass value="${mass}" />

Commit message: Fixing the orientatio of the airplane to the standard downward-facing frame

File: rotors_description/urdf/fixed_wing_base.xacro (robot description, xacro)
@@ -35,5 +35,5 @@
     <link name="${robot_namespace}/base_link"></link>
     <joint name="${robot_namespace}/base_joint" type="fixed">
-      <origin xyz="0 0 0" rpy="0 0 0" />
+      <origin xyz="0 0 0" rpy="3.1415926535897931 0 0" />
       <parent link="${robot_namespace}/base_link" />
       <child link="${robot_namespace}/base_link_inertia" />
@@ -42,5 +42,5 @@
       <inertial>
         <mass value="${mass}" />
-        <xacro:insert_block name="cog" />
+        <origin xyz="0 0 0" rpy="0 0 0" />
         <xacro:insert_block name="inertia" />
       </inertial>

Commit message: Adding the techpod body mesh

File: rotors_description/urdf/fixed_wing_base.xacro (robot description, xacro)
@@ -54,5 +54,5 @@
             <box size="${length} ${width} ${height}" />
           </xacro:unless>-->
-          <mesh filename="package://rotors_gazebo/models/body.dae"
+          <mesh filename="package://rotors_description/meshes/techpod/techpod_body.dae"
               scale="0.2 0.2 0.2" />
         </geometry>
