Commit message: Applying new description of techpod

File: rotors_description/urdf/techpod.xacro (robot description, xacro)
@@ -14,71 +14,55 @@
 <robot name="techpod" xmlns:xacro="http://ros.org/wiki/xacro">
   <!-- Global properties -->
-  <xacro:property name="namespace" value="$(arg uav_name)" />
-  <xacro:property name="propeller_velocity_slowdown_sim" value="10" />
+  <xacro:property name="namespace" value="$(arg namespace)" />
+  <xacro:property name="rotor_velocity_slowdown_sim" value="10" />
   <xacro:property name="use_mesh" value="true" />
   <!-- Constants -->
   <xacro:property name="PI" value="3.1415926535897931" />
   <!-- Component masses -->
-  <xacro:property name="mass_fuselage" value="2.65" /> <!-- [kg] -->
-  <xacro:property name="mass_wheel" value="0.05" /> <!-- [kg] -->
-  <xacro:property name="mass_wing" value="0.25" /> <!-- [kg] -->
-  <xacro:property name="mass_vertical_stabilizer" value="0.2" /> <!-- [kg] -->
-  <xacro:property name="mass_tail" value="0.15" /> <!-- [kg] -->
-  <xacro:property name="mass_propeller" value="0.01" /> <!-- [kg] -->
+  <xacro:property name="mass_fuselage" value="2.15" /> <!-- [kg] -->
   <xacro:property name="mass_aileron" value="0.2" /> <!-- [kg] -->
   <xacro:property name="mass_elevator" value="0.1" /> <!-- [kg] -->
   <xacro:property name="mass_rudder" value="0.1" /> <!-- [kg] -->
-  <!-- Fuselage properties -->
-  <xacro:property name="body_length" value="1.33" /> <!-- [m] -->
-  <xacro:property name="body_width" value="2.65" /> <!-- [m] -->
-  <xacro:property name="body_height" value="0.25" /> <!-- [m] -->
+  <xacro:property name="mass_propeller" value="0.1" /> <!-- [kg] -->
+  <!-- Main body properties -->
+  <xacro:property name="body_length" value="1.088" /> <!-- [m] -->
+  <xacro:property name="body_width" value="2.591" /> <!-- [m] -->
+  <xacro:property name="body_height" value="0.303" /> <!-- [m] -->
   <xacro:property name="body_color" value="Gray" />
+  <!-- Aileron properties -->
+  <xacro:property name="aileron_length" value="0.053" /> <!-- [m] -->
+  <xacro:property name="aileron_width" value="0.349" /> <!-- [m] -->
+  <xacro:property name="aileron_height" value="0.013" /> <!-- [m] -->
+  <xacro:property name="aileron_min_angle" value="-0.349066" /> <!-- [rad] -->
+  <xacro:property name="aileron_max_angle" value="0.349066" /> <!-- [rad] -->
+  <xacro:property name="aileron_color" value="Red" />
+  <!-- Elevator properties -->
+  <xacro:property name="elevator_length" value="0.051" /> <!-- [m] -->
+  <xacro:property name="elevator_width" value="0.457" /> <!-- [m] -->
+  <xacro:property name="elevator_height" value="0.012" /> <!-- [m] -->
+  <xacro:property name="elevator_min_angle" value="-0.349066" /> <!-- [rad] -->
+  <xacro:property name="elevator_max_angle" value="0.349066" /> <!-- [rad] -->
+  <xacro:property name="elevator_color" value="Blue" />
+  <!-- Rudder properties -->
+  <xacro:property name="rudder_length" value="0.129" />
+  <xacro:property name="rudder_width" value="0.018" />
+  <xacro:property name="rudder_height" value="0.241" />
+  <xacro:property name="rudder_min_angle" value="-0.349066" />
+  <xacro:property name="rudder_max_angle" value="0.349066" />
+  <xacro:property name="rudder_color" value="Orange" />
   <!-- Propeller properties -->
-  <xacro:property name="propeller_offset" value="0.025" /> <!-- [m] -->
-  <xacro:property name="radius_propeller" value="0.15" /> <!-- [m] -->
-  <xacro:property name="motor_constant" value="2.14858e-04" /> <!-- [kg m/s^2] -->
-  <xacro:property name="moment_constant" value="0.016" /> <!-- [m] -->
-  <xacro:property name="time_constant_up" value="0.0125" /> <!-- [s] -->
-  <xacro:property name="time_constant_down" value="0.025" /> <!-- [s] -->
-  <xacro:property name="max_propeller_velocity" value="838" /> <!-- [rad/s] -->
-  <xacro:property name="rotor_drag_coefficient" value="8.06428e-05" />
-  <xacro:property name="rolling_moment_coefficient" value="0.000001" />
-  <!-- Aileron properties -->
-  <xacro:property name="aileron_length" value="${0.5 * root_chord}" />
-  <xacro:property name="aileron_width" value="${0.5 * wing_width}" />
-  <xacro:property name="aileron_height" value="0.02" />
-  <xacro:property name="aileron_gain" value="2.0" />
-  <xacro:property name="aileron_min_angle" value="-0.349066" />
-  <xacro:property name="aileron_max_angle" value="0.349066" />
-  <xacro:property name="aileron_channel" value="0" />
-  <!-- Elevator properties -->
-  <xacro:property name="elevator_length" value="0.1" />
-  <xacro:property name="elevator_width" value="0.2" />
-  <xacro:property name="elevator_height" value="0.02" />
-  <xacro:property name="elevator_gain" value="2.0" />
-  <xacro:property name="elevator_min_angle" value="-0.349066" />
-  <xacro:property name="elevator_max_angle" value="0.349066" />
-  <xacro:property name="elevator_channel" value="1" />
-  <!-- Rudder properties -->
-  <xacro:property name="rudder_length" value="0.2" /> <!-- [m] -->
-  <xacro:property name="rudder_width" value="0.1" /> <!-- [m] -->
-  <xacro:property name="rudder_height" value="0.5" /> <!-- [m] -->
-  <xacro:property name="rudder_gain" value="2.0" />
-  <xacro:property name="rudder_min_angle" value="-0.349066" /> <!-- [rad] -->
-  <xacro:property name="rudder_max_angle" value="0.349066" /> <!-- [rad] -->
-  <xacro:property name="rudder_channel" value="2" />
-  <!-- Inertia of the fuselage -->
+  <xacro:property name="propeller_direction" value="cw" />
+  <xacro:property name="propeller_radius" value="0.1" />
+  <xacro:property name="propeller_height" value="0.003" />
+  <xacro:property name="propeller_color" value="Gray" />
+  <!-- Inertia of the main body -->
   <xacro:property name="body_inertia">
-    <xacro:box_inertia x="${body_length}" y="${body_width}" z="${body_height}" mass="${mass_fuselage}" />
+    <inertia ixx="0.16632" ixy="0.0" ixz="0.0755" iyy="0.3899" iyz="0.0" izz="0.5243" />
   </xacro:property>
-  <!-- Inertia of the propeller, assuming it is a cuboid. Height=3mm, width=40mm -->
-  <xacro:property name="propeller_inertia">
-    <xacro:box_inertia x="${2.0 * radius_propeller}" y="0.04" z="0.003" mass="${mass_propeller * propeller_velocity_slowdown_sim}" />
-  </xacro:property>
-  <!-- Inertia of a single aileron, assuming it is a cuboid -->
+  <!-- Inertia of the aileron, assuming it is a cuboid -->
   <xacro:property name="aileron_inertia">
     <xacro:box_inertia x="${aileron_length}" y="${aileron_width}" z="${aileron_height}" mass="${mass_aileron}" />
   </xacro:property>
-  <!-- Inertia of a single elevator, assuming it is a cuboid -->
+  <!-- Inertia of the elevator, assuming it is a cuboid -->
   <xacro:property name="elevator_inertia">
     <xacro:box_inertia x="${elevator_length}" y="${elevator_width}" z="${elevator_height}" mass="${mass_elevator}" />
@@ -87,4 +71,8 @@
   <xacro:property name="rudder_inertia">
     <xacro:box_inertia x="${rudder_length}" y="${rudder_width}" z="${rudder_height}" mass="${mass_rudder}" />
+  </xacro:property>
+  <!-- Inertia of the propeller, assuming it is a cylinder -->
+  <xacro:property name="propeller_inertia">
+    <xacro:cylinder_inertia r="${propeller_radius}" h="${propeller_height}" mass="${mass_propeller*rotor_velocity_slowdown_sim}" />
   </xacro:property>
   <!-- Included URDF Files -->
@@ -99,91 +87,56 @@
     color="${body_color}"
     use_mesh_file="${use_mesh}"
-    mesh_file="package://rotors_description/meshes/techpod/techpod_body.dae"
-    reset_model_service_name="reset_model">
-    <origin xyz="0 0 0" rpy="3.1415926535897931 0 0" />
-    <inertia ixx="${0.1512 * 1.1}" ixy="0.0" ixz="0.0755" iyy="${0.2785 * 1.4}" iyz="0.0" izz="${0.3745 * 1.4}" />
-    <!--<xacro:insert_block name="body_inertia" />-->
+    mesh_file="package://rotors_description/meshes/techpod/techpod_body.dae">
+    <origin xyz="0 0 0" rpy="${PI} 0 0" />
+    <xacro:insert_block name="body_inertia" />
   </xacro:fixed_wing_base_macro>
-  <!-- Instantiate the propeller -->
-<!--  <xacro:propeller
-    robot_namespace="${namespace}"
-    direction="cw"
-    motor_constant="${motor_constant}"
-    moment_constant="${moment_constant}"
-    parent="${namespace}/base_link"
-    mass="${mass_propeller}"
-    radius="${radius_propeller}"
-    time_constant_up="${time_constant_up}"
-    time_constant_down="${time_constant_down}"
-    max_propeller_velocity="${max_propeller_velocity}"
-    motor_number="0"
-    rotor_drag_coefficient="${rotor_drag_coefficient}"
-    rolling_moment_coefficient="${rolling_moment_coefficient}"
-    color="Blue"
-    use_own_mesh="false"
-    mesh="">
-    <origin xyz="${0.5 * body_length + propeller_offset} 0.0 0.0" rpy="0.0 ${0.5 * PI} 0.0" />
-    <xacro:insert_block name="propeller_inertia" />
-  </xacro:propeller>-->
   <!-- Instantiate the ailerons -->
-<!--  <xacro:aero_surface
+  <xacro:control_surface
     robot_namespace="${namespace}"
     surface_name="aileron_left"
-    surface_type="aileron"
-    parent="${namespace}/wing_left"
+    parent="${namespace}/base_link"
     mass_surface="${mass_aileron}"
-    joint_gain="${aileron_gain}"
-    positive_direction="ccw"
     min_angle="${aileron_min_angle}"
     max_angle="${aileron_max_angle}"
-    channel="${aileron_channel}"
-    color="Orange"
-    use_mesh="false"
-    mesh=""
+    color="${aileron_color}"
+    use_mesh_file="${use_mesh}"
+    mesh_file="package://rotors_description/meshes/techpod/techpod_aileron_left.dae"
+    surface_length="${aileron_length}"
+    surface_width="${aileron_width}"
+    surface_height="${aileron_height}">
+    <axis xyz="0 -1 0" />
+    <origin xyz="0.1095 -0.99245 -0.115" rpy="0.0 0.0 0.0" />
+    <origin xyz="0.0 0.0 0.0" rpy="${PI} 0.0 0.0" />
+    <xacro:insert_block name="aileron_inertia" />
+  </xacro:control_surface>
+  <xacro:control_surface
+    robot_namespace="${namespace}"
+    surface_name="aileron_right"
+    parent="${namespace}/base_link"
+    mass_surface="${mass_aileron}"
+    min_angle="${aileron_min_angle}"
+    max_angle="${aileron_max_angle}"
+    color="${aileron_color}"
+    use_mesh_file="${use_mesh}"
+    mesh_file="package://rotors_description/meshes/techpod/techpod_aileron_right.dae"
     surface_length="${aileron_length}"
     surface_width="${aileron_width}"
     surface_height="${aileron_height}">
     <axis xyz="0 1 0" />
-    <origin xyz="${-0.5 * root_chord} ${wing_width - 0.5 * aileron_width} 0.0" rpy="0.0 0.0 0.0" />
-    <origin xyz="${-0.5 * aileron_length} 0.0 0.0" rpy="0.0 0.0 0.0" />
+    <origin xyz="0.1095 0.99245 -0.115" rpy="0.0 0.0 0.0" />
+    <origin xyz="0.0 0.0 0.0" rpy="${PI} 0.0 0.0" />
     <xacro:insert_block name="aileron_inertia" />
-  </xacro:aero_surface>
-  <xacro:aero_surface
-    robot_namespace="${namespace}"
-    surface_name="aileron_right"
-    surface_type="aileron"
-    parent="${namespace}/wing_right"
-    mass_surface="${mass_aileron}"
-    joint_gain="${aileron_gain}"
-    positive_direction="cw"
-    min_angle="${aileron_min_angle}"
-    max_angle="${aileron_max_angle}"
-    channel="${aileron_channel}"
-    color="Orange"
-    use_mesh="false"
-    mesh=""
-    surface_length="${aileron_length}"
-    surface_width="${aileron_width}"
-    surface_height="${aileron_height}">
-    <axis xyz="0 1 0" />
-    <origin xyz="${-0.5 * root_chord} ${-(wing_width - 0.5 * aileron_width)} 0.0" rpy="0.0 0.0 0.0" />
-    <origin xyz="${-0.5 * aileron_length} 0.0 0.0" rpy="0.0 0.0 0.0" />
-    <xacro:insert_block name="aileron_inertia" />
-  </xacro:aero_surface>-->
-  <!-- Instantiate the elevators -->
-  <!--<xacro:aero_surface
+  </xacro:control_surface>
+  <!-- Instantiate the elevator(s) -->
+  <xacro:control_surface
     robot_namespace="${namespace}"
     surface_name="elevator"
-    surface_type="elevator"
     parent="${namespace}/base_link"
     mass_surface="${mass_elevator}"
-    joint_gain="${elevator_gain}"
-    positive_direction="ccw"
     min_angle="${elevator_min_angle}"
     max_angle="${elevator_max_angle}"
-    channel="${elevator_channel}"
-    color="Gray"
-    use_mesh="true"
-    mesh="package://rotors_description/meshes/techpod/techpod_elevator.dae"
+    color="${elevator_color}"
+    use_mesh_file="${use_mesh}"
+    mesh_file="package://rotors_description/meshes/techpod/techpod_elevator.dae"
     surface_length="${elevator_length}"
     surface_width="${elevator_width}"
@@ -193,27 +146,36 @@
     <origin xyz="0.0 0.0 0.0" rpy="${PI} 0.0 0.0" />
     <xacro:insert_block name="elevator_inertia" />
-  </xacro:aero_surface>-->
+  </xacro:control_surface>
   <!-- Instantiate the rudder -->
-  <!--<xacro:aero_surface
+  <xacro:control_surface
     robot_namespace="${namespace}"
     surface_name="rudder"
-    surface_type="rudder"
     parent="${namespace}/base_link"
     mass_surface="${mass_rudder}"
-    joint_gain="${rudder_gain}"
-    positive_direction="cw"
     min_angle="${rudder_min_angle}"
     max_angle="${rudder_max_angle}"
-    channel="${rudder_channel}"
-    color="Gray"
-    use_mesh="true"
-    mesh="package://rotors_description/meshes/techpod/techpod_rudder.dae"
+    color="${rudder_color}"
+    use_mesh_file="${use_mesh}"
+    mesh_file="package://rotors_description/meshes/techpod/techpod_rudder.dae"
     surface_length="${rudder_length}"
     surface_width="${rudder_width}"
     surface_height="${rudder_height}">
     <axis xyz="0 0 1" />
-    <origin xyz="0.0 0.0 0.0" rpy="0.0 0.0 0.0" />
-    <origin xyz="0.0 0.0 0.0" rpy="0.0 0.0 0.0" />
+    <origin xyz="-0.428 0.0 0.0" rpy="0.0 0.25 0.0" />
+    <origin xyz="0.0 0.0 0.0" rpy="${PI} -0.25 0.0" />
     <xacro:insert_block name="rudder_inertia" />
-  </xacro:aero_surface>-->
+  </xacro:control_surface>
+  <!-- Instantiate the propeller -->
+  <xacro:propeller
+    robot_namespace="${namespace}"
+    suffix=""
+    parent="${namespace}/base_link"
+    mass_propeller="${mass_propeller}"
+    propeller_radius="${propeller_radius}"
+    color="${propeller_color}"
+    use_mesh_file="${use_mesh}"
+    mesh_file="package://rotors_description/meshes/propeller_${propeller_direction}.dae">
+    <origin xyz="-0.025 0.0 -0.15" rpy="0.0 ${-0.5*PI} 0.0" />
+    <xacro:insert_block name="propeller_inertia" />
+  </xacro:propeller>
 </robot>

Commit message: Adding flaps to techpod and service for registering control surfaces

File: rotors_description/urdf/fixed_wing_base.xacro (robot description, xacro)
@@ -71,6 +71,6 @@
   <!-- Control surface joint and link -->
   <xacro:macro name="control_surface"
-    params="robot_namespace surface_name parent mass_surface min_angle
-      max_angle color use_mesh_file mesh_file surface_length surface_width
+    params="robot_namespace surface_name parent mass_surface surface_type
+      min_angle max_angle color use_mesh_file mesh_file surface_length surface_width
       surface_height *axis *joint_origin *link_origin *inertia">
     <joint name="${robot_namespace}/${surface_name}_joint" type="revolute">
@@ -110,4 +110,13 @@
       </collision>
     </link>
+    <gazebo>
+      <plugin name="${robot_namespace}_base" filename="librotors_gazebo_control_surface_plugin.so">
+        <robotNamespace>${robot_namespace}</robotNamespace>
+        <jointName>${robot_namespace}/${surface_name}_joint</jointName>
+        <surfaceType>${surface_type}</surfaceType>
+        <angleMin>${min_angle}</angleMin>
+        <angleMax>${max_angle}</angleMax>
+      </plugin>
+    </gazebo>
     <gazebo reference="${robot_namespace}/${surface_name}">
       <material>Gazebo/${color}</material>

File: rotors_description/urdf/techpod.xacro (robot description, xacro)
@@ -20,6 +20,7 @@
   <xacro:property name="PI" value="3.1415926535897931" />
   <!-- Component masses -->
-  <xacro:property name="mass_fuselage" value="2.15" /> <!-- [kg] -->
-  <xacro:property name="mass_aileron" value="0.2" /> <!-- [kg] -->
+  <xacro:property name="mass_fuselage" value="2.05" /> <!-- [kg] -->
+  <xacro:property name="mass_aileron" value="0.1" /> <!-- [kg] -->
+  <xacro:property name="mass_flap" value="0.1" /> <!-- [kg] -->
   <xacro:property name="mass_elevator" value="0.1" /> <!-- [kg] -->
   <xacro:property name="mass_rudder" value="0.1" /> <!-- [kg] -->
@@ -37,4 +38,11 @@
   <xacro:property name="aileron_max_angle" value="0.349066" /> <!-- [rad] -->
   <xacro:property name="aileron_color" value="Red" />
+  <!-- Flap properties -->
+  <xacro:property name="flap_length" value="0.076" /> <!-- [m] -->
+  <xacro:property name="flap_width" value="0.459" /> <!-- [m] -->
+  <xacro:property name="flap_height" value="0.016" /> <!-- [m] -->
+  <xacro:property name="flap_min_angle" value="0.0" /> <!-- [rad] -->
+  <xacro:property name="flap_max_angle" value="0.0" /> <!-- [rad] -->
+  <xacro:property name="flap_color" value="Yellow" />
   <!-- Elevator properties -->
   <xacro:property name="elevator_length" value="0.051" /> <!-- [m] -->
@@ -64,4 +72,8 @@
     <xacro:box_inertia x="${aileron_length}" y="${aileron_width}" z="${aileron_height}" mass="${mass_aileron}" />
   </xacro:property>
+  <!-- Inertia of the flap, assuming it is a cuboid -->
+  <xacro:property name="flap_inertia">
+    <xacro:box_inertia x="${flap_length}" y="${flap_width}" z="${flap_height}" mass="${mass_flap}" />
+  </xacro:property>
   <!-- Inertia of the elevator, assuming it is a cuboid -->
   <xacro:property name="elevator_inertia">
@@ -97,4 +109,5 @@
     parent="${namespace}/base_link"
     mass_surface="${mass_aileron}"
+    surface_type="aileron"
     min_angle="${aileron_min_angle}"
     max_angle="${aileron_max_angle}"
@@ -115,4 +128,5 @@
     parent="${namespace}/base_link"
     mass_surface="${mass_aileron}"
+    surface_type="aileron"
     min_angle="${aileron_min_angle}"
     max_angle="${aileron_max_angle}"
@@ -128,4 +142,43 @@
     <xacro:insert_block name="aileron_inertia" />
   </xacro:control_surface>
+  <!-- Instantiate the flaps -->
+  <xacro:control_surface
+    robot_namespace="${namespace}"
+    surface_name="flap_left"
+    parent="${namespace}/base_link"
+    mass_surface="${mass_flap}"
+    surface_type="flap"
+    min_angle="${flap_min_angle}"
+    max_angle="${flap_max_angle}"
+    color="${flap_color}"
+    use_mesh_file="${use_mesh}"
+    mesh_file="package://rotors_description/meshes/techpod/techpod_flap_left.dae"
+    surface_length="${flap_length}"
+    surface_width="${flap_width}"
+    surface_height="${flap_height}">
+    <axis xyz="0 -1 0" />
+    <origin xyz="0.101 -0.382 -0.1185" rpy="0.0 0.0 0.0" />
+    <origin xyz="0.0 0.0 0.0" rpy="${PI} 0.0 0.0" />
+    <xacro:insert_block name="flap_inertia" />
+  </xacro:control_surface>
+  <xacro:control_surface
+    robot_namespace="${namespace}"
+    surface_name="flap_right"
+    parent="${namespace}/base_link"
+    mass_surface="${mass_flap}"
+    surface_type="flap"
+    min_angle="${flap_min_angle}"
+    max_angle="${flap_max_angle}"
+    color="${flap_color}"
+    use_mesh_file="${use_mesh}"
+    mesh_file="package://rotors_description/meshes/techpod/techpod_flap_right.dae"
+    surface_length="${flap_length}"
+    surface_width="${flap_width}"
+    surface_height="${flap_height}">
+    <axis xyz="0 1 0" />
+    <origin xyz="0.101 0.382 -0.1185" rpy="0.0 0.0 0.0" />
+    <origin xyz="0.0 0.0 0.0" rpy="${PI} 0.0 0.0" />
+    <xacro:insert_block name="flap_inertia" />
+  </xacro:control_surface>
   <!-- Instantiate the elevator(s) -->
   <xacro:control_surface
@@ -134,4 +187,5 @@
     parent="${namespace}/base_link"
     mass_surface="${mass_elevator}"
+    surface_type="elevator"
     min_angle="${elevator_min_angle}"
     max_angle="${elevator_max_angle}"
@@ -153,4 +207,5 @@
     parent="${namespace}/base_link"
     mass_surface="${mass_rudder}"
+    surface_type="rudder"
     min_angle="${rudder_min_angle}"
     max_angle="${rudder_max_angle}"

Commit message: Fixing control surface actuation

File: rotors_description/urdf/fixed_wing_base.xacro (robot description, xacro)
@@ -79,5 +79,5 @@
       <parent link="${parent}" />
       <child link="${robot_namespace}/${surface_name}" />
-      <limit upper="${max_angle}" lower="${min_angle}" effort="0" velocity="0" />
+      <limit upper="${max_angle}" lower="${min_angle}" effort="5" velocity="1" />
     </joint>
     <link name="${robot_namespace}/${surface_name}">

File: rotors_description/urdf/techpod.xacro (robot description, xacro)
@@ -118,5 +118,5 @@
     surface_width="${aileron_width}"
     surface_height="${aileron_height}">
-    <axis xyz="0 -1 0" />
+    <axis xyz="0 1 0" />
     <origin xyz="0.1095 -0.99245 -0.115" rpy="0.0 0.0 0.0" />
     <origin xyz="0.0 0.0 0.0" rpy="${PI} 0.0 0.0" />
@@ -137,5 +137,5 @@
     surface_width="${aileron_width}"
     surface_height="${aileron_height}">
-    <axis xyz="0 1 0" />
+    <axis xyz="0 -1 0" />
     <origin xyz="0.1095 0.99245 -0.115" rpy="0.0 0.0 0.0" />
     <origin xyz="0.0 0.0 0.0" rpy="${PI} 0.0 0.0" />
@@ -216,5 +216,5 @@
     surface_width="${rudder_width}"
     surface_height="${rudder_height}">
-    <axis xyz="0 0 1" />
+    <axis xyz="0 0 -1" />
     <origin xyz="-0.428 0.0 0.0" rpy="0.0 0.25 0.0" />
     <origin xyz="0.0 0.0 0.0" rpy="${PI} -0.25 0.0" />
