Commit message: Adding the rotors_gazebo_gui_plugins package

File: rotors_description/urdf/fixed_wing_base.xacro (robot description, xacro)
@@ -55,10 +55,5 @@
         <origin xyz="0 0 0" rpy="0 0 0" />
         <geometry>
-          <xacro:if value="${use_mesh_file}">
-            <mesh filename="${mesh_file}" scale="1 1 1" />
-          </xacro:if>
-          <xacro:unless value="${use_mesh_file}">
-            <box size="${length} ${width} ${height}" />
-          </xacro:unless>
+          <box size="${length} ${width} ${height}" />
         </geometry>
       </collision>

File: rotors_description/urdf/techpod.xacro (robot description, xacro)
@@ -88,5 +88,5 @@
     use_mesh_file="${use_mesh}"
     mesh_file="package://rotors_description/meshes/techpod/techpod_body.dae">
-    <origin xyz="0 0 0" rpy="${PI} 0 0" />
+    <origin xyz="0 0 0" rpy="0 0 0" />
     <xacro:insert_block name="body_inertia" />
   </xacro:fixed_wing_base_macro>
@@ -106,6 +106,6 @@
     surface_height="${aileron_height}">
     <axis xyz="0 -1 0" />   <!-- Joint axis -->
-    <origin xyz="0.1095 -0.99245 -0.115" rpy="0.0 0.0 0.0" />   <!-- Joint origin -->
-    <origin xyz="0.0 0.0 0.0" rpy="${PI} 0.0 0.0" />   <!-- Link origin -->
+    <origin xyz="0.1095 0.99245 0.115" rpy="0.0 0.0 0.0" />   <!-- Joint origin -->
+    <origin xyz="0.0 0.0 0.0" rpy="0.0 0.0 0.0" />   <!-- Link origin -->
     <xacro:insert_block name="aileron_inertia" />
   </xacro:control_surface>
@@ -124,6 +124,6 @@
     surface_height="${aileron_height}">
     <axis xyz="0 1 0" />   <!-- Joint axis -->
-    <origin xyz="0.1095 0.99245 -0.115" rpy="0.0 0.0 0.0" />   <!-- Joint origin -->
-    <origin xyz="0.0 0.0 0.0" rpy="${PI} 0.0 0.0" />   <!-- Link origin -->
+    <origin xyz="0.1095 -0.99245 0.115" rpy="0.0 0.0 0.0" />   <!-- Joint origin -->
+    <origin xyz="0.0 0.0 0.0" rpy="0.0 0.0 0.0" />   <!-- Link origin -->
     <xacro:insert_block name="aileron_inertia" />
   </xacro:control_surface>
@@ -142,7 +142,7 @@
     surface_width="${elevator_width}"
     surface_height="${elevator_height}">
-    <axis xyz="0 1 0" />   <!-- Joint axis -->
-    <origin xyz="-0.555 0.0 -0.26" rpy="0.0 0.0 0.0" />   <!-- Joint origin -->
-    <origin xyz="0.0 0.0 0.0" rpy="${PI} 0.0 0.0" />   <!-- Link origin -->
+    <axis xyz="0 -1 0" />   <!-- Joint axis -->
+    <origin xyz="-0.555 0.0 0.26" rpy="0.0 0.0 0.0" />   <!-- Joint origin -->
+    <origin xyz="0.0 0.0 0.0" rpy="0.0 0.0 0.0" />   <!-- Link origin -->
     <xacro:insert_block name="elevator_inertia" />
   </xacro:control_surface>
@@ -162,10 +162,10 @@
     surface_height="${rudder_height}">
     <axis xyz="0 0 1" />   <!-- Joint axis -->
-    <origin xyz="-0.428 0.0 0.0" rpy="0.0 0.25 0.0" />   <!-- Joint origin -->
-    <origin xyz="0.0 0.0 0.0" rpy="${PI} -0.25 0.0" />   <!-- Link origin -->
+    <origin xyz="-0.428 0.0 0.0" rpy="0.0 -0.25 0.0" />   <!-- Joint origin -->
+    <origin xyz="0.0 0.0 0.0" rpy="0.0 0.25 0.0" />   <!-- Link origin -->
     <xacro:insert_block name="rudder_inertia" />
   </xacro:control_surface>
   <!-- Instantiate the propeller -->
-  <xacro:propeller
+  <!--<xacro:propeller
     robot_namespace="${namespace}"
     suffix=""
@@ -178,4 +178,4 @@
     <origin xyz="-0.025 0.0 -0.15" rpy="0.0 ${-0.5*PI} 0.0" />
     <xacro:insert_block name="propeller_inertia" />
-  </xacro:propeller>
+  </xacro:propeller>-->
 </robot>

Commit message: Adding joystick interface for fixed-wing aircraft

File: rotors_description/urdf/fixed_wing_base.xacro (robot description, xacro)
@@ -28,5 +28,5 @@
   <xacro:macro name="fixed_wing_base_macro"
     params="robot_namespace mass length width height color use_mesh_file
-      mesh_file *origin *inertia">
+      mesh_file joy_input *origin *inertia">
     <link name="${robot_namespace}/base_link"></link>
     <joint name="${robot_namespace}/base_joint" type="fixed">
@@ -60,8 +60,8 @@
     </link>
     <gazebo>
-      <!--<plugin name="${robot_namespace}_base" filename="librotors_gazebo_fixedwing_base_plugin.so">-->
       <plugin name="${robot_namespace}_base" filename="librotors_gazebo_aerodynamics_plugin.so">
         <robotNamespace>${robot_namespace}</robotNamespace>
         <linkName>${robot_namespace}/base_link</linkName>
+        <joyInput>${joy_input}</joyInput>
       </plugin>
     </gazebo>

File: rotors_description/urdf/techpod.xacro (robot description, xacro)
@@ -17,4 +17,5 @@
   <xacro:property name="rotor_velocity_slowdown_sim" value="10" />
   <xacro:property name="use_mesh" value="true" />
+  <xacro:property name="joy_input" value="$(arg joy_input)" />
   <!-- Constants -->
   <xacro:property name="PI" value="3.1415926535897931" />
@@ -100,5 +101,6 @@
     color="${body_color}"
     use_mesh_file="${use_mesh}"
-    mesh_file="package://rotors_description/meshes/techpod/techpod_body.dae">
+    mesh_file="package://rotors_description/meshes/techpod/techpod_body.dae"
+    joy_input="${joy_input}">
     <origin xyz="0 0 0" rpy="0 0 0" />
     <xacro:insert_block name="body_inertia" />
